File: BMS_hw/BMSV1.0.brd (EAGLE design)
At the start: 272 x 60 mm, 181 parts, among them IC1 MC33771BEP, IC2 SFH6156, IC3 MIC28515V1, J2 NTC, X2 87758-1816

Commit message: push_2
Parts:
- CELL1+, CELL1-, CELL10+, CELL11+, CELL12+, CELL13+, CELL14+, CELL2+, CELL3+, CELL4+, CELL5+, CELL6+, CELL7+, CELL8+, CELL9+: device GreenFuel:GF_BMS_CELL_PAD -> GreenFuel:CELL_PAD
- moved R8 7.62 mm to (-21.6, -83.8)
Connections:
- removed net CS: IC1.41
- removed net N$14: C9.1, R7.2, R8.2
- net GND: now also C9.1, R7.2, R8.2

Commit message: push_3
Parts:
- added D1: 8.2v, diode:SOD80C
- added R29, R30: 10k, adafruit:R0805
- added T1, T2, T3, T4: IPT020N10N3V1, GreenFuel:PG-HSOF-9
Connections:
- new net CHG_MOSFET: D1.C, R30.2, T1.1, T3.1
- new net DSG_MOSFET: R29.2, T2.1, T4.1
- new net N$29: T1.10, T1.11, T1.9, T2.10, T2.11, T2.9, T3.10, T3.11, T3.9, T4.10, T4.11, T4.9
- new net N$61: R29.1, T2.2, T2.3, T2.4, T2.5, T2.6, T2.7, T2.8, T4.2, T4.3, T4.4, T4.5, T4.6, T4.7, T4.8
- new net N$67: D1.A, R30.1, T1.2, T1.3, T1.4, T1.5, T1.6, T1.7, T1.8, T3.2, T3.3, T3.4, T3.5, T3.6, T3.7, T3.8
Changed lines of the file:
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@@
 <element name="C26" library="adafruit" package="C0805" value="47nF" x="-111.5" y="-225.5"/>
 <element name="R25" library="adafruit" package="R0805" value="127E" x="-111.5" y="-231.5"/>
+<element name="T1" library="GreenFuel" package="PG-HSOF-9" value="IPT020N10N3V1" x="-121.92" y="-223.52"/>
+<element name="T2" library="GreenFuel" package="PG-HSOF-9" value="IPT020N10N3V1" x="-121.92" y="-243.84"/>
+<element name="T3" library="GreenFuel" package="PG-HSOF-9" value="IPT020N10N3V1" x="-121.92" y="-264.16"/>
+<element name="T4" library="GreenFuel" package="PG-HSOF-9" value="IPT020N10N3V1" x="-121.92" y="-284.48"/>
+<element name="R29" library="adafruit" package="R0805" value="10k" x="-124.46" y="-299.72"/>
+<element name="R30" library="adafruit" package="R0805" value="10k" x="-124.46" y="-307.34"/>
+<element name="D1" library="diode" library_urn="urn:adsk.eagle:library:210" package="SOD80C" package3d_urn="urn:adsk.eagle:package:43405/2" value="8.2v" x="-124.46" y="-314.96"/>
 </elements>
 <signals>
@@
 <wire x1="-108.5" y1="-160.617" x2="-112.5" y2="-183.5" width="0" layer="19" extent="1-1"/>
 </signal>
+<signal name="N$29">
+<contactref element="T2" pad="9"/>
+<contactref element="T2" pad="10"/>
+<contactref element="T2" pad="11"/>
+<contactref element="T1" pad="11"/>
+<contactref element="T1" pad="10"/>
+<contactref element="T1" pad="9"/>
+<contactref element="T4" pad="11"/>
+<contactref element="T4" pad="10"/>
+<contactref element="T4" pad="9"/>
+<contactref element="T3" pad="11"/>
+<contactref element="T3" pad="10"/>
+<contactref element="T3" pad="9"/>
+<wire x1="-121.92" y1="-281.27" x2="-121.92" y2="-284.57" width="0" layer="19" extent="1-1"/>
+<wire x1="-121.92" y1="-279.12" x2="-121.92" y2="-281.27" width="0" layer="19" extent="1-1"/>
+<wire x1="-121.92" y1="-264.25" x2="-121.92" y2="-279.12" width="0" layer="19" extent="1-1"/>
+<wire x1="-121.92" y1="-260.95" x2="-121.92" y2="-264.25" width="0" layer="19" extent="1-1"/>
+<wire x1="-121.92" y1="-258.8" x2="-121.92" y2="-260.95" width="0" layer="19" extent="1-1"/>
+<wire x1="-121.92" y1="-243.93" x2="-121.92" y2="-258.8" width="0" layer="19" extent="1-1"/>
+<wire x1="-121.92" y1="-240.63" x2="-121.92" y2="-243.93" width="0" layer="19" extent="1-1"/>
+<wire x1="-121.92" y1="-238.48" x2="-121.92" y2="-240.63" width="0" layer="19" extent="1-1"/>
+<wire x1="-121.92" y1="-223.61" x2="-121.92" y2="-238.48" width="0" layer="19" extent="1-1"/>
+<wire x1="-121.92" y1="-220.31" x2="-121.92" y2="-223.61" width="0" layer="19" extent="1-1"/>
+<wire x1="-121.92" y1="-218.16" x2="-121.92" y2="-220.31" width="0" layer="19" extent="1-1"/>
+</signal>
+<signal name="N$61">
+<contactref element="T4" pad="8"/>
+<contactref element="T4" pad="7"/>
+<contactref element="T4" pad="6"/>
+<contactref element="T4" pad="5"/>
+<contactref element="T4" pad="4"/>
+<contactref element="T4" pad="3"/>
+<contactref element="T4" pad="2"/>
+<contactref element="T2" pad="8"/>
+<contactref element="T2" pad="7"/>
+<contactref element="T2" pad="6"/>
+<contactref element="T2" pad="5"/>
+<contactref element="T2" pad="4"/>
+<contactref element="T2" pad="3"/>
+<contactref element="T2" pad="2"/>
+<contactref element="R29" pad="1"/>
+<wire x1="-124.92" y1="-290.32" x2="-125.46" y2="-299.72" width="0" layer="19" extent="1-1"/>
+<wire x1="-123.72" y1="-290.32" x2="-124.92" y2="-290.32" width="0" layer="19" extent="1-1"/>
+<wire x1="-122.52" y1="-290.32" x2="-123.72" y2="-290.32" width="0" layer="19" extent="1-1"/>
+<wire x1="-121.32" y1="-290.32" x2="-122.52" y2="-290.32" width="0" layer="19" extent="1-1"/>
+<wire x1="-120.12" y1="-290.32" x2="-121.32" y2="-290.32" width="0" layer="19" extent="1-1"/>
+<wire x1="-118.92" y1="-290.32" x2="-120.12" y2="-290.32" width="0" layer="19" extent="1-1"/>
+<wire x1="-117.72" y1="-290.32" x2="-118.92" y2="-290.32" width="0" layer="19" extent="1-1"/>
+<wire x1="-124.92" y1="-249.68" x2="-124.92" y2="-290.32" width="0" layer="19" extent="1-1"/>
+<wire x1="-123.72" y1="-249.68" x2="-124.92" y2="-249.68" width="0" layer="19" extent="1-1"/>
+<wire x1="-122.52" y1="-249.68" x2="-123.72" y2="-249.68" width="0" layer="19" extent="1-1"/>
+<wire x1="-121.32" y1="-249.68" x2="-122.52" y2="-249.68" width="0" layer="19" extent="1-1"/>
+<wire x1="-120.12" y1="-249.68" x2="-121.32" y2="-249.68" width="0" layer="19" extent="1-1"/>
+<wire x1="-118.92" y1="-249.68" x2="-120.12" y2="-249.68" width="0" layer="19" extent="1-1"/>
+<wire x1="-117.72" y1="-249.68" x2="-118.92" y2="-249.68" width="0" layer="19" extent="1-1"/>
+</signal>
+<signal name="N$67">
+<contactref element="T3" pad="2"/>
+<contactref element="T3" pad="3"/>
+<contactref element="T3" pad="4"/>
+<contactref element="T3" pad="5"/>
+<contactref element="T3" pad="6"/>
+<contactref element="T3" pad="7"/>
+<contactref element="T3" pad="8"/>
+<contactref element="T1" pad="8"/>
+<contactref element="T1" pad="7"/>
+<contactref element="T1" pad="6"/>
+<contactref element="T1" pad="5"/>
+<contactref element="T1" pad="4"/>
+<contactref element="T1" pad="3"/>
+<contactref element="T1" pad="2"/>
+<contactref element="R30" pad="1"/>
+<contactref element="D1" pad="A"/>
+<wire x1="-125.46" y1="-307.34" x2="-122.76" y2="-314.96" width="0" layer="19" extent="1-1"/>
+<wire x1="-124.92" y1="-270" x2="-125.46" y2="-307.34" width="0" layer="19" extent="1-1"/>
+<wire x1="-123.72" y1="-270" x2="-124.92" y2="-270" width="0" layer="19" extent="1-1"/>
+<wire x1="-122.52" y1="-270" x2="-123.72" y2="-270" width="0" layer="19" extent="1-1"/>
+<wire x1="-121.32" y1="-270" x2="-122.52" y2="-270" width="0" layer="19" extent="1-1"/>
+<wire x1="-120.12" y1="-270" x2="-121.32" y2="-270" width="0" layer="19" extent="1-1"/>
+<wire x1="-118.92" y1="-270" x2="-120.12" y2="-270" width="0" layer="19" extent="1-1"/>
+<wire x1="-117.72" y1="-270" x2="-118.92" y2="-270" width="0" layer="19" extent="1-1"/>
+<wire x1="-124.92" y1="-229.36" x2="-124.92" y2="-270" width="0" layer="19" extent="1-1"/>
+<wire x1="-123.72" y1="-229.36" x2="-124.92" y2="-229.36" width="0" layer="19" extent="1-1"/>
+<wire x1="-122.52" y1="-229.36" x2="-123.72" y2="-229.36" width="0" layer="19" extent="1-1"/>
+<wire x1="-121.32" y1="-229.36" x2="-122.52" y2="-229.36" width="0" layer="19" extent="1-1"/>
+<wire x1="-120.12" y1="-229.36" x2="-121.32" y2="-229.36" width="0" layer="19" extent="1-1"/>
+<wire x1="-118.92" y1="-229.36" x2="-120.12" y2="-229.36" width="0" layer="19" extent="1-1"/>
+<wire x1="-117.72" y1="-229.36" x2="-118.92" y2="-229.36" width="0" layer="19" extent="1-1"/>
+</signal>
+<signal name="DSG_MOSFET">
+<contactref element="T4" pad="1"/>
+<contactref element="T2" pad="1"/>
+<contactref element="R29" pad="2"/>
+<wire x1="-126.12" y1="-290.32" x2="-123.46" y2="-299.72" width="0" layer="19" extent="1-1"/>
+<wire x1="-126.12" y1="-249.68" x2="-126.12" y2="-290.32" width="0" layer="19" extent="1-1"/>
+</signal>
+<signal name="CHG_MOSFET">
+<contactref element="T1" pad="1"/>
+<contactref element="T3" pad="1"/>
+<contactref element="R30" pad="2"/>
+<contactref element="D1" pad="C"/>
+<wire x1="-123.46" y1="-307.34" x2="-126.16" y2="-314.96" width="0" layer="19" extent="1-1"/>
+<wire x1="-126.12" y1="-270" x2="-123.46" y2="-307.34" width="0" layer="19" extent="1-1"/>
+<wire x1="-126.12" y1="-229.36" x2="-126.12" y2="-270" width="0" layer="19" extent="1-1"/>
+</signal>
 </signals>

Commit message: gate pull up diode added in schematic and board
Parts:
- added D2: GF1, diode:SMA-DO214AC
Connections:
- net CHG_MOSFET: now also D2.K
Changed lines of the file:
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@@
 <element name="R30" library="adafruit" package="R0805" value="10k" x="-124.46" y="-307.34"/>
 <element name="D1" library="diode" library_urn="urn:adsk.eagle:library:210" package="SOD80C" package3d_urn="urn:adsk.eagle:package:43405/2" value="8.2v" x="-124.46" y="-314.96"/>
+<element name="D2" library="diode" library_urn="urn:adsk.eagle:library:210" package="SMA-DO214AC" package3d_urn="urn:adsk.eagle:package:43452/2" value="GF1" x="-124.46" y="-322.58"/>
 </elements>
 <signals>
@@
 <contactref element="R30" pad="2"/>
 <contactref element="D1" pad="C"/>
+<contactref element="D2" pad="K"/>
+<wire x1="-126.16" y1="-314.96" x2="-122.41" y2="-322.58" width="0" layer="19" extent="1-1"/>
 <wire x1="-123.46" y1="-307.34" x2="-126.16" y2="-314.96" width="0" layer="19" extent="1-1"/>
 <wire x1="-126.12" y1="-270" x2="-123.46" y2="-307.34" width="0" layer="19" extent="1-1"/>

Commit message: chg and dsg mosfet circuit final submission
Parts:
- added Q1: IRLML5203, transistor-power:MICRO3
- added R38: 10k, adafruit:R0805
Connections:
- net DSG_MOSFET renamed DSG_GATE
- removed net CHG_MOSFET: D1.C, D2.K, R30.2, T1.1, T3.1
- new net CHG_GATE: Q1.2, T1.1
- new net N$19: D2.A, Q1.3, R38.2
- new net N$23: D1.C, D2.K, R30.2, R38.1, T3.1
- net GND: now also Q1.1
Changed lines of the file:
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@@
 <element name="D1" library="diode" library_urn="urn:adsk.eagle:library:210" package="SOD80C" package3d_urn="urn:adsk.eagle:package:43405/2" value="8.2v" x="-124.46" y="-314.96"/>
 <element name="D2" library="diode" library_urn="urn:adsk.eagle:library:210" package="SMA-DO214AC" package3d_urn="urn:adsk.eagle:package:43452/2" value="GF1" x="-124.46" y="-322.58"/>
+<element name="R38" library="adafruit" package="R0805" value="10k" x="-124.46" y="-330.2"/>
+<element name="Q1" library="transistor-power" library_urn="urn:adsk.eagle:library:400" package="MICRO3" package3d_urn="urn:adsk.eagle:package:29512/2" value="IRLML5203" x="-124.46" y="-337.82"/>
 </elements>
 <signals>
@@
 <contactref element="R8" pad="2"/>
 <contactref element="C9" pad="1"/>
+<contactref element="Q1" pad="1"/>
 <wire x1="-110.65" y1="-156" x2="-110.5" y2="-144" width="0" layer="19" extent="1-1"/>
 <wire x1="-110.65" y1="-126" x2="-110.5" y2="-144" width="0" layer="19" extent="1-1"/>
@@
 <wire x1="-17.015" y1="-83.82" x2="-48.68" y2="-43.18" width="0" layer="19" extent="1-1"/>
 <wire x1="-20.825" y1="-100.33" x2="-17.015" y2="-83.82" width="0" layer="19" extent="1-1"/>
+<wire x1="-125.41" y1="-338.82" x2="-110.65" y2="-225.5" width="0" layer="19" extent="1-1"/>
 </signal>
 <signal name="CB_14">
@@
 <wire x1="-117.72" y1="-229.36" x2="-118.92" y2="-229.36" width="0" layer="19" extent="1-1"/>
 </signal>
-<signal name="DSG_MOSFET">
+<signal name="N$19">
+<contactref element="D2" pad="A"/>
+<contactref element="R38" pad="2"/>
+<contactref element="Q1" pad="3"/>
+<wire x1="-123.46" y1="-330.2" x2="-124.46" y2="-336.82" width="0" layer="19" extent="1-1"/>
+<wire x1="-126.51" y1="-322.58" x2="-123.46" y2="-330.2" width="0" layer="19" extent="1-1"/>
+</signal>
+<signal name="CHG_GATE">
+<contactref element="Q1" pad="2"/>
+<contactref element="T1" pad="1"/>
+<wire x1="-126.12" y1="-229.36" x2="-123.51" y2="-338.82" width="0" layer="19" extent="1-1"/>
+</signal>
+<signal name="DSG_GATE">
+<contactref element="T2" pad="1"/>
 <contactref element="T4" pad="1"/>
-<contactref element="T2" pad="1"/>
 <contactref element="R29" pad="2"/>
 <wire x1="-126.12" y1="-290.32" x2="-123.46" y2="-299.72" width="0" layer="19" extent="1-1"/>
 <wire x1="-126.12" y1="-249.68" x2="-126.12" y2="-290.32" width="0" layer="19" extent="1-1"/>
 </signal>
-<signal name="CHG_MOSFET">
-<contactref element="T1" pad="1"/>
+<signal name="N$23">
+<contactref element="D2" pad="K"/>
+<contactref element="R38" pad="1"/>
 <contactref element="T3" pad="1"/>
+<contactref element="D1" pad="C"/>
 <contactref element="R30" pad="2"/>
-<contactref element="D1" pad="C"/>
-<contactref element="D2" pad="K"/>
+<wire x1="-122.41" y1="-322.58" x2="-125.46" y2="-330.2" width="0" layer="19" extent="1-1"/>
 <wire x1="-126.16" y1="-314.96" x2="-122.41" y2="-322.58" width="0" layer="19" extent="1-1"/>
 <wire x1="-123.46" y1="-307.34" x2="-126.16" y2="-314.96" width="0" layer="19" extent="1-1"/>
 <wire x1="-126.12" y1="-270" x2="-123.46" y2="-307.34" width="0" layer="19" extent="1-1"/>
-<wire x1="-126.12" y1="-229.36" x2="-126.12" y2="-270" width="0" layer="19" extent="1-1"/>
 </signal>
 </signals>
