File: BMS_hw/BMSV1.0.brd (EAGLE design)
At the start: 272 x 60 mm, 191 parts, among them IC1 MC33771BEP, IC2 SFH6156, IC3 MIC28515V1, J2 NTC, Q1 IRLML5203, T1 IPT020N10N3V1, T2 IPT020N10N3V1, T3 IPT020N10N3V1, T4 IPT020N10N3V1, X2 87758-1816

Commit message: Invalid polygon in gf board
Parts:
- added IC4, IC5, IC6: FOD8384-COC, GreenFuel:SOP5
- added Q2: IRLML5203, transistor-power:MICRO3
- added R40, R41, R42, R8: 10k, ipc-7351-resistor:RESC1005X40AN
- added X1, X4: 87758-2016, con-molex:87758-2016
- C1, C10, C100, C101, C102, C103, C104, C105, C106, C107, C108, C11, C12, C13, C14, C15, C16, C17, C18, C19, C2, C20, C21, C22, C23, C24, C25, C26, C27, C28, C29, C3, C31, C32, C33, C34, C35, C36, C37, C4, C5, C6, C66, C67, C7, C71, C72, C73, C74, C75, C76, C77, C78, C79, C8, C80, C81, C82, C83, C84, C85, C86, C87, C88, C89, C9, C90, C91, C92, C93, C94, C95, C96, C97, C98, C99: device adafruit:C0805 -> ipc-7351-capacitor:CAPC1005X60N
- R1, R10, R100, R101, R102, R103, R104, R105, R11, R12, R13, R14, R15, R16, R17, R18, R19, R2, R20, R21, R22, R23, R24, R25, R26, R27, R28, R29, R3, R30, R31, R32, R33, R34, R35, R36, R37, R38, R4, R46, R5, R6, R64, R66, R67, R70, R71, R72, R73, R74, R75, R76, R77, R78, R79, R80, R81, R82, R83, R84, R85, R86, R87, R88, R89, R9, R90, R91, R99: device adafruit:R0805 -> ipc-7351-resistor:RESC1005X40AN
- moved T2 527.6 mm to (228.0, 40.6)
- moved T4 521.4 mm to (202.6, 21.6)
- moved T3 518.6 mm to (202.6, 40.6)
- moved T1 506.1 mm to (228.6, 22.2)
- moved IC3 264.2 mm to (107.4, 34.0)
- moved J2 245.1 mm to (144.8, 43.8)
- moved R92 161.2 mm to (31.8, 46.4)
- moved R64 91.3 mm to (67.3, 40.0), turned to 270 degrees
- moved R66 85.3 mm to (46.1, 31.6)
- moved X2 83.9 mm to (5.71, 32.4), turned to 90 degrees
- moved R67 74.7 mm to (33.9, 40.6), turned to 90 degrees
- moved R9 68.3 mm to (27.3, 34.9)
- moved R6 65.7 mm to (27.3, 33.7)
- moved R26 60.4 mm to (-33.7, 44.5)
- moved IC1 3.69 mm to (37.1, 32.4), flipped to the top
Connections:
- removed net N$29: T1.9, T2.9, T3.9, T4.9
- new net 15V_AUX: IC4.6, IC5.6, IC6.6, X1.17, X4.17
- new net CHG_FET: IC4.1
- new net C_FET: X1.9, X4.9
- new net DSG_FET: IC6.1
- new net D_FET: X1.19, X4.19
- new net FAULT: X1.5, X4.5
- new net ISP: X1.11, X4.11
- new net N$20: IC4.3, R8.1
- new net N$25: IC6.3, R40.1
- new net N$27: IC5.3, R41.1
- new net N$28: Q2.3, R42.2
- new net N$38: IC5.5
- new net PCHG_FET: IC5.1, Q2.1, X1.4, X4.4
- new net PWR_DRAIN: Q2.2, T1.9, T2.9, T3.9, T4.9
- new net VBATT-: R42.1
- new net VDD: X1.12, X1.13, X4.12, X4.13
- net CHG_GATE: now also IC6.5
- net DSG_GATE: now also IC4.5
- net GND: now also IC4.4, IC5.4, IC6.4, R40.2, R41.2, R8.2, X1.1, X1.10, X1.14, X1.15, X1.16, X1.18, X1.2, X1.20, X1.3, X1.6, X1.7, X1.8, X4.1, X4.10, X4.14, X4.15, X4.16, X4.18, X4.2, X4.20, X4.3, X4.6, X4.7, X4.8

Commit message: board finnnnalo
Parts:
- moved R42 601.2 mm to (191.1, 23.5)
- moved X4 597.3 mm to (168.3, 39.4)
- moved Q2 594.5 mm to (193.7, 22.2)
- moved X1 590.6 mm to (168.3, 23.4)
- moved R39 586.9 mm to (255.3, 28.6), turned to 90 degrees
- moved R40 571.0 mm to (185.0, 9.02), turned to 180 degrees
- moved IC5 563.1 mm to (191.8, 39.4), turned to 180 degrees
- moved R7 559.5 mm to (244.5, 28.6), turned to 90 degrees
- moved IC4 549.2 mm to (182.2, 38.1)
- moved IC6 548.4 mm to (184.2, 17.1)
- moved R41 539.7 mm to (112.4, 21.6)
- moved R8 534.0 mm to (112.1, 24.9)
- moved R38 508.5 mm to (245.7, 18.4), turned to 90 degrees
- moved Q1 502.8 mm to (217.2, 31.1)
- moved D2 501.5 mm to (243.2, 18.4), turned to 270 degrees
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Connections:
- removed net N$39: C78.1, R70.2
- net CT_7: now also C78.1, R70.2
Routing:
- net GND: track 0.00 -> 567.1 mm, vias 0 -> 52
- net CELL14+: track 0.00 -> 264.7 mm, vias 0 -> 2
- net CB_13/12_C: track 0.00 -> 241.5 mm, vias 0 -> 6
- net CB_14/13_C: track 0.00 -> 241.3 mm, vias 0 -> 7
- net CB_13/12_C1: track 0.00 -> 201.4 mm, vias 0 -> 2
- net V-: track 0.00 -> 188.3 mm, vias 0 -> 2
- net CB_12/11_C: track 0.00 -> 184.0 mm, vias 0 -> 6
- net CB_10/9_C: track 0.00 -> 176.9 mm, vias 0 -> 7
- net CB_8/7_C: track 0.00 -> 175.3 mm, vias 0 -> 5
- net CB_13/12_C2: track 0.00 -> 172.9 mm, vias 0 -> 2
- net N$55: track 0.00 -> 140.0 mm, vias 0 -> 4
- net VPWR: track 0.00 -> 135.1 mm, vias 0 -> 2
- net CHG_GATE: track 0.00 -> 130.8 mm
- net CB_13/12_C6: track 0.00 -> 129.5 mm, vias 0 -> 2
- net CB_6/5_C: track 0.00 -> 126.7 mm, vias 0 -> 4
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
Commit message: layout airwire reduced
Routing:
- net GND: track 567.1 -> 623.7 mm, vias 52 -> 63
- net GPIO6: track 59.6 -> 61.9 mm

Commit message: via added
Routing:
- net GND: vias 63 -> 71
Changed lines of the file:
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@@
 <wire x1="90.424" y1="30.0736" x2="90.424" y2="30.226" width="0.1524" layer="1"/>
 <wire x1="89.6112" y1="30.0736" x2="89.535" y2="30.041" width="0.1524" layer="1"/>
+<via x="106.045" y="35.56" extent="1-16" drill="0.35"/>
+<via x="109.22" y="35.56" extent="1-16" drill="0.35"/>
+<via x="50.8" y="33.655" extent="1-16" drill="0.35"/>
+<via x="50.8" y="29.845" extent="1-16" drill="0.35"/>
+<via x="54.61" y="29.845" extent="1-16" drill="0.35"/>
+<via x="53.34" y="33.655" extent="1-16" drill="0.35"/>
+<via x="52.705" y="29.845" extent="1-16" drill="0.35"/>
+<via x="52.07" y="33.02" extent="1-16" drill="0.35"/>
 <wire x1="94.557" y1="39.936" x2="95.065" y2="39.37" width="0" layer="19" extent="1-16"/>
 <wire x1="62.415" y1="44.45" x2="62.865" y2="44.45" width="0" layer="19" extent="1-16"/>
-<wire x1="108.83666875" y1="33.80973125" x2="107.4928" y2="35.1536" width="0" layer="19" extent="1-16"/>
 <wire x1="85.725" y1="27.305" x2="85.344" y2="28.0416" width="0" layer="19" extent="1-16"/>
 <wire x1="96.705" y1="33.02" x2="96.774" y2="31.75" width="0" layer="19" extent="1-1"/>

Commit message: all clearnance done !
Parts:
- moved X4 0.30 mm to (168.6, 39.4)
- moved C105 0.25 mm to (92.1, 28.8)
- moved C4 0.13 mm to (32.3, 19.7)
- moved C83 0.13 mm to (55.1, 22.2)
- moved R10 0.13 mm to (33.8, 19.9)
Routing:
- net CB_14: track 102.4 -> 79.7 mm
- net VDD: track 20.6 -> 2.83 mm
- net CB_4: track 73.0 -> 59.4 mm, vias 4 -> 3
- net GPIO2: track 43.7 -> 32.7 mm, vias 4 -> 3
- net VPWR: track 135.1 -> 124.3 mm
- net CT_1: track 107.7 -> 99.7 mm
- net N$55: track 140.0 -> 132.4 mm
- net CB_3: track 64.5 -> 58.2 mm
- net CB_2: track 87.8 -> 82.9 mm
- net VCOM: track 56.7 -> 55.3 mm
- net BST: track 67.6 -> 66.2 mm
- net N$49: track 85.6 -> 84.5 mm
- net N$21: track 35.4 -> 34.5 mm
- net CHG_GATE: track 130.8 -> 131.5 mm
- net N$51: track 89.7 -> 88.9 mm
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
Commit message: brd sch and lbr of vqfn-32 updated, error resolved !
Parts:
- moved X4 191.1 mm to (60.3, -118.1)
- moved R16 190.9 mm to (35.8, -127.8)
- moved R5 190.9 mm to (-33.0, -134.0)
- moved C100 190.9 mm to (-22.9, -128.9)
- moved C101 190.9 mm to (-17.9, -132.8)
- moved C102 190.9 mm to (-34.3, -118.7)
- moved C103 190.9 mm to (-22.2, -120.0)
- moved C105 190.9 mm to (-15.9, -128.7)
- moved C106 190.9 mm to (-10.8, -124.5)
- moved C107 190.9 mm to (-27.9, -120.0)
- moved C108 190.9 mm to (-21.0, -131.4)
- moved C11 190.9 mm to (-73.0, -128.3)
- moved C12 190.9 mm to (-74.0, -134.0)
- moved C13 190.9 mm to (-3.81, -132.7)
- moved C14 190.9 mm to (-1.92, -117.8)
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Routing:
- net GND: track 623.3 -> 0.00 mm, vias 71 -> 0
- net CELL14+: track 264.8 -> 0.00 mm, vias 2 -> 0
- net CB_13/12_C: track 241.5 -> 0.00 mm, vias 6 -> 0
- net CB_14/13_C: track 241.3 -> 0.15 mm, vias 7 -> 0
- net CB_13/12_C1: track 201.4 -> 0.19 mm, vias 2 -> 0
- net V-: track 188.1 -> 0.00 mm, vias 2 -> 0
- net CB_12/11_C: track 184.0 -> 0.00 mm, vias 6 -> 0
- net CB_10/9_C: track 177.4 -> 0.15 mm, vias 7 -> 0
- net CB_8/7_C: track 175.3 -> 0.00 mm, vias 5 -> 0
- net CB_13/12_C2: track 173.3 -> 0.00 mm, vias 2 -> 0
- net N$55: track 132.4 -> 0.00 mm, vias 4 -> 0
- net CHG_GATE: track 131.5 -> 0.00 mm
- net CB_13/12_C6: track 129.5 -> 0.19 mm, vias 2 -> 0
- net CB_6/5_C: track 126.8 -> 0.00 mm, vias 4 -> 0
- net VPWR: track 124.3 -> 0.00 mm, vias 2 -> 0
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
Commit message: sch brd lib placment comptd!
Parts:
- added D3, D4, D5: SFH48225, GreenFuel:SFH482
- added JP1: (no value), GreenFuel:OLED-CON
- added LED1: L-59EGW-CAGR, GreenFuel:L-59EGW-CA
- added R43, R44, R45, R47, R48, R49, R50, R51, R52, R53, R54, R55, R56, R57, R58: (no value), ipc-7351-resistor:RESC1005X40AN
- added R59, R60, R61, R62: 10k, ipc-7351-resistor:RESC1005X40AN
- L1: value (none) -> XAL1010-822MEB; device inductor-neosid:MS85 -> GreenFuel:DUALPAD
- R39, R7: value LRMAP3920 -> LRMAP3920SUNT
- moved C10 323.5 mm to (223.5, 5.08), turned to 180 degrees
- moved R17 323.2 mm to (226.1, 5.08)
- moved R10 282.3 mm to (144.8, 40.6), turned to 90 degrees
- moved R2 279.6 mm to (144.8, 35.6)
- moved R75 279.6 mm to (142.2, 40.6), turned to 90 degrees
- moved R81 278.3 mm to (127.0, 43.2), turned to 270 degrees
- moved C75 276.9 mm to (132.1, 43.2), turned to 90 degrees
- moved R87 276.1 mm to (121.9, 43.2), turned to 270 degrees
- moved C37 274.5 mm to (139.7, 40.6), turned to 90 degrees
- moved C20 274.3 mm to (142.2, 38.1)
- moved C12 273.7 mm to (144.8, 30.5), turned to 0 degrees
- moved R19 273.5 mm to (144.8, 33.0)
- moved R82 273.3 mm to (124.5, 43.2)
- moved C19 272.6 mm to (147.3, 35.6), turned to 0 degrees
- moved R28 272.0 mm to (142.2, 35.6), turned to 90 degrees
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Connections:
- new net 3.3V: JP1.3, R59.2, X1.16
- new net N$29: CELL14+.P$1, R43.1
- new net N$33: CELL6+.P$1, R49.1
- new net N$35: CELL5+.P$1, R50.1
- new net N$37: CELL12+.P$1, R44.1
- new net N$39: CELL10+.P$1, R45.1
- new net N$40: CELL8+.P$1, R47.1
- new net N$43: CELL7+.P$1, R48.1
- new net N$58: CELL4+.P$1, R51.1
- new net N$59: CELL3+.P$1, R54.1
- new net N$60: CELL2+.P$1, R52.1
- new net N$62: CELL1+.P$1, R55.1
- new net N$63: CELL1-.P$1, R53.1
- new net N$64: CELL11+.P$1, R56.1
- new net N$65: CELL13+.P$1, R57.1
- new net N$66: CELL9+.P$1, R58.2
- new net N$68: C9.1, R39.5, R7.5
- new net N$70: C5.1, D15.C, R3.1, R39.2, R7.2
- new net N$71: LED1.1, R59.1
- new net N$72: D4.K, R62.1
- new net N$73: D5.K, R60.1
- new net N$74: D3.K, R61.1
- new net OLED_SCL: JP1.2, X1.6
- new net OLED_SDA: JP1.1, X1.4
- new net RDTX_OUT+: IC1.48, X1.5
- new net RDTX_OUT-: IC1.45, X1.9
- new net S-LED_1: LED1.3, X1.11
- new net S-LED_2: LED1.2, X1.13
- new net S-LED_3: D3.A, X1.15
- new net S-LED_4: D5.A, X1.17
- new net S-LED_5: D4.A, X1.19
- net 15V_AUX: no longer X1.17
- net CB_10/9_C: now also R58.1; no longer CELL9+.P$1
- net CB_12/11_C: now also R56.2; no longer CELL11+.P$1
- net CB_13/12_C: now also R44.2; no longer CELL12+.P$1
- net CB_13/12_C1: now also R45.2; no longer CELL10+.P$1
- net CB_13/12_C2: now also R47.2; no longer CELL8+.P$1
- net CB_13/12_C6: now also R49.2; no longer CELL6+.P$1
- net CB_13/12_C7: now also R51.2; no longer CELL4+.P$1
- net CB_13/12_C8: now also R52.2; no longer CELL2+.P$1
- net CB_14/13_C: now also R57.2; no longer CELL13+.P$1
- net CB_2/1_C: now also R55.2; no longer CELL1+.P$1
- net CB_4/3_C: now also R54.2; no longer CELL3+.P$1
- net CB_6/5_C: now also R50.2; no longer CELL5+.P$1
- net CB_8/7_C: now also R48.2; no longer CELL7+.P$1
- net CELL1-: now also R53.2; no longer CELL1-.P$1
- net CELL14+: now also R43.2; no longer CELL14+.P$1
- net C_FET: no longer X1.9
- net D_FET: no longer X1.19
- net FAULT: no longer X1.5
- net GND: now also JP1.4, R39.4, R39.6, R60.2, R61.2, R62.2, R7.4, R7.6; no longer C9.1, IC1.45, IC1.48, R39.P$2, R7.P$2, X1.15, X1.16, X1.6
- net ISP: no longer X1.11
- net PCHG_FET: no longer X1.4
- net V-: now also R39.1, R39.3, R7.1, R7.3; no longer C5.1, D15.C, R3.1, R39.P$1, R7.P$1
- net VDD: no longer X1.13
Routing:
- net GND: track 0.00 -> 4.07 mm, vias 0 -> 8

Commit message: brd lbr sch updated to new version
Parts:
- D10, D11, D12, D13, D14, D15, D16, D17, D18: device diode:SOD80C -> ipc-7351-diode:SOD3718X135N
- R92, R93, R94, R95, R96, R97, R98: device adafruit:R0805 -> ipc-7351-resistor:RESC1005X40AN
- moved C1 166.2 mm to (262.9, 97.2), turned to 270 degrees
- moved C7 162.6 mm to (276.2, 97.8), turned to 0 degrees
- moved R13 160.1 mm to (276.2, 99.7), turned to 180 degrees
- moved C90 157.0 mm to (25.4, -80.0), turned to 0 degrees
- moved R6 156.4 mm to (273.1, 100.3)
- moved R4 156.2 mm to (275.0, 104.1)
- moved C11 154.0 mm to (280.7, 97.8)
- moved C28 153.0 mm to (269.9, 102.2)
- moved R32 152.6 mm to (266.7, 106.0), turned to 0 degrees
- moved R27 152.2 mm to (273.1, 102.2)
- moved R14 151.7 mm to (273.1, 105.4)
- moved C12 151.7 mm to (278.1, 102.9)
- moved R18 151.7 mm to (278.1, 100.3)
- moved R19 151.7 mm to (278.1, 105.4)
- moved R2 151.7 mm to (278.1, 108.0)
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Connections:
- removed net N$15: D17.C, R5.1
- net GND: now also D16.K, D18.K; no longer D16.C, D18.C
- net N$68: now also D17.K, R5.1
- net N$70: now also D15.K; no longer D15.C
- net VPWR: now also D10.K, D11.K, D12.K, D13.K, D14.K; no longer D10.C, D11.C, D12.C, D13.C, D14.C
