File: BMS_hw/BMS_MCUV1.0.brd (EAGLE design)
At the start: 60 x 30 mm, 48 parts, among them IC2 SST25VF020B804ISA, J1 22-27-2051-05, J2 22-27-2051-05, J3 22-27-2041-04, J4 22-27-2051-05, Q2 32.768kHz, U1 NCP1117LP-PG, X1 87758-2016

Commit message: DRC setup
Parts:
- moved C9 1.27 mm to (16.4, 27.9)
- moved C10 0.64 mm to (21.0, 27.9)
Routing:
- net CANH: track 132.3 -> 133.5 mm
Changed lines of the file:
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@@
 <grid distance="25" unitdist="mil" unit="mil" style="dots" multiple="1" display="yes" altdistance="5" altunitdist="mil" altunit="mil"/>
 <layers>
-<layer number="1" name="Top" color="4" fill="1" visible="no" active="yes"/>
+<layer number="1" name="Top" color="4" fill="1" visible="yes" active="yes"/>
 <layer number="2" name="Route2" color="16" fill="1" visible="yes" active="yes"/>
 <layer number="3" name="Route3" color="17" fill="1" visible="no" active="no"/>
@@
 <layer number="13" name="Route13" color="21" fill="1" visible="no" active="no"/>
 <layer number="14" name="Route14" color="22" fill="1" visible="no" active="no"/>
-<layer number="15" name="Route15" color="23" fill="1" visible="no" active="yes"/>
-<layer number="16" name="Bottom" color="1" fill="1" visible="no" active="yes"/>
-<layer number="17" name="Pads" color="2" fill="1" visible="no" active="yes"/>
+<layer number="15" name="Route15" color="23" fill="1" visible="yes" active="yes"/>
+<layer number="16" name="Bottom" color="1" fill="1" visible="yes" active="yes"/>
+<layer number="17" name="Pads" color="2" fill="1" visible="yes" active="yes"/>
 <layer number="18" name="Vias" color="2" fill="1" visible="yes" active="yes"/>
 <layer number="19" name="Unrouted" color="6" fill="1" visible="yes" active="yes"/>
-<layer number="20" name="Dimension" color="24" fill="1" visible="no" active="yes"/>
-<layer number="21" name="tPlace" color="7" fill="1" visible="no" active="yes"/>
-<layer number="22" name="bPlace" color="7" fill="1" visible="no" active="yes"/>
-<layer number="23" name="tOrigins" color="15" fill="1" visible="no" active="yes"/>
-<layer number="24" name="bOrigins" color="15" fill="1" visible="no" active="yes"/>
-<layer number="25" name="tNames" color="7" fill="1" visible="no" active="yes"/>
-<layer number="26" name="bNames" color="7" fill="1" visible="no" active="yes"/>
+<layer number="20" name="Dimension" color="24" fill="1" visible="yes" active="yes"/>
+<layer number="21" name="tPlace" color="7" fill="1" visible="yes" active="yes"/>
+<layer number="22" name="bPlace" color="7" fill="1" visible="yes" active="yes"/>
+<layer number="23" name="tOrigins" color="15" fill="1" visible="yes" active="yes"/>
+<layer number="24" name="bOrigins" color="15" fill="1" visible="yes" active="yes"/>
+<layer number="25" name="tNames" color="7" fill="1" visible="yes" active="yes"/>
+<layer number="26" name="bNames" color="7" fill="1" visible="yes" active="yes"/>
 <layer number="27" name="tValues" color="7" fill="1" visible="no" active="yes"/>
 <layer number="28" name="bValues" color="7" fill="1" visible="no" active="yes"/>
@@
 <layer number="37" name="tTest" color="7" fill="1" visible="no" active="yes"/>
 <layer number="38" name="bTest" color="7" fill="1" visible="no" active="yes"/>
-<layer number="39" name="tKeepout" color="4" fill="11" visible="no" active="yes"/>
-<layer number="40" name="bKeepout" color="1" fill="11" visible="no" active="yes"/>
-<layer number="41" name="tRestrict" color="4" fill="10" visible="no" active="yes"/>
-<layer number="42" name="bRestrict" color="1" fill="10" visible="no" active="yes"/>
+<layer number="39" name="tKeepout" color="4" fill="11" visible="yes" active="yes"/>
+<layer number="40" name="bKeepout" color="1" fill="11" visible="yes" active="yes"/>
+<layer number="41" name="tRestrict" color="4" fill="10" visible="yes" active="yes"/>
+<layer number="42" name="bRestrict" color="1" fill="10" visible="yes" active="yes"/>
 <layer number="43" name="vRestrict" color="2" fill="10" visible="no" active="yes"/>
 <layer number="44" name="Drills" color="7" fill="1" visible="no" active="yes"/>
@@
 <layer number="49" name="Reference" color="7" fill="1" visible="no" active="yes"/>
 <layer number="50" name="dxf" color="7" fill="1" visible="no" active="no"/>
-<layer number="51" name="tDocu" color="7" fill="1" visible="no" active="yes"/>
-<layer number="52" name="bDocu" color="7" fill="1" visible="no" active="yes"/>
+<layer number="51" name="tDocu" color="7" fill="1" visible="yes" active="yes"/>
+<layer number="52" name="bDocu" color="7" fill="1" visible="yes" active="yes"/>
 <layer number="53" name="tGND_GNDA" color="7" fill="9" visible="no" active="no"/>
 <layer number="54" name="bGND_GNDA" color="1" fill="9" visible="no" active="no"/>
@@
 <param name="mtCopper" value="0.035mm 0.035mm 0.035mm 0.035mm 0.035mm 0.035mm 0.035mm 0.035mm 0.035mm 0.035mm 0.035mm 0.035mm 0.035mm 0.035mm 0.035mm 0.035mm"/>
 <param name="mtIsolate" value="0.09238125mm 1.2304mm 0.2mm 0.15mm 0.2mm 0.15mm 0.2mm 0.15mm 0.2mm 0.15mm 0.2mm 0.15mm 0.2mm 0.15mm 0.09238125mm"/>
-<param name="mdWireWire" value="6mil"/>
-<param name="mdWirePad" value="6mil"/>
+<param name="mdWireWire" value="10mil"/>
+<param name="mdWirePad" value="8mil"/>
 <param name="mdWireVia" value="6mil"/>
 <param name="mdPadPad" value="6mil"/>
 <param name="mdPadVia" value="6mil"/>
-<param name="mdViaVia" value="6mil"/>
-<param name="mdSmdPad" value="6mil"/>
-<param name="mdSmdVia" value="6mil"/>
-<param name="mdSmdSmd" value="6mil"/>
+<param name="mdViaVia" value="10mil"/>
+<param name="mdSmdPad" value="0mil"/>
+<param name="mdSmdVia" value="0mil"/>
+<param name="mdSmdSmd" value="0mil"/>
 <param name="mdViaViaSameLayer" value="6mil"/>
 <param name="mnLayersViaInSmd" value="2"/>
-<param name="mdCopperDimension" value="40mil"/>
-<param name="mdDrill" value="6mil"/>
+<param name="mdCopperDimension" value="10mil"/>
+<param name="mdDrill" value="10mil"/>
 <param name="mdSmdStop" value="0mil"/>
 <param name="msWidth" value="6mil"/>
-<param name="msDrill" value="0.35mm"/>
-<param name="msMicroVia" value="9.99mm"/>
+<param name="msDrill" value="12mil"/>
+<param name="msMicroVia" value="12mil"/>
 <param name="msBlindViaRatio" value="0.5"/>
 <param name="rvPadTop" value="0.25"/>
@@
 <param name="rlMinPadBottom" value="10mil"/>
 <param name="rlMaxPadBottom" value="20mil"/>
-<param name="rlMinViaOuter" value="8mil"/>
+<param name="rlMinViaOuter" value="6mil"/>
 <param name="rlMaxViaOuter" value="20mil"/>
-<param name="rlMinViaInner" value="8mil"/>
+<param name="rlMinViaInner" value="6mil"/>
 <param name="rlMaxViaInner" value="20mil"/>
 <param name="rlMinMicroViaOuter" value="4mil"/>
@@
 <param name="mvStopFrame" value="1"/>
 <param name="mvCreamFrame" value="0"/>
-<param name="mlMinStopFrame" value="4mil"/>
-<param name="mlMaxStopFrame" value="4mil"/>
+<param name="mlMinStopFrame" value="2mil"/>
+<param name="mlMaxStopFrame" value="2mil"/>
 <param name="mlMinCreamFrame" value="0mil"/>
 <param name="mlMaxCreamFrame" value="0mil"/>
-<param name="mlViaStopLimit" value="0mil"/>
+<param name="mlViaStopLimit" value="100mil"/>
 <param name="srRoundness" value="0"/>
 <param name="srMinRoundness" value="0mil"/>
@@
 <elements>
 <element name="C1" library="adafruit" package="C0805" value="20pF" x="10.795" y="13.335"/>
-<element name="C10" library="adafruit" package="C0805" value="47pF" x="21.6662" y="27.94"/>
+<element name="C10" library="adafruit" package="C0805" value="47pF" x="21.0312" y="27.94"/>
 <element name="C11" library="adafruit" package="C0805" value="4.7uF" x="14.605" y="15.24"/>
 <element name="C12" library="adafruit" package="C0805" value="10uF" x="25.4" y="27.94"/>
@@
 <element name="C7" library="adafruit" package="C0805" value="" x="6.985" y="20.32" rot="R90"/>
 <element name="C8" library="adafruit" package="C0805" value="10uF" x="17.7038" y="25.4"/>
-<element name="C9" library="adafruit" package="C0805" value="47pF" x="17.653" y="27.94"/>
+<element name="C9" library="adafruit" package="C0805" value="47pF" x="16.383" y="27.94"/>
 <element name="IC2" library="GreenFuel" package="SOIC127P600X175-8N" value="SST25VF020B804ISA" x="5.715" y="15.24" rot="R90"/>
 <element name="J1" library="con-molex" library_urn="urn:adsk.eagle:library:165" package="6410-05" value="22-27-2051-05" x="23.495" y="4.445">
@@
 <wire x1="25.146" y1="26.543" x2="26.25" y2="25.439" width="0.1524" layer="1"/>
 <wire x1="26.25" y1="25.439" x2="26.25" y2="25.4" width="0.1524" layer="1"/>
+<wire x1="17.233" y1="27.94" x2="19.685" y2="28.575" width="0" layer="19" extent="1-1"/>
 </signal>
 <signal name="N$1">
@@
 <wire x1="6.858" y1="27.178" x2="13.208" y2="27.178" width="0.1524" layer="1"/>
 <wire x1="5.08" y1="25.4" x2="6.858" y2="27.178" width="0.1524" layer="1"/>
-<wire x1="20.574" y1="27.94" x2="20.8162" y2="27.94" width="0.1524" layer="1"/>
+<wire x1="20.1812" y1="27.94" x2="20.1812" y2="27.5472" width="0.1524" layer="1"/>
 <wire x1="3.048" y1="10.922" x2="3.048" y2="9.652" width="0.1524" layer="1"/>
 <wire x1="3.048" y1="23.368" x2="3.048" y2="10.922" width="0.1524" layer="16"/>
@@
 <via x="53.086" y="20.066" extent="1-16" drill="0.1524"/>
 <wire x1="13.462" y1="26.924" x2="19.558" y2="26.924" width="0.1524" layer="1"/>
-<wire x1="19.558" y1="26.924" x2="20.574" y2="27.94" width="0.1524" layer="1"/>
+<wire x1="19.558" y1="26.924" x2="20.1812" y2="27.5472" width="0.1524" layer="1"/>
 </signal>
 <signal name="N$11">
@@
 <wire x1="5.842" y1="23.622" x2="4.572" y2="23.622" width="0.1524" layer="1"/>
 <wire x1="7.62" y1="25.4" x2="5.842" y2="23.622" width="0.1524" layer="1"/>
-<wire x1="16.764" y1="27.94" x2="16.803" y2="27.94" width="0.1524" layer="1"/>
+<wire x1="15.533" y1="27.94" x2="16.764" y2="27.94" width="0.1524" layer="1"/>
 <wire x1="4.572" y1="10.414" x2="4.572" y2="9.652" width="0.1524" layer="1"/>
 <wire x1="3.048" y1="11.938" x2="4.572" y2="10.414" width="0.1524" layer="1"/>
@@
 <wire x1="9.906" y1="10.922" x2="9.945" y2="10.795" width="0.1524" layer="1"/>
 <wire x1="13.462" y1="19.05" x2="13.5796" y2="19.431" width="0.1524" layer="1"/>
-<via x="8.636" y="11.684" extent="1-16" drill="0.35"/>
+<via x="8.636" y="11.684" extent="1-16" drill="0.2"/>
 <via x="12.446" y="20.066" extent="1-16" drill="0.1524"/>
 </signal>

Commit message: package udated
Parts:
- C1, C14, C15, C16, C2, C21: device adafruit:C0805 -> ipc-7351-capacitor:CAPC1608X92N
- C10, C13, C7, C9: device adafruit:C0805 -> ipc-7351-capacitor:CAPC2012X145AN
- R10, R11, R12, R13, R14, R3, R4, R5, R6, R7, R8, R9: device adafruit:M0805 -> ipc-7351-resistor:RESC2012X70N
- R15, R16: device adafruit:R0805 -> ipc-7351-resistor:RESC1608X55N
Routing:
- net N$17: track 21.2 -> 0.00 mm, vias 2 -> 0
