File: BMS_hw/AFE_PCB/BMSV1.0.brd (EAGLE design)
At the start: 272 x 60 mm, 239 parts, among them IC1 MC33771BEP, IC2 SFH6156, IC3 MIC28515V1, IC4 FOD8384-COC, IC5 FOD8384-COC, IC6 FOD8384-COC, J2 NTC, Q1 IRLML5203, Q2 IRLML5203, T1 IPT020N10N3V1, T2 IPT020N10N3V1, T3 IPT020N10N3V1, T4 IPT020N10N3V1, X1 87758-2016, X2 87758-1816, X3 22-23-2041, X4 87758-2016, X5 22-23-2051

Commit message: updated dcdc sch
Parts:
- moved R50 0.64 mm to (88.3, 13.3)
Routing:
- net N$35: track 6.79 -> 7.42 mm
Changed lines of the file:
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@@
 <attribute name="VALUE" x="127.115" y="48.179" size="1.27" layer="27" font="vector" ratio="10" rot="R180"/>
 </element>
-<element name="R50" library="ipc-7351-resistor" package="RESC1005X40AN" value="" x="88.265" y="12.7" rot="R180">
-<attribute name="NAME" x="89.015" y="12.146" size="1.27" layer="25" font="vector" ratio="10" rot="R180"/>
-<attribute name="VALUE" x="89.015" y="14.524" size="1.27" layer="27" font="vector" ratio="10" rot="R180"/>
+<element name="R50" library="ipc-7351-resistor" package="RESC1005X40AN" value="" x="88.265" y="13.335" rot="R180">
+<attribute name="NAME" x="89.015" y="12.781" size="1.27" layer="25" font="vector" ratio="10" rot="R180"/>
+<attribute name="VALUE" x="89.015" y="15.159" size="1.27" layer="27" font="vector" ratio="10" rot="R180"/>
 </element>
 <element name="R51" library="ipc-7351-resistor" package="RESC1005X40AN" value="" x="88.265" y="46.355" rot="R180">
@@
 <wire x1="58.48438125" y1="15.8548" x2="58.6252" y2="15.8548" width="0.254" layer="1"/>
 <wire x1="58.6252" y1="15.8548" x2="59.24" y2="15.24" width="0.254" layer="1"/>
-<wire x1="64.23863125" y1="25.475078125" x2="87.815" y2="12.7" width="0" layer="19" extent="1-1"/>
+<wire x1="64.23863125" y1="25.475078125" x2="87.815" y2="13.335" width="0" layer="19" extent="1-1"/>
 <wire x1="57.97" y1="16.51" x2="64.23863125" y2="25.475078125" width="0" layer="19" extent="1-1"/>
 </signal>
@@
 <contactref element="CELL5+" pad="P$1"/>
 <contactref element="R50" pad="1"/>
-<wire x1="88.715" y1="12.7" x2="88.715" y2="6.215" width="0.254" layer="1"/>
+<wire x1="88.715" y1="13.335" x2="88.715" y2="6.215" width="0.254" layer="1"/>
 <wire x1="88.715" y1="6.215" x2="88.5" y2="6" width="0.254" layer="1"/>
 </signal>

Commit message: updated sch
Parts:
- removed R68: 0R, ipc-7351-resistor:RESC1608X55N
- C17: value .1uF 100v -> 47nF; device ipc-7351-capacitor:CAPC1608X92N -> ipc-7351-capacitor:CAPC1005X60N
- C24: value .1u 100v -> 47nF
- C26: value 1uF 100v -> 47nF; device ipc-7351-capacitor:CAPC1608X92N -> ipc-7351-capacitor:CAPC1005X60N
- R12, R15, R22, R23: device ipc-7351-resistor:RESC1608X55N -> ipc-7351-resistor:RESC1005X40AN
- R16, R24: value 1.6k -> 127E; device ipc-7351-resistor:RESC1608X55N -> ipc-7351-resistor:RESC1005X40AN
- R21: value 16.2k -> 127E; device ipc-7351-resistor:RESC1608X55N -> ipc-7351-resistor:RESC1005X40AN
- R25: value 2R -> 127E; device ipc-7351-resistor:RESC1608X55N -> ipc-7351-resistor:RESC1005X40AN
- moved X5 277.8 mm to (266.7, 36.8), turned to 270 degrees
- moved D9 270.9 mm to (268.6, 19.7), turned to 90 degrees
- moved D19 270.3 mm to (268.6, 12.1), turned to 90 degrees
- moved JP3 262.2 mm to (257.2, 14.0)
- moved X3 260.4 mm to (259.7, 8.26)
- moved R30 244.4 mm to (179.7, 94.0)
- moved D1 244.0 mm to (182.2, 94.6)
- moved D2 240.7 mm to (186.7, 94.6), turned to 90 degrees
- moved R38 236.6 mm to (186.7, 90.2), turned to 270 degrees
- moved Q1 230.1 mm to (186.7, 86.4)
- moved IC5 224.2 mm to (88.2, 92.7)
- moved R29 220.1 mm to (156.2, 73.7), turned to 90 degrees
- moved IC6 217.5 mm to (104.1, 76.8), turned to 270 degrees
- moved IC4 209.3 mm to (138.4, 83.2)
- moved R103 188.9 mm to (12.7, 41.3), turned to 90 degrees
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Connections:
- net N$67 renamed V+
- removed net N$10: C24.2, R68.2
- removed net N$23: D1.K, D2.K, R30.2, R38.1, T1.1
- removed net N$61: R29.1, T3.2, T3.3, T3.4, T3.5, T3.6, T3.7, T3.8, T4.2, T4.3, T4.4, T4.5, T4.6, T4.7, T4.8
- net CHG_GATE: now also D1.K, D2.K, R30.2, R38.1, T1.1
- net SW: now also C24.2; no longer R68.1
- net V-: now also R29.1, T3.2, T3.3, T3.4, T3.5, T3.6, T3.7, T3.8, T4.2, T4.3, T4.4, T4.5, T4.6, T4.7, T4.8
Routing:
- net CB_14/13_C: track 2.15 -> 212.7 mm, vias 0 -> 2
- net V+: track 0.00 -> 40.1 mm, vias 0 -> 29
- net V-: track 0.00 -> 36.8 mm, vias 0 -> 41
- net GPIO4: track 0.00 -> 25.5 mm
- net CT_14: track 5.74 -> 28.6 mm, vias 0 -> 2
- net CT_12: track 7.88 -> 25.4 mm
- net CHG_GATE: track 0.00 -> 17.1 mm
- net DSG_GATE: track 0.00 -> 16.3 mm
- net CT_13: track 7.71 -> 23.1 mm
- net N$53: track 5.68 -> 20.4 mm
- net CANL: track 0.00 -> 14.0 mm
- net N$29: track 64.0 -> 75.9 mm, vias 2 -> 4
- net N$55: track 6.84 -> 16.5 mm, vias 0 -> 2
- net GPIO0: track 2.28 -> 9.65 mm, vias 0 -> 1
- net CANH: track 0.00 -> 6.45 mm
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- added copper zone on layer 1, net PWR_DRAIN
- added copper zone on layer 16, net PWR_DRAIN1
- added copper zone on layer 1, net V+
- added copper zone on layer 16, net V+
- added copper zone on layer 1, net V-
- added copper zone on layer 16, net V-

Commit message: board layout itt@1
Parts:
- removed C100, C101, C95, C96, C97, C98, C99: 1uF, ipc-7351-capacitor:CAPC1005X60N
- removed C102, C103, C104, C105, C106, C107, C108: 2.2uF, ipc-7351-capacitor:CAPC1005X60N
- removed C79, C81, C83, C84, C85, C87, C89, C90, C91, C93, C94: 0.047uF, ipc-7351-capacitor:CAPC1005X60N
- removed C80, C82, C86, C88, C92: 0.47uF, ipc-7351-capacitor:CAPC1005X60N
- removed J2: NTC, con-molex:6410-08
- removed R105: 10k, ipc-7351-resistor:RESC1005X40AN
- added C39: 0.47uF, ipc-7351-capacitor:CAPC3215X168N
- added C40, C41, C42, C43, C44, C45, C46, C47: 0.047uF, ipc-7351-capacitor:CAPC1005X60N
- added C48, C49, C50, C51, C52, C53, C54: 2.2uF, ipc-7351-capacitor:CAPC1005X60N
- added C55, C56, C57, C58, C59, C60, C62: 1uF, ipc-7351-capacitor:CAPC1005X60N
- added C61: 0.22uF, ipc-7351-capacitor:CAPC1005X60N
- added C63: (no value), ipc-7351-capacitor:CAPAE830X620N
- added C64, C70: 47nF, ipc-7351-capacitor:CAPC3225X168N
- added C65, C68: 47nF, ipc-7351-capacitor:CAPC1005X60N
- added C69: 47nF, ipc-7351-capacitor:CAPC1608X92N
- added J1: NTC, con-molex:6410-08
- added R68, R69: 10k, ipc-7351-resistor:RESC1005X40AN
- added TP1: TPTH7035, simpa:TP7035
- C1: value 0.22uF -> 0.047uF; device ipc-7351-capacitor:CAPC1005X60N -> ipc-7351-capacitor:CAPC1608X92N
- C10, C11, C12, C32, C33, C34, C35, C36, C37, C8: value 0.047uF -> 0.47uF; device ipc-7351-capacitor:CAPC1005X60N -> ipc-7351-capacitor:CAPC3215X168N
- C13, C9: value 47nF -> 0.47uF; device ipc-7351-capacitor:CAPC1005X60N -> ipc-7351-capacitor:CAPC3215X168N
- C14: value 2.2uF -> 0.47uF; device ipc-7351-capacitor:CAPC1005X60N -> ipc-7351-capacitor:CAPC3215X168N
- C15: value 2.2uF -> 0.047uF
- C16: value 1uF -> 0.047uF
- C17: value 47nF -> 0.047uF
- C18, C19, C20, C21: value 0.47uF -> 0.047uF
- C2, C24, C26, C5: value 47nF -> 0.047uF; device ipc-7351-capacitor:CAPC1005X60N -> ipc-7351-capacitor:CAPC1608X92N
- C22: value 47nF -> 2.2uF; device ipc-7351-capacitor:CAPC1608X92N -> ipc-7351-capacitor:CAPC1005X60N
- C23: value 47nF -> .047uF; device ipc-7351-capacitor:CAPC3225X168N -> ipc-7351-capacitor:CAPC1005X60N
- C25: value 47nF -> 0.047uF; device ipc-7351-capacitor:CAPC3225X168N -> ipc-7351-capacitor:CAPC1608X92N
- C27, C28, C29: value 0.47uF -> 0.047uF; device ipc-7351-capacitor:CAPC1005X60N -> ipc-7351-capacitor:CAPC1608X92N
- C3, C31, C4, C7: device ipc-7351-capacitor:CAPC1005X60N -> ipc-7351-capacitor:CAPC1608X92N
- C30: value (none) -> 0.047uF; device ipc-7351-capacitor:CAPC1005X60N -> ipc-7351-capacitor:CAPC1608X92N
- C38: value (none) -> 0.47uF; device ipc-7351-capacitor:CAPAE830X620N -> ipc-7351-capacitor:CAPC3215X168N
- C6: value 6.8uF -> 0.047uF; device ipc-7351-capacitor:CAPC1005X60N -> ipc-7351-capacitor:CAPC1608X92N
- C66: value .047uF -> 47nF
- C67: value 2.2uF -> 47nF
- C71: value 0.047uF -> 47nF
- C72, C74: value 0.47uF -> 47nF
- C73: value 0.047uF -> 1uF
- C75: value 0.047uF -> 6.8uF
- C76: value 0.47uF -> 2.2uF
- C77: value 0.047uF -> 2.2uF
- C78: value 0.047uF -> (none)
- D10: value 8.2v -> (none)
- D11: value 20v -> 8.2v
- D12: value 27v -> (none)
- D13: value 43v -> (none)
- D14: value 75v -> (none)
- D15, D16: value 2v -> (none)
- D17, D18: value 2v -> SFH48225; device ipc-7351-diode:SOD3718X135N -> GreenFuel:SFH482
- D19: value (none) -> SFH48225; device ipc-7351-diode:SOD3718X135N -> GreenFuel:SFH482
- D2: value (none) -> 20v
- D3: value SFH48225 -> 27v; device GreenFuel:SFH482 -> ipc-7351-diode:SOD3718X135N
- D4: value SFH48225 -> 43v; device GreenFuel:SFH482 -> ipc-7351-diode:SOD3718X135N
- D5: value SFH48225 -> 75v; device GreenFuel:SFH482 -> ipc-7351-diode:SOD3718X135N
- D6, D7, D8, D9: value (none) -> 2v
- JP1: device GreenFuel:OLED-CON -> adafruit:1X01-CLEANBIG
- JP3: device adafruit:1X01-CLEANBIG -> GreenFuel:OLED-CON
- R1: value 10 -> (none)
- R10, R9: value 180E -> (none)
- R11: value 2E2 -> 180E; device ipc-7351-resistor:RESC1005X40AN -> ipc-7351-resistor:RESC3225X70N
- R12: value 200k -> 180E; device ipc-7351-resistor:RESC1005X40AN -> ipc-7351-resistor:RESC3225X70N
- R13: value 180E -> 39E; device ipc-7351-resistor:RESC1005X40AN -> ipc-7351-resistor:RESC3225X70N
- R14, R6: device ipc-7351-resistor:RESC1005X40AN -> ipc-7351-resistor:RESC3225X70N
- R15: value 100k -> 3k
- R16, R21: value 127E -> 3k
- R2, R4: value 100 -> (none)
- R22, R23, R24, R25: value 127E -> 2k
- R26, R27, R28: value 3k -> 2k
- R3: value 127E -> (none)
- R31, R70, R72, R74, R78: value 2k -> 10k
- R32, R33, R36, R37: value 2k -> (none)
- R34: value 2k -> 0R
- R35: value 2k -> 100; device ipc-7351-resistor:RESC1005X40AN -> ipc-7351-resistor:RESC3225X70N
- R38, R41, R42, R8: value 10k -> (none)
- R39, R7: value LRMAP3920SUNT -> 100; device GreenFuel:SMD4 -> ipc-7351-resistor:RESC3225X70N
- R40: value 10k -> 100; device ipc-7351-resistor:RESC1005X40AN -> ipc-7351-resistor:RESC3225X70N
- R44, R45, R50, R51, R52, R53, R54, R55: value (none) -> 3k
- R46: value 3k -> 180E; device ipc-7351-resistor:RESC1005X40AN -> ipc-7351-resistor:RESC3225X70N
- R47, R48, R49: value (none) -> 180E; device ipc-7351-resistor:RESC1005X40AN -> ipc-7351-resistor:RESC3225X70N
- R5: value 127E -> 100; device ipc-7351-resistor:RESC1005X40AN -> ipc-7351-resistor:RESC3225X70N
- R56, R57, R58: value (none) -> 2k
- R59, R60, R61, R62, R63: value 10k -> 2k
- R66: value 10k -> 10
- R71, R73, R77: value 3k -> 10k
- R75: value 100 -> 10k
- R76: value 180E -> 10k
- R79, R83, R85: value 3k -> 127E
- R80, R86: value 2k -> 127E
- R81: value 100 -> LRMAP3920SUNT; device ipc-7351-resistor:RESC1005X40AN -> GreenFuel:SMD4
- R82, R88: value 180E -> 127E
- R84: value 2k -> LRMAP3920SUNT; device ipc-7351-resistor:RESC1005X40AN -> GreenFuel:SMD4
- R87: value 100 -> 127E
- R89: value 180E -> 100k
- R90: value 2k -> 200k
- R91: value 3k -> 2E2
- X1: value 87758-2016 -> 87758-1816; device con-molex:87758-2016 -> con-molex:87758-1816
- X2: value 87758-1816 -> 87758-2016; device con-molex:87758-1816 -> con-molex:87758-2016
- X3: value 22-23-2041 -> 87758-2016; device GreenFuel:22-23-2041 -> con-molex:87758-2016
- X4: value 87758-2016 -> 22-23-2051; device con-molex:87758-2016 -> GreenFuel:22-23-2051
- X5: value 22-23-2051 -> 22-23-2041; device GreenFuel:22-23-2051 -> GreenFuel:22-23-2041
- moved R3 241.0 mm to (259.7, 47.0), turned to 180 degrees
- moved JP2 227.6 mm to (257.2, 14.0)
- moved R21 223.7 mm to (23.5, 30.5), turned to 180 degrees
- moved D15 222.4 mm to (268.6, 12.1), turned to 90 degrees
- moved R1 222.4 mm to (240.0, 47.0), turned to 180 degrees
- moved C14 220.7 mm to (21.0, 33.0), turned to 180 degrees
- moved R43 211.1 mm to (51.4, 13.1), turned to 0 degrees
- moved R12 208.3 mm to (27.9, 21.6), turned to 0 degrees
- moved C3 208.0 mm to (256.5, 47.0)
- moved R57 207.1 mm to (34.3, 29.8), turned to 270 degrees
- moved X1 206.8 mm to (7.62, 31.8), turned to 90 degrees
- moved D14 206.8 mm to (268.6, 19.7), turned to 90 degrees
- moved R11 206.4 mm to (27.9, 39.4)
- moved C1 205.8 mm to (236.9, 47.0), turned to 180 degrees
- moved X2 205.4 mm to (212.7, 41.9), turned to 0 degrees
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Connections:
- removed net 15V_AUX: IC4.6, IC5.6, IC6.6, X4.17
- removed net C_FET: X4.9
- removed net D_FET: X4.19
- removed net N$26: C66.1, IC1.60
- removed net N$42: C74.1, R71.2, R72.1
- removed net N$44: C80.1, R77.2, R78.1
- removed net N$45: C82.1, R79.2, R80.1
- removed net N$47: C88.1, R85.2, R86.1
- removed net N$63: CELL1-.P$1, R53.1
- removed net VBATT-: R42.1
- removed net VCC: C22.1, C23.1, L1.2, R22.1
- new net +15V: C69.1, C70.1, IC4.6, IC5.6, IC6.6, L1.2, R85.1, X2.17
- new net BGND: CELL1-.P$1, R34.1, R38.1, R81.4, R81.6, R84.4, R84.6
- new net GATE: D10.K, D11.K, R93.1, R94.2, T3.1, T4.1
- new net N$10: C38.1, R54.2, R62.1
- new net N$16: C37.1, R53.2, R60.1
- new net N$23: C36.1, R52.2, R59.1
- new net PCHG_GATE: IC6.1, X2.4
- new net VANA: C23.1, IC1.60
- net !MCLR: now also X2.10, X4.5; no longer X4.10, X5.5
- net 3.3V: now also JP3.3, R101.2, X2.12, X3.16, X4.4; no longer JP1.3, R59.2, X1.16, X4.12, X5.4
- net AGND: now also X1.1; no longer X2.1
- net BST: now also C65.1; no longer C24.1
- net CANH: now also D15.K, X5.4; no longer D19.K, X3.4
- net CANL: now also D14.K, X5.3; no longer D9.K, X3.3
- net CB_1: now also R49.2; no longer R89.2
- net CB_10/9_C: now also C7.1, D2.A, R10.1, R17.1; no longer C12.1, D11.A, R19.1, R58.1
- net CB_11: now also R6.2; no longer R4.2
- net CB_12: now also D4.A, R11.2; no longer D13.A, R9.2
- net CB_12/11_C: now also C6.1, R16.1, R9.2; no longer C11.1, R18.1, R56.2
- net CB_13: now also R7.2; no longer R6.2
- net CB_13/12_C: now also C1.1, R1.2, R11.1, R20.1, R7.1; no longer C3.1, R27.1, R44.2, R6.1, R9.1
- net CB_13/12_C1: now also C4.1, R21.1, R4.2, R6.1; no longer C8.1, R28.1, R4.1, R45.2
- net CB_13/12_C2: now also C2.1, R12.1, R18.1, R2.2, R5.1; no longer C4.1, R10.1, R2.1, R20.1, R47.2
- net CB_13/12_C6: now also C26.1, R36.2, R39.1, R46.1, R51.1; no longer C73.1, R49.2, R71.1, R75.1, R76.1
- net CB_13/12_C7: now also C24.1, R32.2, R35.1, R47.1, R52.1; no longer C79.1, R51.2, R77.1, R81.1, R82.1
- net CB_13/12_C8: now also C28.1, R37.2, R40.1, R48.1, R55.1; no longer C85.1, R52.2, R83.1, R87.1, R88.1
- net CB_14: now also D3.A; no longer D12.A
- net CB_14/13_C: now also C5.1, R15.1, R8.2; no longer C10.1, R17.1, R57.2
- net CB_2: now also R48.2; no longer R88.2
- net CB_2/1_C: now also C31.1, R41.2, R54.1; no longer C87.1, R55.2, R85.1
- net CB_3: now also R40.2; no longer R87.2
- net CB_4: now also R47.2; no longer R82.2
- net CB_4/3_C: now also C30.1, R43.2, R53.1; no longer C81.1, R54.2, R79.1
- net CB_5: now also R35.2; no longer R81.2
- net CB_6: now also R46.2; no longer R76.2
- net CB_6/5_C: now also C25.1, R33.2, R44.1; no longer C75.1, R50.2, R73.1
- net CB_7: now also R39.2; no longer R75.2
- net CB_8: now also R12.2; no longer R10.2
- net CB_8/7_C: now also C29.1, D1.A, R42.2, R50.1; no longer C71.1, D10.A, R46.1, R48.2
- net CB_9: now also R5.2; no longer R2.2
- net CELL1-: now also C27.1, R38.2, R45.1, R49.1, R98.1; no longer C91.1, R53.2, R89.1, R91.1
- net CELL14+: now also C3.1, R19.1, R3.2, R66.1; no longer C7.1, R1.1, R26.1, R43.2
- net CHG_FET: now also IC5.5, Q1.2; no longer IC4.1
- net CHG_GATE: now also IC5.1, X2.9; no longer D1.K, D2.K, IC6.5, Q1.2, R30.2, R38.1, T1.1, T2.1
- net CT_1: now also C45.2, C46.1, R62.2; no longer C89.2, C93.1, R86.2
- net CT_10: now also C18.2, C19.1, R26.2; no longer C34.2, C35.1, R35.2
- net CT_11: now also C17.2, C18.1, R25.2; no longer C33.2, C34.1, R34.2
- net CT_12: now also C16.2, C17.1, R24.2; no longer C32.2, C33.1, R33.2
- net CT_13: now also C15.2, C16.1, R23.2; no longer C31.2, C32.1, R32.2
- net CT_14: now also C15.1, R22.2; no longer C31.1, R31.2
- net CT_2: now also C44.2, C45.1, R61.2; no longer C89.1, C90.2, R84.2
- net CT_3: now also C43.2, C44.1, R60.2; no longer C83.2, C90.1, R80.2
- net CT_4: now also C42.2, C43.1, R59.2; no longer C83.1, C84.2, R78.2
- net CT_5: now also C41.2, C42.1, R58.2; no longer C77.2, C84.1, R74.2
- net CT_6: now also C40.2, C41.1, R57.2; no longer C77.1, C78.2, R72.2
- net CT_7: now also C21.2, C40.1, R56.2; no longer C37.2, C78.1, R70.2
- net CT_8: now also C20.2, C21.1, R28.2; no longer C36.2, C37.1, R37.2
- net CT_9: now also C19.2, C20.1, R27.2; no longer C35.2, C36.1, R36.2
- net CT_REF: now also C46.2, C47.1, R63.2; no longer C93.2, C94.1, R90.2
- net C_HIGH(VC14): now also X1.18; no longer X2.18
- net DSG_FET: now also IC4.5, R92.2, T1.1, T2.1; no longer IC6.1
- net DSG_GATE: now also IC4.1, X2.19; no longer IC4.5, R29.2, T3.1, T4.1
- net FAULT: now also X2.5; no longer X4.5
- net FB: now also C66.2, R85.2, R86.1; no longer C17.2, R22.2, R23.1
- net GND: now also C24.2, C30.2, C31.2, C32.2, C33.2, C34.2, C35.2, C36.2, C37.2, C38.2, C39.2, C47.2, C48.2, C49.2, C50.2, C51.2, C52.2, C53.2, C54.2, C55.2, C56.2, C57.2, C58.2, C59.2, C6.2, C60.2, C61.2, C62.2, C63.-, C64.2, C68.2, C69.2, C70.2, C77.2, C78.1, D15.A, D16.A, D5.A, D7.K, D9.K, J1.1, JP3.4, R100.2, R102.2, R103.2, R104.2, R30.2, R34.2, R86.2, R89.2, R95.2, R96.2, R97.2, X1.11, X2.1, X2.15, X2.18, X2.2, X2.20, X2.3, X2.6, X2.7, X2.8, X3.1, X3.10, X3.14, X3.18, X3.2, X3.20, X3.3, X3.7, X3.8; no longer C100.2, C101.2, C102.2, C103.2, C104.2, C105.2, C106.2, C107.2, C108.2, C15.2, C16.2, C18.2, C19.2, C20.2, C21.2, C30.1, C38.-, C66.2, C75.2, C79.2, C80.2, C81.2, C82.2, C85.2, C86.2, C87.2, C88.2, C91.2, C92.2, C94.2, C95.2, C96.2, C97.2, C98.2, C99.2, D16.K, D18.K, D19.A, D6.A, D9.A, J2.1, JP1.4, R15.2, R23.2, R39.4, R39.6, R40.2, R41.2, R60.2, R61.2, R62.2, R65.2, R67.2, R7.4, R7.6, R8.2, X1.1, X1.10, X1.14, X1.18, X1.2, X1.20, X1.3, X1.7, X1.8, X2.11, X4.15, X4.18, X4.2, X4.20, X4.3, X4.6, X4.7, X4.8, X5.1
- net GPIO0: now also C59.1, R72.1; no longer C95.1, R99.1
- net GPIO1: now also C55.1, R73.1; no longer C96.1, R100.1
- net GPIO2: now also C56.1, R74.1; no longer C97.1, R101.1
- net GPIO3: now also C57.1, R75.1; no longer C98.1, R102.1
- net GPIO4: now also C58.1, R76.1; no longer C99.1, R103.1
- net GPIO5: now also C62.1, R77.1; no longer C100.1, R104.1
- net GPIO6: now also C60.1, R78.1; no longer C101.1, R105.1
- net ILIM: now also R80.1, R82.1; no longer R16.1, R24.1
- net INTL_IN2: now also D12.A, X5.1; no longer D7.A, X3.1
- net INTL_OUT1: now also JP2.1, X5.2; no longer JP3.1, X3.2
- net ISENSE+: now also C71.1, C75.1, R87.2; no longer C13.1, C6.1, R5.2
- net ISENSE-: now also C72.1, C75.2, R88.2; no longer C2.1, C6.2, R3.2
- net ISP: now also X2.11; no longer X4.11
- net KEY-IN: now also D12.K, D13.K, R99.1; no longer D7.K, D8.K, R63.1
- net N$1: now also C12.1, R19.2, R22.1; no longer C27.1, R26.2, R31.1
- net N$11: now also D6.A, D7.A; no longer D17.A, D18.A
- net N$17: now also R89.1, R90.1; no longer R12.1, R15.1
- net N$18: now also C73.1; no longer C16.1
- net N$19: now also D10.A, R93.2; no longer D2.A, R38.2
- net N$2: now also C11.1, R18.2, R28.1; no longer C21.1, R20.2, R37.1
- net N$20: now also IC5.3, R96.1; no longer IC4.3, R8.1
- net N$21: now also C74.1, R79.2; no longer C26.1, R25.2
- net N$24: now also C66.1, R83.2; no longer C17.1, R21.2
- net N$25: now also IC4.3, R95.1; no longer IC6.3, R40.1
- net N$27: now also IC6.3, R97.1; no longer IC5.3, R41.1
- net N$28: now also R98.2; no longer R42.2
- net N$29: now also C63.+, C64.1, R3.1, R79.1; no longer C25.1, C38.+, R25.1, R43.1
- net N$3: now also D8.A, D9.A; no longer D15.A, D16.A
- net N$30: now also R31.1; no longer R64.1
- net N$31: now also R31.2; no longer R64.2
- net N$33: now also R36.1; no longer R49.1
- net N$34: now also R29.1; no longer R66.1
- net N$35: now also R33.1; no longer R50.1
- net N$37: now also R1.1; no longer R44.1
- net N$38: now also C35.1, R51.2, R57.1; no longer IC5.5
- net N$39: now also R4.1; no longer R45.1
- net N$4: now also C14.1, R21.2, R26.1; no longer C29.1, R28.2, R35.1
- net N$40: now also R2.1; no longer R47.1
- net N$41: now also C34.1, R50.2, R56.1; no longer C72.1, R46.2, R70.1
- net N$43: now also R42.1; no longer R48.1
- net N$46: now also C39.1, R55.2, R61.1; no longer C86.1, R83.2, R84.1
- net N$48: now also C33.1, R45.2, R63.1; no longer C92.1, R90.1, R91.2
- net N$49: now also C48.1, J1.8, R64.1, R72.2; no longer C102.1, J2.8, R92.1, R99.2
- net N$5: now also C13.1, R20.2, R24.1; no longer C28.1, R27.2, R33.1
- net N$50: now also C49.1, J1.7, R65.1, R73.2; no longer C103.1, J2.7, R100.2, R93.1
- net N$51: now also C50.1, J1.6, R67.1, R74.2; no longer C104.1, J2.6, R101.2, R94.1
- net N$52: now also C52.1, J1.5, R68.1, R75.2; no longer C105.1, J2.5, R102.2, R95.1
- net N$53: now also C53.1, J1.4, R69.1, R76.2; no longer C106.1, J2.4, R103.2, R96.1
- net N$54: now also C51.1, J1.3, R70.1, R77.2; no longer C107.1, J2.3, R104.2, R97.1
- net N$55: now also C54.1, J1.2, R71.1, R78.2; no longer C108.1, J2.2, R105.2, R98.1
- net N$58: now also R32.1; no longer R51.1
- net N$59: now also R43.1; no longer R54.1
- net N$6: now also C8.1, R15.2, R23.1; no longer C18.1, R17.2, R32.1
- net N$60: now also R37.1; no longer R52.1
- net N$62: now also R41.1; no longer R55.1
- net N$64: now also R9.1; no longer R56.1
- net N$65: now also R8.1; no longer R57.1
- net N$66: now also R10.2; no longer R58.2
- net N$68: now also C67.1, D6.K, R81.5, R84.5, R87.1; no longer C9.1, D17.K, R39.5, R5.1, R7.5
- net N$7: now also C10.1, R17.2, R27.1; no longer C20.1, R19.2, R36.1
- net N$70: now also C68.1, D8.K, R81.2, R84.2, R88.1; no longer C5.1, D15.K, R3.1, R39.2, R7.2
- net N$71: now also R101.1; no longer R59.1
- net N$72: now also D19.K, R104.1; no longer D4.K, R62.1
- net N$73: now also D18.K, R103.1; no longer D5.K, R60.1
- net N$74: now also D17.K, R102.1; no longer D3.K, R61.1
- net N$78: now also D13.A, JP1.1; no longer D8.A, JP2.1
- net N$8: now also C32.1, R44.2, R58.1; no longer C76.1, R73.2, R74.1
- net N$9: now also C9.1, R16.2, R25.1; no longer C19.1, R18.2, R34.1
- net OLED_SCL: now also JP3.2, X3.6; no longer JP1.2, X1.6
- net OLED_SDA: now also JP3.1, X3.4; no longer JP1.1, X1.4
- net PCHG_FET: now also IC6.5; no longer IC5.1, X4.4
- net PVDD: now also C77.1, R91.1; no longer C15.1, R11.1
- net RDTX_OUT+: now also X3.5; no longer X1.5
- net RDTX_OUT-: now also X3.9; no longer X1.9
- net RESET: now also R30.1; no longer R67.1
- net RX_O: now also X2.14, X4.2; no longer X4.14, X5.2
- net S-LED_1: now also X3.11; no longer X1.11
- net S-LED_2: now also X3.13; no longer X1.13
- net S-LED_3: now also D17.A, X3.15; no longer D3.A, X1.15
- net S-LED_4: now also D18.A, X3.17; no longer D5.A, X1.17
- net S-LED_5: now also D19.A, X3.19; no longer D4.A, X1.19
- net SW: now also C65.2, R80.2, R82.2, R83.1; no longer C24.2, R16.2, R21.1, R24.2
- net T: now also X1.10; no longer X2.10
- net TX_O: now also X2.16, X4.3; no longer X4.16, X5.3
- net T_SUPPLY: now also X1.2; no longer X2.2
- net V+: now also D11.A, R94.1, T3.2, T3.3, T3.4, T3.5, T3.6, T3.7, T3.8, T4.2, T4.3, T4.4, T4.5, T4.6, T4.7, T4.8; no longer D1.A, R30.1, T1.2, T1.3, T1.4, T1.5, T1.6, T1.7, T1.8, T2.2, T2.3, T2.4, T2.5, T2.6, T2.7, T2.8
- net V-: now also R81.1, R81.3, R84.1, R84.3, R92.1, T1.2, T1.3, T1.4, T1.5, T1.6, T1.7, T1.8, T2.2, T2.3, T2.4, T2.5, T2.6, T2.7, T2.8; no longer R29.1, R39.1, R39.3, R7.1, R7.3, T3.2, T3.3, T3.4, T3.5, T3.6, T3.7, T3.8, T4.2, T4.3, T4.4, T4.5, T4.6, T4.7, T4.8
- net VC1: now also X1.3; no longer X2.3
- net VC10: now also X1.16; no longer X2.16
- net VC11: now also X1.8; no longer X2.8
- net VC12: now also X1.17; no longer X2.17
- net VC13: now also X1.9; no longer X2.9
- net VC2: now also X1.12; no longer X2.12
- net VC3: now also X1.4; no longer X2.4
- net VC4: now also X1.13; no longer X2.13
- net VC5: now also X1.5; no longer X2.5
- net VC6: now also X1.14; no longer X2.14
- net VC7: now also X1.6; no longer X2.6
- net VC8: now also X1.15; no longer X2.15
- net VC9: now also X1.7; no longer X2.7
- net VCOM: now also C22.1, R29.2, R64.2, R65.2, R67.2, R68.2, R69.2, R70.2, R71.2; no longer C67.1, R66.2, R92.2, R93.2, R94.2, R95.2, R96.2, R97.2, R98.2
- net VDD: now also C76.1, R91.2, X2.13, X3.12; no longer C14.1, R11.2, X1.12, X4.13
- net VIN: now also R90.2; no longer R12.2
- net VPWR: now also C61.1, D1.K, D2.K, D3.K, D4.K, D5.K, R66.2; no longer C1.1, D10.K, D11.K, D12.K, D13.K, D14.K, R1.2
- net WAKE: now also C78.2, D16.K, R100.1, R99.2; no longer C30.2, D6.K, R63.2, R65.1
Routing:
- net CB_14/13_C: track 212.7 -> 1.92 mm, vias 2 -> 0
- net CELL14+: track 3.06 -> 175.9 mm
- net +15V: track 0.00 -> 152.7 mm, vias 0 -> 1
- net N$9: track 3.02 -> 146.3 mm, vias 0 -> 2
- net CB_2/1_C: track 1.88 -> 84.3 mm, vias 0 -> 4
- net CELL1-: track 84.5 -> 5.76 mm
- net N$1: track 3.07 -> 72.7 mm, vias 0 -> 2
- net N$6: track 3.06 -> 71.5 mm
- net CB_4/3_C: track 1.89 -> 65.2 mm, vias 0 -> 2
- net CB_8/7_C: track 1.88 -> 54.4 mm, vias 0 -> 1
- net DSG_FET: track 0.00 -> 50.5 mm, vias 0 -> 1
- net CB_9: track 0.00 -> 49.8 mm, vias 0 -> 2
- net VCC: track 47.7 -> 0.00 mm
- net CT_8: track 7.13 -> 51.8 mm
- net CB_10: track 0.00 -> 42.5 mm, vias 0 -> 4
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
Commit message: afe board and schematic files are updatd !
Parts:
- moved IC2 106.4 mm to (114.9, 132.7)
- moved R35 106.3 mm to (-59.7, -12.1)
- moved R39 106.3 mm to (-59.7, -3.17)
- moved R46 106.3 mm to (-59.7, -7.62)
- moved R29 88.9 mm to (95.2, 113.7)
- moved R31 88.9 mm to (93.3, 114.3)
- moved C49 85.1 mm to (132.7, 125.7)
- moved C50 85.1 mm to (130.2, 125.7)
- moved C51 85.1 mm to (122.6, 125.7)
- moved C52 85.1 mm to (127.6, 125.7)
- moved C53 85.1 mm to (125.1, 125.7)
- moved C54 85.1 mm to (120.0, 125.7)
- moved R64 85.1 mm to (135.3, 116.8), turned to 270 degrees
- moved R65 85.1 mm to (132.7, 116.8), turned to 270 degrees
- moved R67 85.1 mm to (130.2, 116.8), turned to 270 degrees
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Connections:
- net C_HIGH(VC14) renamed N$33
- net N$64 renamed CELL11+
- net N$65 renamed CELL13
- net VC10 renamed N$26
- removed net AGND: X1.1
- removed net N$33 (its old number): CELL6+.P$1, R36.1
- removed net N$35: CELL5+.P$1, R33.1
- removed net N$37: CELL12+.P$1, R1.1
- removed net N$39: CELL10+.P$1, R4.1
- removed net N$40: CELL8+.P$1, R2.1
- removed net N$43: CELL7+.P$1, R42.1
- removed net N$58: CELL4+.P$1, R32.1
- removed net N$59: CELL3+.P$1, R43.1
- removed net N$60: CELL2+.P$1, R37.1
- removed net N$62: CELL1+.P$1, R41.1
- removed net N$66: CELL9+.P$1, R10.2
- removed net T: X1.10
- removed net T_SUPPLY: X1.2
- removed net VC1: X1.3
- removed net VC11: X1.8
- removed net VC12: X1.17
- removed net VC13: X1.9
- removed net VC2: X1.12
- removed net VC3: X1.4
- removed net VC4: X1.13
- removed net VC5: X1.5
- removed net VC6: X1.14
- removed net VC7: X1.6
- removed net VC8: X1.15
- removed net VC9: X1.7
- new net CELL1+: CELL1+.P$1, R41.1, X1.2, X1.9
- new net CELL10+: CELL10+.P$1, R4.1, X1.10
- new net CELL12+: CELL12+.P$1, R1.1, X1.12
- new net CELL2+: CELL2+.P$1, R37.1, X1.5
- new net CELL3+: CELL3+.P$1, R43.1, X1.11
- new net CELL4+: CELL4+.P$1, R32.1, X1.3, X1.4
- new net CELL5+: CELL5+.P$1, R33.1, X1.13
- new net CELL6+: CELL6+.P$1, R36.1, X1.1, X1.6
- new net CELL7+: CELL7+.P$1, R42.1, X1.15
- new net CELL8+: CELL8+.P$1, R2.1, X1.8
- new net CELL9+: CELL9+.P$1, R10.2, X1.17
- net BGND: now also X1.7
- net CELL14+: now also CELL14+.P$1, R3.1, X1.14
- net GND: no longer X1.11
- net N$29: no longer CELL14+.P$1, R3.1
Routing:
- net CELL9+: track 0.00 -> 176.3 mm, vias 0 -> 1
- net CELL8+: track 0.00 -> 156.5 mm, vias 0 -> 1
- net CELL7+: track 0.00 -> 143.8 mm, vias 0 -> 1
- net CELL5+: track 0.00 -> 130.1 mm, vias 0 -> 1
- net CELL14+: track 175.9 -> 302.1 mm, vias 0 -> 3
- net CELL6+: track 0.00 -> 123.5 mm, vias 0 -> 1
- net N$9: track 146.3 -> 40.3 mm, vias 2 -> 1
- net CELL4+: track 0.00 -> 94.5 mm, vias 0 -> 1
- net CELL3+: track 0.00 -> 88.3 mm, vias 0 -> 1
- net CB_2/1_C: track 84.3 -> 11.2 mm, vias 4 -> 0
- net N$1: track 72.7 -> 0.00 mm, vias 2 -> 0
- net N$6: track 71.5 -> 0.00 mm
- net CELL2+: track 0.00 -> 64.8 mm, vias 0 -> 1
- net N$70: track 11.6 -> 69.5 mm
- net CB_4/3_C: track 65.2 -> 8.44 mm, vias 2 -> 0
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- added copper zone on layer 16, net PWR_DRAIN
- removed copper zone on layer 16, net PWR_DRAIN1

Commit message: brd, lyout changed
Parts:
- moved R15 48.5 mm to (60.3, -31.8)
- moved C8 48.5 mm to (56.5, -29.8)
- moved C11 39.9 mm to (22.2, -10.2)
- moved R34 33.1 mm to (-22.9, 42.5)
- moved C31 20.3 mm to (10.8, -6.35)
- moved R9 13.6 mm to (191.8, 4.45)
- moved R1 13.5 mm to (229.9, 55.9)
- moved R3 13.5 mm to (250.2, 56.5)
- moved R8 13.0 mm to (231.8, 3.17)
- moved R10 12.9 mm to (153.7, 5.71)
- moved R4 11.8 mm to (193.0, 54.0)
- moved R42 11.7 mm to (116.2, 6.99)
- moved R2 10.4 mm to (156.2, 52.7)
- moved C27 10.2 mm to (5.08, 45.1), turned to 180 degrees
- moved R36 9.69 mm to (118.1, 51.4)
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Connections:
- net CELL13 renamed CELL13+
- removed net N$26: X1.16
- removed net N$33: X1.18
- new net CB_14/13_C78: C3.1, R13.2, R19.1, R3.2, X1.5
- net BGND: now also R98.1; no longer X1.7
- net CB_10/9_C: now also X1.15
- net CB_12/11_C: now also X1.13
- net CB_13/12_C: now also X1.3
- net CB_13/12_C1: now also X1.1
- net CB_13/12_C2: now also X1.2
- net CB_13/12_C6: now also X1.4
- net CB_13/12_C7: now also X1.6
- net CB_13/12_C8: now also X1.8
- net CB_14/13_C: now also X1.11
- net CB_2/1_C: now also X1.9
- net CB_4/3_C: now also X1.16
- net CB_6/5_C: now also X1.18
- net CB_8/7_C: now also X1.17
- net CELL1+: no longer X1.2, X1.9
- net CELL1-: now also X1.7; no longer R98.1
- net CELL10+: no longer X1.10
- net CELL12+: no longer X1.12
- net CELL14+: no longer C3.1, R13.2, R19.1, R3.2, X1.14
- net CELL2+: no longer X1.5
- net CELL3+: no longer X1.11
- net CELL4+: no longer X1.3, X1.4
- net CELL5+: no longer X1.13
- net CELL6+: no longer X1.1, X1.6
- net CELL7+: no longer X1.15
- net CELL8+: no longer X1.8
- net CELL9+: no longer X1.17
Routing:
- net CELL14+: track 302.1 -> 38.2 mm, vias 3 -> 2
- net CB_14/13_C78: track 0.00 -> 254.7 mm, vias 0 -> 1
- net CB_14/13_C: track 1.92 -> 254.2 mm, vias 0 -> 1
- net CB_13/12_C: track 1.93 -> 228.2 mm, vias 0 -> 1
- net CB_12/11_C: track 3.92 -> 212.0 mm, vias 0 -> 1
- net CB_13/12_C1: track 1.93 -> 183.7 mm, vias 0 -> 1
- net CELL9+: track 176.3 -> 10.5 mm, vias 1 -> 0
- net CB_10/9_C: track 2.56 -> 164.5 mm, vias 0 -> 1
- net CELL8+: track 156.5 -> 8.38 mm, vias 1 -> 0
- net CB_13/12_C2: track 1.93 -> 143.6 mm, vias 0 -> 1
- net CELL7+: track 143.8 -> 6.66 mm, vias 1 -> 0
- net CELL5+: track 130.1 -> 8.34 mm, vias 1 -> 0
- net CELL6+: track 123.5 -> 9.00 mm, vias 1 -> 0
- net CB_8/7_C: track 6.68 -> 119.4 mm, vias 0 -> 1
- net CB_13/12_C6: track 1.93 -> 106.6 mm, vias 0 -> 1
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
Commit message: @AFE board and layout afe itt@3
Parts:
- moved C3 245.1 mm to (11.4, 47.0), turned to 180 degrees
- moved C5 229.1 mm to (9.53, 35.6)
- moved C1 199.1 mm to (38.1, 35.6)
- moved C4 162.4 mm to (38.1, 27.9)
- moved C6 162.4 mm to (38.1, 31.8)
- moved R16 159.7 mm to (41.3, 31.8), turned to 0 degrees
- moved R19 143.7 mm to (-15.9, -47.6), turned to 0 degrees
- moved R22 143.5 mm to (-13.3, -47.6), turned to 0 degrees
- moved C2 137.2 mm to (24.1, 43.2)
- moved C10 128.8 mm to (42.5, 26.0), turned to 180 degrees
- moved C12 127.3 mm to (-15.2, -45.7), turned to 180 degrees
- moved C7 124.4 mm to (38.1, 24.1)
- moved R17 123.6 mm to (41.3, 24.1)
- moved R23 119.5 mm to (-13.3, -52.7), turned to 0 degrees
- moved R27 117.9 mm to (44.5, 24.1), turned to 0 degrees
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Routing:
- net CB_13/12_C: track 228.2 -> 460.5 mm, vias 1 -> 3
- net CB_13/12_C1: track 183.7 -> 347.4 mm, vias 1 -> 2
- net CB_14/13_C78: track 254.7 -> 387.4 mm, vias 1 -> 3
- net CB_4/3_C: track 38.3 -> 164.2 mm, vias 1 -> 3
- net CB_10/9_C: track 164.5 -> 39.4 mm, vias 1 -> 2
- net CB_12/11_C: track 212.0 -> 98.0 mm, vias 1 -> 2
- net CT_2: track 21.6 -> 117.2 mm, vias 0 -> 3
- net CT_14: track 0.00 -> 92.1 mm
- net CT_REF: track 11.4 -> 99.6 mm, vias 0 -> 1
- net CB_13/12_C8: track 35.0 -> 112.6 mm
- net CB_14/13_C: track 254.2 -> 331.2 mm, vias 1 -> 2
- net CB_6/5_C: track 77.4 -> 6.17 mm
- net CB_8: track 0.00 -> 59.4 mm
- net CB_13/12_C6: track 106.6 -> 164.6 mm, vias 1 -> 2
- net CT_1: track 9.91 -> 64.6 mm
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
Commit message: brd : layout :sch update@4
Parts:
- removed R95, R97: 10k, ipc-7351-resistor:RESC1005X40AN
- removed X1: 87758-1816, con-molex:87758-1816
- added C79: 0.1uF, ipc-7351-capacitor:CAPC1608X92N
- added D20: 8.2V, ipc-7351-diode:SOD3718X135N
- added JP5: (no value), GreenFuel:1X15
- added R105, R106: 127E, ipc-7351-resistor:RESC1608X55N
- C22, C67, C68: device ipc-7351-capacitor:CAPC1005X60N -> ipc-7351-capacitor:CAPC1608X92N
- C61: device ipc-7351-capacitor:CAPC1005X60N -> ipc-7351-capacitor:CAPC2012X145AN
- D1: value 8.2v -> 43V; device ipc-7351-diode:SOD3718X135N -> ipc-7351-diode:SOD2514X100N
- D2: value 20v -> 27V
- D3: value 27v -> 8.2V
- D4: value 43v -> 20V
- D5: value 75v -> 75V
- R87, R88: device ipc-7351-resistor:RESC1005X40AN -> ipc-7351-resistor:RESC1608X55N
- R96: value 10k -> 127E; device ipc-7351-resistor:RESC1005X40AN -> ipc-7351-resistor:RESC1608X55N
- moved R96 220.5 mm to (-41.3, -22.2), flipped to the top, turned to 0 degrees
- moved R7 110.6 mm to (54.0, 38.7), flipped to the bottom, turned to 180 degrees
- moved C8 107.6 mm to (42.5, 40.0)
- moved R23 107.1 mm to (44.5, 37.5)
- moved C12 107.1 mm to (42.5, 44.5)
- moved R15 106.8 mm to (41.3, 37.5)
- moved R22 106.6 mm to (44.5, 41.9)
- moved R19 106.2 mm to (41.3, 41.9)
- moved R6 96.0 mm to (44.5, 38.7), flipped to the bottom, turned to 180 degrees
- moved R11 58.8 mm to (44.5, 43.2)
- moved R14 56.3 mm to (44.5, 34.3)
- moved R12 51.9 mm to (44.5, 24.1)
- moved C57 44.8 mm to (79.8, 77.0), turned to 0 degrees
- moved C51 44.7 mm to (111.1, 82.5)
- moved C53 44.7 mm to (113.7, 82.5)
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Connections:
- removed net N$25: IC4.3, R95.1
- removed net N$27: IC6.3, R97.1
- new net CB_5/4_C: JP5.4
- new net CB_7/6_C: JP5.6
- new net N$26: D20.A, D3.K
- new net N$33: IC5.1, R96.2
- new net N$35: IC6.1, R106.2
- net CB_10/9_C: now also JP5.14; no longer X1.15
- net CB_12/11_C: now also JP5.12; no longer X1.13
- net CB_13/12_C: now also JP5.11; no longer X1.3
- net CB_13/12_C1: now also JP5.13; no longer X1.1
- net CB_13/12_C2: now also JP5.15, JP5.9; no longer X1.2
- net CB_13/12_C6: no longer X1.4
- net CB_13/12_C7: no longer X1.6
- net CB_13/12_C8: no longer X1.8
- net CB_14/13_C: now also JP5.10; no longer X1.11
- net CB_14/13_C78: no longer X1.5
- net CB_2/1_C: now also JP5.2; no longer X1.9
- net CB_4/3_C: now also JP5.3; no longer X1.16
- net CB_6/5_C: now also JP5.5; no longer X1.18
- net CB_8/7_C: now also JP5.7, JP5.8; no longer X1.17
- net CELL1-: now also JP5.1; no longer X1.7
- net CHG_GATE: now also R96.1; no longer IC5.1
- net DSG_GATE: now also R105.1; no longer IC4.1
- net GND: now also C79.2, IC4.3, IC5.3, IC6.3; no longer R95.2, R96.2, R97.2
- net N$20: now also IC4.1, R105.2; no longer IC5.3, R96.1
- net PCHG_GATE: now also R106.1; no longer IC6.1
- net VCOM: now also C79.1
- net VPWR: now also D20.K; no longer D3.K
Routing:
- net CB_13/12_C: track 460.5 -> 76.1 mm, vias 3 -> 4
- net CB_14/13_C78: track 387.4 -> 50.1 mm, vias 3 -> 2
- net CB_14/13_C: track 331.2 -> 22.3 mm
- net CB_13/12_C1: track 347.4 -> 112.7 mm, vias 2 -> 3
- net CB_13/12_C6: track 164.6 -> 36.8 mm
- net CB_13/12_C2: track 186.7 -> 70.1 mm, vias 1 -> 2
- net CB_13/12_C7: track 122.9 -> 28.5 mm
- net CB_13/12_C8: track 112.6 -> 22.4 mm
- net CB_4/3_C: track 164.2 -> 75.4 mm, vias 3 -> 2
- net CB_6/5_C: track 6.17 -> 78.8 mm, vias 1 -> 2
- net CT_14: track 92.1 -> 27.3 mm
- net CB_2/1_C: track 23.9 -> 85.3 mm, vias 2 -> 1
- net CB_7: track 0.00 -> 57.8 mm, vias 0 -> 1
- net CB_6: track 0.00 -> 56.4 mm, vias 0 -> 1
- net CB_2: track 14.5 -> 65.0 mm
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