File: BMS_hw/AFE_PCB/BMSV1.0.brd (EAGLE design)
At the start: 272 x 60 mm, 242 parts, among them IC1 MC33771BEP, IC2 SFH6156, IC3 MIC28515V1, IC4 FOD8384-COC, IC5 FOD8384-COC, IC6 FOD8384-COC, J1 NTC, Q1 IRLML5203, Q2 IRLML5203, T1 IPT020N10N3V1, T2 IPT020N10N3V1, T3 IPT020N10N3V1, T4 IPT020N10N3V1, X2 87758-2016, X3 87758-2016, X4 22-23-2051, X5 22-23-2041

Commit message: itt@5
Connections:
- net CB_13/12_C8 renamed CB_3/2_C
- removed net CB_13/12_C1: C4.1, JP5.13, R14.1, R21.1, R4.2, R6.1
- removed net CB_13/12_C6: C26.1, R36.2, R39.1, R46.1, R51.1
- removed net CB_13/12_C7: C24.1, R32.2, R35.1, R47.1, R52.1
- removed net CB_14/13_C78: C3.1, R13.2, R19.1, R3.2
- new net CB_11/10_C: C4.1, JP5.10, R14.1, R21.1, R4.2, R6.1
- new net CB_14+/14_C: C3.1, JP5.14, R13.2, R19.1, R3.2
- new net CB_9/8_C: C2.1, JP5.8, R12.1, R18.1, R2.2, R5.1
- net CB_10/9_C: now also JP5.9; no longer JP5.14
- net CB_12/11_C: now also JP5.11; no longer JP5.12
- net CB_13/12_C: now also JP5.12; no longer JP5.11
- net CB_13/12_C2: no longer C2.1, JP5.9, R12.1, R18.1, R2.2, R5.1
- net CB_14/13_C: now also JP5.13; no longer JP5.10
- net CB_5/4_C: now also C24.1, R32.2, R35.1, R47.1, R52.1
- net CB_7/6_C: now also C26.1, R36.2, R39.1, R46.1, R51.1
- net CB_8/7_C: no longer JP5.8
Routing:
- net CB_13/12_C1: track 112.7 -> 0.00 mm, vias 3 -> 0
- net CB_11/10_C: track 0.00 -> 112.7 mm, vias 0 -> 3
- net CB_13/12_C2: track 70.1 -> 0.00 mm, vias 2 -> 0
- net CB_9/8_C: track 0.00 -> 65.4 mm, vias 0 -> 2
- net CB_14/13_C78: track 50.1 -> 0.00 mm, vias 2 -> 0
- net CB_14+/14_C: track 0.00 -> 50.1 mm, vias 0 -> 2
- net CB_7/6_C: track 0.00 -> 36.8 mm, vias 0 -> 2
- net CB_13/12_C6: track 36.8 -> 0.00 mm, vias 2 -> 0
- net CB_5/4_C: track 0.00 -> 28.5 mm, vias 0 -> 2
- net CB_13/12_C7: track 28.5 -> 0.00 mm, vias 2 -> 0
- net CB_8/7_C: track 90.0 -> 84.9 mm
