File: BMS_hw/AFE_PCB/BMSV1.0.brd (EAGLE design)
At the start: 272 x 60 mm, 242 parts, among them IC1 MC33771BEP, IC2 SFH6156, IC3 MIC28515V1, IC4 FOD8384-COC, IC5 FOD8384-COC, IC6 FOD8384-COC, J1 NTC, Q1 IRLML5203, Q2 IRLML5203, T1 IPT020N10N3V1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

Commit message: itt@6 itt@6
Parts:
- moved R96 5.12 mm to (-41.9, -17.1)
Changed lines of the file:
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@@
 <attribute name="VALUE" x="-23.475" y="26.5375" size="1.27" layer="27" font="vector" ratio="10"/>
 </element>
-<element name="R96" library="ipc-7351-resistor" package="RESC1608X55N" value="127E" x="-41.275" y="-22.225">
-<attribute name="NAME" x="-42.525" y="-21.4075" size="1.27" layer="25" font="vector" ratio="10"/>
-<attribute name="VALUE" x="-42.525" y="-24.3125" size="1.27" layer="27" font="vector" ratio="10"/>
+<element name="R96" library="ipc-7351-resistor" package="RESC1608X55N" value="127E" x="-41.91" y="-17.145">
+<attribute name="NAME" x="-43.16" y="-16.3275" size="1.27" layer="25" font="vector" ratio="10"/>
+<attribute name="VALUE" x="-43.16" y="-19.2325" size="1.27" layer="27" font="vector" ratio="10"/>
 </element>
 <element name="R105" library="ipc-7351-resistor" package="RESC1608X55N" value="127E" x="-41.275" y="-27.94">
@@
 <contactref element="X2" pad="9"/>
 <contactref element="R96" pad="1"/>
-<wire x1="-42.075" y1="-22.225" x2="211.725" y2="40.91" width="0" layer="19" extent="1-1"/>
+<wire x1="-42.71" y1="-17.145" x2="211.725" y2="40.91" width="0" layer="19" extent="1-1"/>
 </signal>
 <signal name="+15V">
@@
 <contactref element="R96" pad="2"/>
 <contactref element="IC5" pad="1"/>
-<wire x1="-40.475" y1="-22.225" x2="166.095" y2="38.1" width="0" layer="19" extent="1-16"/>
+<wire x1="-41.11" y1="-17.145" x2="166.095" y2="38.1" width="0" layer="19" extent="1-16"/>
 </signal>
 <signal name="N$35">

Commit message: itt@7
Connections:
- removed net CB_13/12_C2: JP5.15
- removed net CB_14/13C: IC1.5
- net CB_10/9_C: now also JP5.10; no longer JP5.9
- net CB_11/10_C: now also JP5.11; no longer JP5.10
- net CB_12/11_C: now also JP5.12; no longer JP5.11
- net CB_13/12_C: now also JP5.13; no longer JP5.12
- net CB_14+/14_C: now also JP5.15; no longer JP5.14
- net CB_14/13_C: now also IC1.5, JP5.14; no longer JP5.13
- net CB_3/2_C: now also JP5.3
- net CB_4/3_C: now also JP5.4; no longer JP5.3
- net CB_5/4_C: now also JP5.5; no longer JP5.4
- net CB_6/5_C: now also JP5.6; no longer JP5.5
- net CB_7/6_C: now also JP5.7; no longer JP5.6
- net CB_8/7_C: now also JP5.8; no longer JP5.7
- net CB_9/8_C: now also JP5.9; no longer JP5.8
Routing:
- net CB_14/13_C: track 22.3 -> 92.4 mm, vias 2 -> 4
- net CB_14/13C: track 33.9 -> 0.00 mm, vias 1 -> 0
- net CB_14+/14_C: track 50.1 -> 79.0 mm
- net CB_12/11_C: track 91.7 -> 117.1 mm
- net CB_13/12_C: track 76.1 -> 99.9 mm
- net CB_10/9_C: track 81.7 -> 94.5 mm
- net CB_11/10_C: track 112.7 -> 123.0 mm
- net CB_5/4_C: track 28.5 -> 35.9 mm
- net CB_3/2_C: track 22.4 -> 29.6 mm
- net CB_8/7_C: track 84.9 -> 90.0 mm
- net CB_7/6_C: track 36.8 -> 41.8 mm
- net CB_6/5_C: track 78.8 -> 83.7 mm
- net CB_9/8_C: track 65.4 -> 70.1 mm

Commit message: itt@7
Parts:
- removed J1: NTC, con-molex:6410-08
- added TP2, TP3, TP4, TP5, TP6, TP7, TP8, TP9: TPTH7035, simpa:TP7035
- C48, C49, C50, C51, C52, C53, C54: value 2.2uF -> 2200pF
- C55, C56, C57, C58, C59, C60, C62: value 1uF -> 1nF
- R72, R73, R74, R75, R76, R77, R78: value 10k -> 1k
- moved C23 65.3 mm to (59.7, 103.5)
- moved R30 65.3 mm to (57.1, 103.5)
- moved R74 54.0 mm to (95.2, 29.8), turned to 315 degrees
- moved R75 51.2 mm to (96.5, 31.1), turned to 315 degrees
- moved R73 50.9 mm to (94.0, 28.6)
- moved R72 49.3 mm to (92.7, 27.3)
- moved C56 46.9 mm to (92.1, 33.0)
- moved C55 46.6 mm to (90.8, 31.8)
- moved C57 44.8 mm to (93.3, 34.3), turned to 315 degrees
- moved C59 44.2 mm to (89.5, 30.5)
- moved IC2 18.7 mm to (97.8, 71.8)
- moved R76 15.4 mm to (97.8, 32.4)
- moved R77 15.3 mm to (99.1, 33.7)
- moved R78 15.3 mm to (100.3, 34.9), turned to 315 degrees
- moved C60 14.8 mm to (97.2, 38.1), turned to 315 degrees
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Connections:
- new net CSB: IC1.41
- net GND: now also TP8.P$1; no longer J1.1
- net N$49: now also TP2.P$1; no longer J1.8
- net N$50: now also TP3.P$1; no longer J1.7
- net N$51: now also TP4.P$1; no longer J1.6
- net N$52: now also TP5.P$1; no longer J1.5
- net N$53: now also TP6.P$1; no longer J1.4
- net N$54: now also TP7.P$1; no longer J1.3
- net N$55: now also TP9.P$1; no longer J1.2
Routing:
- net GND: track 48.3 -> 30.6 mm
- net CT_REF: track 60.0 -> 70.4 mm
- net N$68: track 58.5 -> 50.6 mm
- net GPIO5: track 7.07 -> 1.35 mm, vias 0 -> 1
- net GPIO6: track 6.86 -> 1.35 mm, vias 0 -> 1
- net ISENSE+: track 5.49 -> 10.7 mm
- net VANA: track 4.10 -> 0.00 mm
- net GPIO1: track 0.00 -> 3.72 mm, vias 0 -> 1
- net CT_6: track 57.6 -> 60.7 mm
- net ISENSE-: track 6.41 -> 9.46 mm
- net GPIO4: track 4.34 -> 1.35 mm, vias 0 -> 1
- net CB_7/6_C: track 41.8 -> 39.1 mm
- net RESET: track 2.61 -> 0.00 mm
- net GPIO0: track 0.00 -> 2.18 mm, vias 0 -> 1
- net GPIO3: track 0.00 -> 1.35 mm, vias 0 -> 1
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
Commit message: itt@8
Parts:
- removed TP1: TPTH7035, simpa:TP7035
- added BGND, PACK-: (no value), simpa:WPAD
- R31: value 10k -> 127E
- moved TP9 170.4 mm to (91.4, 45.7)
- moved TP7 164.5 mm to (88.9, 45.7)
- moved TP6 160.5 mm to (86.4, 45.7)
- moved TP5 156.6 mm to (83.8, 45.7)
- moved TP8 154.7 mm to (73.7, 45.7)
- moved TP4 152.7 mm to (81.3, 45.7)
- moved TP3 148.7 mm to (78.7, 45.7)
- moved TP2 144.8 mm to (76.2, 45.7)
- moved R30 68.5 mm to (84.5, 40.6), turned to 45 degrees
- moved C23 68.0 mm to (87.0, 41.3)
- moved C49 61.3 mm to (93.3, 27.9), flipped to the bottom, turned to 225 degrees
- moved C50 58.5 mm to (94.6, 29.2), flipped to the bottom, turned to 225 degrees
- moved R64 58.2 mm to (93.3, 24.1), flipped to the bottom, turned to 225 degrees
- moved C52 55.9 mm to (95.9, 30.5), flipped to the bottom, turned to 225 degrees
- moved R65 55.1 mm to (94.6, 25.4), flipped to the bottom, turned to 225 degrees
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Connections:
- net BGND: now also BGND.1
- net V+: now also PACK-.1
Routing:
- net GND: track 30.6 -> 59.7 mm
- net RDTX_OUT-: track 0.00 -> 14.6 mm
- net SCLK: track 0.00 -> 14.4 mm
- net GPIO6: track 1.35 -> 15.7 mm
- net MOSI: track 0.00 -> 14.1 mm
- net RDTX_OUT+: track 0.00 -> 13.9 mm
- net N$30: track 0.00 -> 12.3 mm
- net N$34: track 0.00 -> 12.1 mm
- net MISO: track 0.00 -> 12.0 mm
- net GPIO5: track 1.35 -> 13.2 mm
- net CSB: track 0.00 -> 11.6 mm
- net CB_2/1_C: track 85.3 -> 73.9 mm
- net CB_2: track 65.0 -> 55.1 mm
- net CT_1: track 69.7 -> 62.3 mm
- net CT_REF: track 70.4 -> 62.9 mm
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
Commit message: itt @ coil-craft MSS library created, @afe layout 90% complete ! @schhematic altr @3!
Parts:
- added D21: 8.2V, ipc-7351-diode:SOD3718X135N
- added IC7, IC8: SFH6156-1, optocoupler:SFH
- added R95, R97: 127E, ipc-7351-resistor:RESC1005X40AN
- D2: value 27V -> 33V
- IC2: value SFH6156 -> SFH6156-1
- L1: value XAL1010-822MEB -> MSS1278-D; device GreenFuel:DUALPAD -> GreenFuel:MSS1278D/T
- PACK-: value (none) -> PACK-
- moved D4 59.4 mm to (74.9, 36.8), turned to 0 degrees
- moved IC2 53.4 mm to (95.9, 18.4)
- moved C48 26.1 mm to (77.5, 48.3), turned to 135 degrees
- moved C49 24.3 mm to (80.0, 48.3), turned to 135 degrees
- moved C50 22.6 mm to (82.2, 48.1), turned to 135 degrees
- moved C52 21.1 mm to (84.5, 48.3), turned to 135 degrees
- moved C53 19.4 mm to (87.0, 48.3), turned to 135 degrees
- moved C51 16.7 mm to (89.5, 48.3), turned to 135 degrees
- moved C79 14.9 mm to (-33.7, 19.1)
- moved C54 14.8 mm to (92.1, 48.3), turned to 135 degrees
- moved R34 9.94 mm to (-33.7, 48.9)
- moved R64 6.87 mm to (89.5, 29.8)
- moved R68 6.87 mm to (93.3, 33.7)
- moved R67 6.87 mm to (92.1, 32.4)
- moved R69 6.87 mm to (94.6, 34.9)
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Connections:
- new net N$25: IC7.1, R95.2
- new net N$27: IC8.1, R97.2
- new net N$36: D21.K, R95.1
- net FAULT_OUT: now also IC7.3, IC8.3
- net GND: now also IC7.2, IC8.2
- net VCORE: now also IC7.4, IC8.4
Routing:
- net +15V: track 152.7 -> 42.6 mm, vias 1 -> 0
- net CELL1-: track 25.3 -> 66.6 mm
- net N$49: track 4.93 -> 24.2 mm
- net N$50: track 4.93 -> 22.4 mm
- net VCOM: track 4.07 -> 21.4 mm, vias 0 -> 1
- net N$9: track 35.1 -> 18.3 mm, vias 1 -> 0
- net CB_14+/14_C: track 79.0 -> 62.3 mm
- net CB_2/1_C: track 73.9 -> 90.4 mm, vias 1 -> 2
- net N$51: track 4.93 -> 20.4 mm
- net N$52: track 4.93 -> 18.6 mm
- net GND: track 59.7 -> 47.2 mm
- net N$54: track 2.87 -> 15.0 mm
- net GATE: track 16.6 -> 4.55 mm, vias 2 -> 0
- net N$53: track 4.93 -> 16.8 mm
- net N$55: track 2.87 -> 13.2 mm
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
Commit message: board afe and layout
Parts:
- removed C69: 47nF, ipc-7351-capacitor:CAPC1608X92N
- removed C70: 47nF, ipc-7351-capacitor:CAPC3225X168N
- added C80: 2.2uF 100V, ipc-7351-capacitor:CAPC3225X168N
- C63: value (none) -> 0.1uF 100V; device ipc-7351-capacitor:CAPAE830X620N -> ipc-7351-capacitor:CAPC1608X92N
- C64: value 47nF -> 2.2uF 100V
- C65: value 47nF -> 0.1uF 100V; device ipc-7351-capacitor:CAPC1005X60N -> ipc-7351-capacitor:CAPC1608X92N
- C66, C73, C74, C76, C77: device ipc-7351-capacitor:CAPC1005X60N -> ipc-7351-capacitor:CAPC1608X92N
- R79, R85, R89, R90, R91: device ipc-7351-resistor:RESC1005X40AN -> ipc-7351-resistor:RESC1608X55N
- R80, R82: value 127E -> 1.6k; device ipc-7351-resistor:RESC1005X40AN -> ipc-7351-resistor:RESC1608X55N
- R83: value 127E -> 16.2k; device ipc-7351-resistor:RESC1005X40AN -> ipc-7351-resistor:RESC1608X55N
- moved C63 340.6 mm to (-64.8, -82.5)
- moved C64 331.5 mm to (-63.5, -87.6)
- moved D20 89.3 mm to (66.7, 47.6), flipped to the bottom, turned to 180 degrees
- moved R29 56.3 mm to (92.7, 16.5), turned to 315 degrees
- moved R31 53.6 mm to (94.0, 16.5), turned to 315 degrees
- moved D3 43.8 mm to (66.7, 45.7), turned to 0 degrees
- moved D2 41.2 mm to (61.6, 48.3)
- moved C61 40.6 mm to (71.1, 47.0), flipped to the bottom, turned to 270 degrees
- moved D5 38.4 mm to (66.7, 49.7), turned to 180 degrees
- moved D1 36.9 mm to (59.1, 48.9)
- moved IC2 5.75 mm to (101.6, 17.8)
Connections:
- net +15V: no longer C69.1, C70.1
- net CB_10/9_C: now also JP5.4; no longer JP5.10
- net CB_12/11_C: now also JP5.5; no longer JP5.12
- net CB_13/12_C: now also JP5.10; no longer JP5.13
- net CB_14+/14_C: now also JP5.9; no longer JP5.15
- net CB_14/13_C: now also JP5.6; no longer JP5.14
- net CB_2/1_C: now also JP5.7; no longer JP5.2
- net CB_3/2_C: now also JP5.15; no longer JP5.3
- net CB_4/3_C: now also JP5.1; no longer JP5.4
- net CB_5/4_C: now also JP5.14; no longer JP5.5
- net CB_6/5_C: now also JP5.2; no longer JP5.6
- net CB_7/6_C: now also JP5.13; no longer JP5.7
- net CB_8/7_C: now also JP5.3; no longer JP5.8
- net CB_9/8_C: now also JP5.12; no longer JP5.9
- net CELL1-: now also JP5.8; no longer JP5.1
- net GND: now also C63.1, C64.1, C80.1; no longer C63.-, C64.2, C69.2, C70.2
- net N$29: now also C63.2, C64.2, C80.2; no longer C63.+, C64.1
Routing:
- net CB_14+/14_C: track 62.3 -> 318.0 mm
- net CB_13/12_C: track 100.5 -> 330.5 mm
- net CB_11/10_C: track 123.7 -> 317.2 mm
- net CB_9/8_C: track 70.7 -> 218.2 mm
- net CELL1-: track 66.6 -> 45.5 mm
- net CB_7/6_C: track 39.8 -> 20.1 mm, vias 2 -> 1
- net CB_12/11_C: track 116.4 -> 99.1 mm
- net CB_14/13_C: track 93.0 -> 77.4 mm
- net CB_8/7_C: track 90.6 -> 75.0 mm
- net CB_10/9_C: track 95.1 -> 80.8 mm
- net VCOM: track 21.4 -> 32.8 mm, vias 1 -> 2
- net VPWR: track 0.50 -> 11.4 mm, vias 0 -> 2
- net N$29: track 48.8 -> 39.7 mm
- net CB_6/5_C: track 84.3 -> 75.7 mm
- net CB_5/4_C: track 35.9 -> 28.5 mm
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- added copper zone on layer 1, net VPWR

Commit message: aaaaaaaaaaaaaa
Parts:
- moved R97 259.0 mm to (179.7, 40.6), turned to 270 degrees
- moved IC8 247.3 mm to (178.4, 33.0)
- moved R106 242.8 mm to (195.6, 19.7)
- moved IC7 228.2 mm to (172.7, 44.5), turned to 90 degrees
- moved R95 226.9 mm to (162.6, 44.5)
- moved R96 219.8 mm to (170.8, 38.1)
- moved R105 198.5 mm to (153.0, 12.7)
- moved C63 128.5 mm to (23.5, 10.8)
- moved C79 127.1 mm to (93.3, 14.0), turned to 315 degrees
- moved C16 52.1 mm to (70.5, 41.9)
- moved R34 39.5 mm to (5.71, 45.7)
- moved R66 23.3 mm to (62.2, 44.5), turned to 0 degrees
- moved C61 18.2 mm to (63.5, 63.5)
- moved D2 15.6 mm to (58.4, 63.5)
- moved D1 14.9 mm to (55.9, 63.5)
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Routing:
- net CB_14/13_C: track 77.4 -> 332.4 mm, vias 4 -> 6
- net CB_12/11_C: track 99.1 -> 347.6 mm, vias 5 -> 9
- net CB_8/7_C: track 75.0 -> 253.9 mm, vias 3 -> 4
- net CB_10/9_C: track 80.8 -> 259.3 mm, vias 4 -> 5
- net CB_7/6_C: track 20.1 -> 149.6 mm, vias 1 -> 3
- net CB_6/5_C: track 75.7 -> 176.0 mm
- net CB_5/4_C: track 28.5 -> 116.3 mm, vias 2 -> 3
- net CB_3/2_C: track 25.1 -> 80.0 mm, vias 2 -> 3
- net CB_4/3_C: track 69.4 -> 122.1 mm
- net CB_9/8_C: track 218.2 -> 247.8 mm, vias 2 -> 4
- net CELL1-: track 45.5 -> 70.3 mm, vias 1 -> 3
- net CB_13/12_C: track 330.5 -> 347.5 mm, vias 4 -> 6
- net CB_2/1_C: track 92.5 -> 106.5 mm, vias 1 -> 2
- net VPWR: track 11.4 -> 24.3 mm
- net CB_11/10_C: track 317.2 -> 329.7 mm, vias 3 -> 6
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
Commit message: itt@8
Parts:
- added R107: (no value), ipc-7351-resistor:RESC1608X55N
- PACK-: value PACK- -> (none)
- moved D21 245.0 mm to (148.6, 45.7), flipped to the bottom
- moved C80 138.9 mm to (30.5, 8.89), turned to 180 degrees
- moved C64 131.4 mm to (23.5, 10.8), flipped to the bottom
- moved R94 6.54 mm to (157.5, 42.5)
- moved IC2 5.12 mm to (104.1, 13.3)
- moved IC6 3.18 mm to (175.3, 18.4)
- moved Q2 2.01 mm to (173.4, 18.4)
- moved PACK- 1.42 mm to (167.6, 30.5), flipped to the top
- moved BGND 1.42 mm to (104.1, 30.5)
Connections:
- removed net FAULT: X2.5
- new net N$12: IC3.24, R107.1
- net CSB: now also X3.7
- net FAULT_OUT: now also X2.5
- net GND: now also IC3.26; no longer X3.7
- net VIN: now also R107.2
Routing:
- net CB_14/13_C: track 332.4 -> 363.8 mm, vias 6 -> 8
- net CB_10/9_C: track 259.3 -> 283.9 mm, vias 5 -> 6
- net V+: track 44.0 -> 39.5 mm
- net N$31: track 3.14 -> 6.47 mm
- net CB_7/6_C: track 149.6 -> 146.4 mm
- net N$49: track 24.2 -> 22.5 mm
- net PWR_DRAIN: track 25.4 -> 27.1 mm
- net GND: track 47.0 -> 45.6 mm
- net CB_3/2_C: track 80.0 -> 81.2 mm
- net CB_9/8_C: track 247.8 -> 247.0 mm
- net CB_11/10_C: track 329.7 -> 329.0 mm
- added copper zone on layer 1, net BGND
- added copper zone on layer 16, net BGND
