File: BMS_hw/AFE_PCB/BMSV1.0.brd (EAGLE design)
At the start: 272 x 60 mm, 255 parts, among them IC1 MC33771BEP, IC2 SFH6156-1, IC3 MIC28515V1, IC4 FOD8384-COC, IC5 FOD8384-COC, IC6 FOD8384-COC, IC7 SFH6156-1, IC8 SFH6156-1, Q1 IRLML5203, Q2 IRLML5203, T1 IPT020N10N3V1, T2 IPT020N10N3V1, T3 IPT020N10N3V1, T4 IPT020N10N3V1, X2 87758-2016, X3 87758-2016, X4 22-23-2051, X5 22-23-2041

Commit message: @ITT9
Parts:
- moved R34 102.4 mm to (102.9, 13.3)
- moved D1 29.9 mm to (37.5, 40.0)
- moved D2 18.9 mm to (46.4, 48.9), turned to 0 degrees
- moved D5 18.0 mm to (71.8, 49.0), turned to 180 degrees
- moved C61 15.5 mm to (61.0, 48.3)
- moved C63 3.86 mm to (19.7, 10.2), turned to 90 degrees
- moved R39 0.46 mm to (29.9, 40.5)
Connections:
- removed net ISP: X2.11
- net GND: no longer X2.1, X2.6
- net MISO: now also X2.11
- net MOSI: now also X2.6
- net SCLK: now also X2.1
Routing:
- net CB_8/7_C: track 253.7 -> 224.1 mm, vias 4 -> 6
- net VPWR: track 24.3 -> 47.4 mm
- net CB_9/8_C: track 247.0 -> 226.4 mm, vias 4 -> 2
- net GND: track 45.6 -> 62.1 mm, vias 59 -> 79
- net CB_5/4_C: track 116.3 -> 101.7 mm
- net BGND: track 11.5 -> 21.4 mm
- net CB_14+/14_C: track 310.3 -> 318.1 mm, vias 2 -> 4
- net CELL1-: track 70.3 -> 65.7 mm
- net N$17: track 4.02 -> 0.32 mm
- net N$18: track 2.85 -> 0.00 mm
- net CB_7/6_C: track 146.4 -> 149.2 mm
- net ILIM: track 6.20 -> 3.51 mm
- net CB_10/9_C: track 283.9 -> 282.4 mm
- net CB_7: track 57.6 -> 58.6 mm
- net CB_3/2_C: track 81.2 -> 80.5 mm

Commit message: @board layout schmeatic itt@10
Parts:
- moved Q1 33.5 mm to (187.3, 50.2)
- moved D10 22.5 mm to (181.6, 50.8)
- moved R94 19.5 mm to (175.9, 48.9)
- moved R93 19.3 mm to (175.9, 51.4)
- moved IC7 16.0 mm to (188.6, 42.5), flipped to the bottom
- moved D1 15.4 mm to (50.8, 47.6), turned to 0 degrees
- moved R95 10.5 mm to (172.7, 47.0)
- moved D8 9.94 mm to (104.1, 51.4)
- moved D9 9.94 mm to (109.9, 51.4)
- moved C3 8.84 mm to (57.8, 44.4)
- moved R66 7.24 mm to (66.7, 50.2), turned to 180 degrees
- moved C68 6.75 mm to (113.7, 48.9), turned to 270 degrees
- moved C67 5.85 mm to (118.1, 46.4)
- moved D11 5.85 mm to (167.0, 48.9)
- moved IC2 5.85 mm to (108.0, 17.8)
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Connections:
- net CB_14+/14_C: now also R66.1
- net CELL14+: no longer R66.1
Routing:
- net CB_11/10_C: track 329.4 -> 282.3 mm
- net DSG_FET: track 38.3 -> 0.00 mm
- net CB_14+/14_C: track 318.1 -> 296.6 mm
- net CB_13/12_C: track 347.5 -> 326.3 mm
- net CELL14+: track 38.2 -> 18.0 mm
- net N$9: track 18.3 -> 4.20 mm
- net N$71: track 13.9 -> 0.00 mm
- net CB_8/7_C: track 224.1 -> 236.1 mm, vias 6 -> 9
- net CB_5/4_C: track 101.7 -> 111.6 mm, vias 3 -> 6
- net N$68: track 50.6 -> 59.3 mm
- net CT_14: track 19.2 -> 24.9 mm
- net N$70: track 56.5 -> 62.0 mm
- net N$25: track 5.16 -> 0.00 mm
- net CB_10/9_C: track 282.4 -> 287.2 mm, vias 6 -> 8
- net CB_9/8_C: track 226.4 -> 223.1 mm
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
Commit message: hjhk
Parts:
- removed X2, X3: 87758-2016, con-molex:87758-2016
- added JP4, JP6: (no value), GreenFuel:1X15
- moved R107 132.0 mm to (230.5, 29.2), turned to 270 degrees
- moved R34 6.48 mm to (105.4, 24.1), turned to 135 degrees
- moved C67 2.01 mm to (116.2, 47.0), turned to 90 degrees
- moved C68 1.90 mm to (113.7, 50.8), turned to 90 degrees
- moved R36 0.64 mm to (118.7, 51.4)
Connections:
- net !MCLR: no longer X2.10
- net +15V: no longer X2.17
- net 3.3V: no longer X2.12, X3.16
- net CHG_GATE: no longer X2.9
- net CSB: no longer X3.7
- net DSG_GATE: no longer X2.19
- net FAULT_OUT: no longer X2.5
- net GND: no longer X2.15, X2.18, X2.2, X2.20, X2.3, X2.7, X2.8, X3.1, X3.10, X3.14, X3.18, X3.2, X3.20, X3.3, X3.8
- net MISO: no longer X2.11
- net MOSI: no longer X2.6
- net OLED_SCL: no longer X3.6
- net OLED_SDA: no longer X3.4
- net PCHG_GATE: no longer X2.4
- net RDTX_OUT+: no longer X3.5
- net RDTX_OUT-: no longer X3.9
- net RX_O: no longer X2.14
- net S-LED_1: no longer X3.11
- net S-LED_2: no longer X3.13
- net S-LED_3: no longer X3.15
- net S-LED_4: no longer X3.17
- net S-LED_5: no longer X3.19
- net SCLK: no longer X2.1
- net TX_O: no longer X2.16
- net VDD: no longer X2.13, X3.12
Routing:
- net GND: track 61.3 -> 53.5 mm, vias 101 -> 114
- net N$68: track 59.3 -> 55.2 mm
- net BGND: track 21.4 -> 20.3 mm
- net N$70: track 62.0 -> 61.0 mm
- net CELL6+: track 9.00 -> 8.37 mm
- net CB_7/6_C: track 151.7 -> 152.3 mm

Commit message: asdasd
Parts:
- added S1: PGBRD6030-6030, GreenFuel:PIG6030
- moved JP4 254.7 mm to (224.2, 42.5)
- moved JP6 251.3 mm to (224.2, 19.7)
- moved C73 117.0 mm to (348.6, 6.35)
- moved C74 117.0 mm to (359.4, 0.01)
- moved C77 117.0 mm to (348.6, 8.90)
- moved C78 117.0 mm to (336.6, 15.2)
- moved D16 117.0 mm to (336.6, 13.3)
- moved JP1 117.0 mm to (339.7, 3.81)
- moved R100 117.0 mm to (332.1, 13.3)
- moved R79 117.0 mm to (359.4, 3.17)
- moved R80 117.0 mm to (363.9, 6.35)
- moved R83 117.0 mm to (362.6, 1.91)
- moved R85 117.0 mm to (356.9, -1.91)
- moved R91 117.0 mm to (349.3, 4.45)
- moved R99 117.0 mm to (339.7, 10.8)
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Routing:
- net N$29: track 31.1 -> 94.6 mm, vias 2 -> 0
- net SW: track 35.4 -> 0.00 mm, vias 2 -> 0
- net GND: track 53.5 -> 27.9 mm, vias 114 -> 104
- net +15V: track 41.3 -> 17.5 mm
- net KEY-IN: track 16.2 -> 0.00 mm
- net N$24: track 16.0 -> 0.00 mm, vias 2 -> 0
- net CANL: track 14.0 -> 0.00 mm
- net WAKE: track 10.7 -> 0.00 mm
- net PVDD: track 10.1 -> 0.00 mm, vias 2 -> 0
- net FB: track 8.85 -> 0.35 mm
- net CELL14+: track 18.0 -> 9.90 mm, vias 2 -> 0
- net CANH: track 6.45 -> 0.00 mm
- net N$21: track 5.32 -> 0.00 mm
- net ILIM: track 3.51 -> 0.00 mm
- net VDD: track 2.61 -> 0.00 mm
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
Commit message: ITT@112
Parts:
- moved C22 1.42 mm to (88.9, 26.0), turned to 45 degrees
- moved C47 0.90 mm to (90.2, 20.3), turned to 315 degrees
Connections:
- net CSB: now also JP6.4
- net MISO: now also JP6.3
- net MOSI: now also JP6.1
- net SCLK: now also JP6.2
Routing:
- net CSB: track 5.56 -> 142.2 mm
- net SCLK: track 3.79 -> 138.9 mm
- net MISO: track 5.35 -> 139.7 mm
- net MOSI: track 3.58 -> 135.9 mm
- net RDTX_OUT-: track 14.6 -> 0.00 mm
- net RDTX_OUT+: track 13.9 -> 0.00 mm
- net N$71: track 0.00 -> 8.40 mm
- net GND: track 27.9 -> 23.3 mm, vias 104 -> 108
- net VCOM: track 34.4 -> 32.9 mm
- net CT_REF: track 62.9 -> 62.0 mm

Commit message: brd layout and sch updated!
Parts:
- moved IC6 4.58 mm to (175.3, 20.3)
Connections:
- net 3.3V: now also JP4.1
Routing:
- net 3.3V: track 0.00 -> 54.1 mm, vias 0 -> 1
- net CT_1: track 62.3 -> 61.1 mm
- net CT_REF: track 62.0 -> 61.2 mm
- net CT_2: track 63.0 -> 62.3 mm
- net MOSI: track 135.9 -> 135.4 mm
- net MISO: track 139.7 -> 139.1 mm
- net CSB: track 142.2 -> 141.7 mm
- net SCLK: track 138.9 -> 138.4 mm
- net GND: track 23.3 -> 23.2 mm, vias 108 -> 112

Commit message: board layout and schematic files updated@12
Parts:
- added C69, C70: 10uF, ipc-7351-capacitor:CAPC1005X60N
- added C81, C82: 10uF, ipc-7351-capacitor:CAPC1608X92N
- added U1, U2: NCP1117LP-PG, GreenFuel:SOT-223
Connections:
- new net 15V_AUX: C70.2, C82.2, U1.3, U2.3
- new net 5V: C81.2, U2.2
- net 3.3V: now also C69.2, U1.2
- net GND: now also C69.1, C70.1, C81.1, C82.1, U1.1, U1.4, U2.1, U2.4

Commit message: @itt@17
Parts:
- added R108: 0R, ipc-7351-resistor:RESC1608X55N
- C77: value 2.2uF -> 4.7uF; device ipc-7351-capacitor:CAPC1608X92N -> ipc-7351-capacitor:CAPC2012X145AN
- R107: value (none) -> 100k
- R91: value 2E2 -> 1R
Connections:
- removed net N$29: C63.2, C64.2, C80.2, IC3.10, IC3.11, IC3.5, IC3.6, IC3.7, IC3.8, IC3.9, R79.1
- new net N$13: C65.2, R108.1
- net SW: now also R108.2; no longer C65.2
- net VIN: now also C63.2, C64.2, C80.2, IC3.10, IC3.11, IC3.5, IC3.6, IC3.7, IC3.8, IC3.9, R79.1
Routing:
- net VIN: track 0.00 -> 94.6 mm
- net N$29: track 94.6 -> 0.00 mm
Changed lines of the file:
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@@
 <attribute name="VALUE" x="355.026" y="2.675" size="1.27" layer="27" font="vector" ratio="10" rot="R270"/>
 </element>
-<element name="C77" library="ipc-7351-capacitor" package="CAPC1608X92N" value="2.2uF" x="348.617" y="8.897" rot="R90">
+<element name="C77" library="ipc-7351-capacitor" package="CAPC2012X145AN" value="4.7uF" x="348.617" y="8.897" rot="R90">
 <attribute name="NAME" x="348.038" y="8.122" size="1.27" layer="25" font="vector" ratio="10" rot="R90"/>
 <attribute name="VALUE" x="350.466" y="8.122" size="1.27" layer="27" font="vector" ratio="10" rot="R90"/>
 </element>
-<element name="R91" library="ipc-7351-resistor" package="RESC1608X55N" value="2E2" x="349.252" y="4.447">
+<element name="R91" library="ipc-7351-resistor" package="RESC1608X55N" value="1R" x="349.252" y="4.447">
 <attribute name="NAME" x="348.502" y="5.001" size="1.27" layer="25" font="vector" ratio="10"/>
 <attribute name="VALUE" x="348.502" y="2.623" size="1.27" layer="27" font="vector" ratio="10"/>
@@
 <attribute name="VALUE" x="32.555" y="11.8275" size="1.27" layer="27" font="vector" ratio="10" rot="R180"/>
 </element>
-<element name="R107" library="ipc-7351-resistor" package="RESC1608X55N" value="" x="346.075" y="10.795" rot="R270">
+<element name="R107" library="ipc-7351-resistor" package="RESC1608X55N" value="100k" x="346.075" y="10.795" rot="R270">
 <attribute name="NAME" x="346.8925" y="12.045" size="0.508" layer="25" font="vector" ratio="12" rot="R270"/>
 <attribute name="VALUE" x="343.9875" y="12.045" size="1.27" layer="27" font="vector" ratio="10" rot="R270"/>
@@
 <attribute name="VALUE" x="-71.1" y="-36.3275" size="1.27" layer="27" font="vector" ratio="10"/>
 </element>
+<element name="R108" library="ipc-7351-resistor" package="RESC1608X55N" value="0R" x="-69.85" y="-50.165">
+<attribute name="NAME" x="-71.1" y="-49.3475" size="1.27" layer="25" font="vector" ratio="10"/>
+<attribute name="VALUE" x="-71.1" y="-52.2525" size="1.27" layer="27" font="vector" ratio="10"/>
+</element>
 </elements>
 <signals>
@@
 <wire x1="337" y1="15.24" x2="331.655" y2="13.335" width="0" layer="19" extent="1-1"/>
 <wire x1="338.25" y1="13.335" x2="337" y2="15.24" width="0" layer="19" extent="1-1"/>
-<wire x1="348.617" y1="9.697" x2="338.25" y2="13.335" width="0" layer="19" extent="1-1"/>
-<wire x1="351.9145" y1="9.895" x2="348.617" y2="9.697" width="0" layer="19" extent="1-1"/>
+<wire x1="348.617" y1="9.797" x2="338.25" y2="13.335" width="0" layer="19" extent="1-1"/>
+<wire x1="351.9145" y1="9.895" x2="348.617" y2="9.797" width="0" layer="19" extent="1-1"/>
 <wire x1="351.9145" y1="9.245" x2="351.9145" y2="9.895" width="0" layer="19" extent="1-1"/>
 <wire x1="351.9145" y1="8.595" x2="351.9145" y2="9.245" width="0" layer="19" extent="1-1"/>
@@
 <wire x1="354.9645" y1="6.35" x2="354.6395" y2="4.57" width="0" layer="19" extent="1-1"/>
 <wire x1="358.0145" y1="5.995" x2="354.9645" y2="6.35" width="0" layer="19" extent="1-1"/>
-<wire x1="347.815" y1="6.35" x2="348.617" y2="9.697" width="0" layer="19" extent="1-1"/>
+<wire x1="347.815" y1="6.35" x2="348.617" y2="9.797" width="0" layer="19" extent="1-1"/>
 <wire x1="356.875" y1="1.1" x2="355.2895" y2="4.57" width="0" layer="19" extent="1-1"/>
 <wire x1="357.323" y1="0.001" x2="356.875" y2="1.1" width="0" layer="19" extent="1-1"/>
@@
 <contactref element="C77" pad="1"/>
 <contactref element="R91" pad="1"/>
-<wire x1="348.617" y1="8.097" x2="351.9145" y2="7.295" width="0" layer="19" extent="1-1"/>
-<wire x1="348.452" y1="4.447" x2="348.617" y2="8.097" width="0" layer="19" extent="1-1"/>
+<wire x1="348.617" y1="7.997" x2="351.9145" y2="7.295" width="0" layer="19" extent="1-1"/>
+<wire x1="348.452" y1="4.447" x2="348.617" y2="7.997" width="0" layer="19" extent="1-1"/>
 </signal>
 <signal name="N$17">
@@
 <contactref element="R90" pad="2"/>
 <contactref element="R107" pad="2"/>
-<wire x1="351.787" y1="1.743" x2="346.075" y2="9.995" width="0" layer="19" extent="1-1"/>
+<contactref element="IC3" pad="9"/>
+<contactref element="IC3" pad="10"/>
+<contactref element="IC3" pad="11"/>
+<contactref element="IC3" pad="5"/>
+<contactref element="IC3" pad="6"/>
+<contactref element="IC3" pad="7"/>
+<contactref element="IC3" pad="8"/>
+<contactref element="R79" pad="1"/>
+<wire x1="367.03" y1="0.635" x2="272.415" y2="0.635" width="0.254" layer="16"/>
+<contactref element="C80" pad="2"/>
+<contactref element="C64" pad="2"/>
+<contactref element="C63" pad="2"/>
+<wire x1="356.5895" y1="10.67" x2="357.2395" y2="10.67" width="0" layer="19" extent="1-1"/>
+<wire x1="355.9395" y1="10.67" x2="356.5895" y2="10.67" width="0" layer="19" extent="1-1"/>
+<wire x1="358.0145" y1="9.895" x2="357.2395" y2="10.67" width="0" layer="19" extent="1-1"/>
+<wire x1="358.0145" y1="9.245" x2="358.0145" y2="9.895" width="0" layer="19" extent="1-1"/>
+<wire x1="358.0145" y1="8.595" x2="358.0145" y2="9.245" width="0" layer="19" extent="1-1"/>
+<wire x1="358.0145" y1="7.945" x2="358.0145" y2="8.595" width="0" layer="19" extent="1-1"/>
+<wire x1="360.21" y1="3.175" x2="358.0145" y2="7.945" width="0" layer="19" extent="1-1"/>
+<wire x1="367.03" y1="0.635" x2="360.21" y2="3.175" width="0" layer="19" extent="1-16"/>
+<wire x1="351.787" y1="1.743" x2="360.21" y2="3.175" width="0" layer="19" extent="1-1"/>
+<wire x1="346.075" y1="9.995" x2="355.9395" y2="10.67" width="0" layer="19" extent="1-1"/>
+<wire x1="28.98" y1="8.89" x2="272.415" y2="0.635" width="0" layer="19" extent="1-16"/>
+<wire x1="21.995" y1="10.795" x2="28.98" y2="8.89" width="0" layer="19" extent="1-16"/>
+<wire x1="19.685" y1="10.96" x2="21.995" y2="10.795" width="0" layer="19" extent="1-16"/>
 </signal>
 <signal name="N$18">
@@
 <signal name="SW">
 <contactref element="R80" pad="2"/>
-<contactref element="C65" pad="2"/>
 <contactref element="R82" pad="2"/>
 <contactref element="IC3" pad="3"/>
@@
 <contactref element="R83" pad="1"/>
 <contactref element="L1" pad="1"/>
-<wire x1="362.75" y1="4.445" x2="364.655" y2="6.35" width="0" layer="19" extent="1-1"/>
+<contactref element="R108" pad="2"/>
+<wire x1="259.275" y1="38.1" x2="-69.05" y2="-50.165" width="0" layer="19" extent="1-1"/>
+<wire x1="351.9145" y1="7.945" x2="259.275" y2="38.1" width="0" layer="19" extent="1-1"/>
+<wire x1="353.3395" y1="10.67" x2="351.9145" y2="7.945" width="0" layer="19" extent="1-1"/>
+<wire x1="353.9895" y1="10.67" x2="353.3395" y2="10.67" width="0" layer="19" extent="1-1"/>
+<wire x1="354.6395" y1="10.67" x2="353.9895" y2="10.67" width="0" layer="19" extent="1-1"/>
+<wire x1="355.2895" y1="10.67" x2="354.6395" y2="10.67" width="0" layer="19" extent="1-1"/>
+<wire x1="358.0145" y1="6.645" x2="355.2895" y2="10.67" width="0" layer="19" extent="1-1"/>
+<wire x1="362.75" y1="4.445" x2="358.0145" y2="6.645" width="0" layer="19" extent="1-1"/>
+<wire x1="364.655" y1="6.35" x2="362.75" y2="4.445" width="0" layer="19" extent="1-1"/>
 <wire x1="361.781" y1="1.906" x2="362.75" y2="4.445" width="0" layer="19" extent="1-1"/>
-<wire x1="361.48" y1="6.985" x2="362.75" y2="4.445" width="0" layer="19" extent="1-1"/>
-<wire x1="358.0145" y1="6.645" x2="361.48" y2="6.985" width="0" layer="19" extent="1-1"/>
-<wire x1="355.2895" y1="10.67" x2="358.0145" y2="6.645" width="0" layer="19" extent="1-1"/>
-<wire x1="354.6395" y1="10.67" x2="355.2895" y2="10.67" width="0" layer="19" extent="1-1"/>
-<wire x1="353.9895" y1="10.67" x2="354.6395" y2="10.67" width="0" layer="19" extent="1-1"/>
-<wire x1="353.3395" y1="10.67" x2="353.9895" y2="10.67" width="0" layer="19" extent="1-1"/>
-<wire x1="351.9145" y1="7.945" x2="353.3395" y2="10.67" width="0" layer="19" extent="1-1"/>
-<wire x1="259.275" y1="38.1" x2="351.9145" y2="7.945" width="0" layer="19" extent="1-1"/>
 </signal>
 <signal name="N$24">
@@
 <wire x1="350.052" y1="4.447" x2="355.9395" y2="4.57" width="0" layer="19" extent="1-1"/>
 </signal>
-<signal name="N$29">
-<contactref element="IC3" pad="9"/>
-<contactref element="IC3" pad="10"/>
-<contactref element="IC3" pad="11"/>
-<contactref element="IC3" pad="5"/>
-<contactref element="IC3" pad="6"/>
-<contactref element="IC3" pad="7"/>
-<contactref element="IC3" pad="8"/>
-<contactref element="R79" pad="1"/>
-<wire x1="367.03" y1="0.635" x2="272.415" y2="0.635" width="0.254" layer="16"/>
-<contactref element="C80" pad="2"/>
-<contactref element="C64" pad="2"/>
-<contactref element="C63" pad="2"/>
-<wire x1="356.5895" y1="10.67" x2="357.2395" y2="10.67" width="0" layer="19" extent="1-1"/>
-<wire x1="355.9395" y1="10.67" x2="356.5895" y2="10.67" width="0" layer="19" extent="1-1"/>
-<wire x1="358.0145" y1="9.895" x2="357.2395" y2="10.67" width="0" layer="19" extent="1-1"/>
-<wire x1="358.0145" y1="9.245" x2="358.0145" y2="9.895" width="0" layer="19" extent="1-1"/>
-<wire x1="358.0145" y1="8.595" x2="358.0145" y2="9.245" width="0" layer="19" extent="1-1"/>
-<wire x1="358.0145" y1="7.945" x2="358.0145" y2="8.595" width="0" layer="19" extent="1-1"/>
-<wire x1="360.21" y1="3.175" x2="358.0145" y2="7.945" width="0" layer="19" extent="1-1"/>
-<wire x1="367.03" y1="0.635" x2="360.21" y2="3.175" width="0" layer="19" extent="1-16"/>
-<wire x1="28.98" y1="8.89" x2="272.415" y2="0.635" width="0" layer="19" extent="1-16"/>
-<wire x1="21.995" y1="10.795" x2="28.98" y2="8.89" width="0" layer="19" extent="1-16"/>
-<wire x1="19.685" y1="10.96" x2="21.995" y2="10.795" width="0" layer="19" extent="1-16"/>
-</signal>
 <signal name="CELL12+">
 <contactref element="CELL12+" pad="P$1"/>
@@
 <wire x1="-25.87" y1="-32.385" x2="-33.02" y2="-39.98" width="0" layer="19" extent="1-1"/>
 </signal>
+<signal name="N$13">
+<contactref element="C65" pad="2"/>
+<contactref element="R108" pad="1"/>
+<wire x1="361.48" y1="6.985" x2="-70.65" y2="-50.165" width="0" layer="19" extent="1-1"/>
+</signal>
 </signals>
