File: BMS_hw/AFE_PCB/BMSV1.0.sch (EAGLE design)
At the start: 238 parts, among them IC1 MC33771BEP, IC2 SFH6156, IC3 MIC28515V1, IC4 FOD8384-COC, IC5 FOD8384-COC, IC6 FOD8384-COC, J2 NTC, Q1 IRLML5203, Q2 IRLML5203, T1 IPT020N10N3V1, T2 IPT020N10N3V1, T3 IPT020N10N3V1, T4 IPT020N10N3V1, X1 87758-2016, X2 87758-1816, X3 22-23-2041, X4 87758-2016, X5 22-23-2051

Commit message: added BOM and DCDC datasheet updated dcdc shematic
Parts:
- added R68: 0R, ipc-7351-resistor:RESISTOR_0603
- C17: value 47nF -> .1uF 100v; device ipc-7351-capacitor:CAPACITOR_0402 -> ipc-7351-capacitor:CAPACITOR_0603
- C24: value 47nF -> .1u 100v
- C26: value 47nF -> 1uF 100v; device ipc-7351-capacitor:CAPACITOR_0402 -> ipc-7351-capacitor:CAPACITOR_0603
- R12, R15, R22, R23: device ipc-7351-resistor:RESISTOR_0402 -> ipc-7351-resistor:RESISTOR_0603
- R16, R24: value 127E -> 1.6k; device ipc-7351-resistor:RESISTOR_0402 -> ipc-7351-resistor:RESISTOR_0603
- R21: value 127E -> 16.2k; device ipc-7351-resistor:RESISTOR_0402 -> ipc-7351-resistor:RESISTOR_0603
- R25: value 127E -> 2R; device ipc-7351-resistor:RESISTOR_0402 -> ipc-7351-resistor:RESISTOR_0603
Connections:
- new net N$10: C24.2, R68.2
- net SW: now also R68.1; no longer C24.2
Other:
- moved on the sheet: C24
Changed lines of the file:
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@@
 <part name="GND24" library="supply1" library_urn="urn:adsk.eagle:library:371" deviceset="GND" device=""/>
 <part name="R11" library="ipc-7351-resistor" deviceset="RESISTOR_" device="0402" value="2E2"/>
-<part name="R12" library="ipc-7351-resistor" deviceset="RESISTOR_" device="0402" value="200k"/>
-<part name="R15" library="ipc-7351-resistor" deviceset="RESISTOR_" device="0402" value="100k"/>
+<part name="R12" library="ipc-7351-resistor" deviceset="RESISTOR_" device="0603" value="200k"/>
+<part name="R15" library="ipc-7351-resistor" deviceset="RESISTOR_" device="0603" value="100k"/>
 <part name="SUPPLY2" library="supply2" library_urn="urn:adsk.eagle:library:372" deviceset="GND" device=""/>
-<part name="R16" library="ipc-7351-resistor" deviceset="RESISTOR_" device="0402" value="127E"/>
+<part name="R16" library="ipc-7351-resistor" deviceset="RESISTOR_" device="0603" value="1.6k"/>
 <part name="C16" library="ipc-7351-capacitor" deviceset="CAPACITOR_" device="0402" value="1uF"/>
 <part name="GND25" library="supply1" library_urn="urn:adsk.eagle:library:371" deviceset="GND" device=""/>
 <part name="L1" library="GreenFuel" deviceset="XAL1010" device="-822MEB"/>
-<part name="R21" library="ipc-7351-resistor" deviceset="RESISTOR_" device="0402" value="127E"/>
-<part name="C17" library="ipc-7351-capacitor" deviceset="CAPACITOR_" device="0402" value="47nF"/>
-<part name="R22" library="ipc-7351-resistor" deviceset="RESISTOR_" device="0402" value="127E"/>
-<part name="R23" library="ipc-7351-resistor" deviceset="RESISTOR_" device="0402" value="127E"/>
+<part name="R21" library="ipc-7351-resistor" deviceset="RESISTOR_" device="0603" value="16.2k"/>
+<part name="C17" library="ipc-7351-capacitor" deviceset="CAPACITOR_" device="0603" value=".1uF 100v"/>
+<part name="R22" library="ipc-7351-resistor" deviceset="RESISTOR_" device="0603" value="127E"/>
+<part name="R23" library="ipc-7351-resistor" deviceset="RESISTOR_" device="0603" value="127E"/>
 <part name="C22" library="ipc-7351-capacitor" deviceset="CAPACITOR_" device="0603" value="47nF"/>
 <part name="C23" library="ipc-7351-capacitor" deviceset="CAPACITOR_" device="1210" value="47nF"/>
@@
 <part name="GND26" library="supply1" library_urn="urn:adsk.eagle:library:371" deviceset="GND" device=""/>
 <part name="SUPPLY5" library="supply2" library_urn="urn:adsk.eagle:library:372" deviceset="GND" device=""/>
-<part name="R24" library="ipc-7351-resistor" deviceset="RESISTOR_" device="0402" value="127E"/>
-<part name="C24" library="ipc-7351-capacitor" deviceset="CAPACITOR_" device="0402" value="47nF"/>
+<part name="R24" library="ipc-7351-resistor" deviceset="RESISTOR_" device="0603" value="1.6k"/>
+<part name="C24" library="ipc-7351-capacitor" deviceset="CAPACITOR_" device="0402" value=".1u 100v"/>
 <part name="VCC" library="supply1" library_urn="urn:adsk.eagle:library:371" deviceset="VCC" device="" value="+15v"/>
 <part name="C25" library="ipc-7351-capacitor" deviceset="CAPACITOR_" device="1210" value="47nF"/>
 <part name="GND30" library="supply1" library_urn="urn:adsk.eagle:library:371" deviceset="GND" device=""/>
-<part name="C26" library="ipc-7351-capacitor" deviceset="CAPACITOR_" device="0402" value="47nF"/>
+<part name="C26" library="ipc-7351-capacitor" deviceset="CAPACITOR_" device="0603" value="1uF 100v"/>
 <part name="GND31" library="supply1" library_urn="urn:adsk.eagle:library:371" deviceset="GND" device=""/>
-<part name="R25" library="ipc-7351-resistor" deviceset="RESISTOR_" device="0402" value="127E"/>
+<part name="R25" library="ipc-7351-resistor" deviceset="RESISTOR_" device="0603" value="2R"/>
 <part name="SUPPLY6" library="supply2" library_urn="urn:adsk.eagle:library:372" deviceset="GND" device=""/>
 <part name="GND32" library="supply1" library_urn="urn:adsk.eagle:library:371" deviceset="GND" device=""/>
@@
 <part name="C38" library="ipc-7351-capacitor" deviceset="POLARISED_" device="CASE_E"/>
 <part name="GND40" library="supply1" library_urn="urn:adsk.eagle:library:371" deviceset="GND" device=""/>
+<part name="R68" library="ipc-7351-resistor" deviceset="RESISTOR_" device="0603" value="0R"/>
 </parts>
 <sheets>
@@
 <attribute name="VALUE" x="266.7" y="85.598" size="1.778" layer="96"/>
 </instance>
-<instance part="C24" gate="G$1" x="274.32" y="104.14" rot="R270">
-<attribute name="NAME" x="276.86" y="106.68" size="1.778" layer="95" rot="R270"/>
-<attribute name="VALUE" x="270.002" y="106.68" size="1.778" layer="96" rot="R270"/>
+<instance part="C24" gate="G$1" x="264.16" y="109.22">
+<attribute name="NAME" x="261.62" y="111.76" size="1.778" layer="95"/>
+<attribute name="VALUE" x="261.62" y="104.902" size="1.778" layer="96"/>
 </instance>
 <instance part="VCC" gate="VCC" x="325.12" y="99.06">
@@
 <attribute name="VALUE" x="251.46" y="114.3" size="1.778" layer="96"/>
 </instance>
+<instance part="R68" gate="G$1" x="274.32" y="101.6" rot="R90">
+<attribute name="NAME" x="272.796" y="99.06" size="1.778" layer="95" rot="R90"/>
+<attribute name="VALUE" x="277.622" y="99.06" size="1.778" layer="96" rot="R90"/>
+</instance>
 </instances>
 <busses>
@@
 <wire x1="274.32" y1="93.98" x2="281.94" y2="93.98" width="0.1524" layer="91"/>
 <junction x="281.94" y="93.98"/>
-<pinref part="C24" gate="G$1" pin="2"/>
-<wire x1="274.32" y1="99.06" x2="274.32" y2="93.98" width="0.1524" layer="91"/>
 <junction x="274.32" y="93.98"/>
 <wire x1="274.32" y1="93.98" x2="269.24" y2="93.98" width="0.1524" layer="91"/>
 <label x="269.24" y="93.98" size="1.778" layer="95"/>
+<pinref part="R68" gate="G$1" pin="1"/>
+<wire x1="274.32" y1="96.52" x2="274.32" y2="93.98" width="0.1524" layer="91"/>
 </segment>
 <segment>
@@
 <segment>
 <pinref part="C24" gate="G$1" pin="1"/>
-<wire x1="274.32" y1="109.22" x2="266.7" y2="109.22" width="0.1524" layer="91"/>
-<label x="266.7" y="109.22" size="1.778" layer="95"/>
+<wire x1="259.08" y1="109.22" x2="251.46" y2="109.22" width="0.1524" layer="91"/>
+<label x="251.46" y="109.22" size="1.778" layer="95"/>
 </segment>
 <segment>
@@
 </segment>
 </net>
+<net name="N$10" class="0">
+<segment>
+<pinref part="C24" gate="G$1" pin="2"/>
+<pinref part="R68" gate="G$1" pin="2"/>
+<wire x1="269.24" y1="109.22" x2="274.32" y2="109.22" width="0.1524" layer="91"/>
+<wire x1="274.32" y1="109.22" x2="274.32" y2="106.68" width="0.1524" layer="91"/>
+</segment>
+</net>

Commit message: updated sch
Parts:
- removed R68: 0R, ipc-7351-resistor:RESISTOR_0603
- C17: value .1uF 100v -> 47nF; device ipc-7351-capacitor:CAPACITOR_0603 -> ipc-7351-capacitor:CAPACITOR_0402
- C24: value .1u 100v -> 47nF
- C26: value 1uF 100v -> 47nF; device ipc-7351-capacitor:CAPACITOR_0603 -> ipc-7351-capacitor:CAPACITOR_0402
- R12, R15, R22, R23: device ipc-7351-resistor:RESISTOR_0603 -> ipc-7351-resistor:RESISTOR_0402
- R16, R24: value 1.6k -> 127E; device ipc-7351-resistor:RESISTOR_0603 -> ipc-7351-resistor:RESISTOR_0402
- R21: value 16.2k -> 127E; device ipc-7351-resistor:RESISTOR_0603 -> ipc-7351-resistor:RESISTOR_0402
- R25: value 2R -> 127E; device ipc-7351-resistor:RESISTOR_0603 -> ipc-7351-resistor:RESISTOR_0402
Connections:
- net N$67 renamed V+
- removed net N$10: C24.2, R68.2
- removed net N$23: D1.K, D2.K, R30.2, R38.1, T1.G
- removed net N$61: R29.1, T3.S, T3.S1, T3.S2, T3.S3, T3.S4, T3.S5, T3.S6, T4.S, T4.S1, T4.S2, T4.S3, T4.S4, T4.S5, T4.S6
- net CHG_GATE: now also D1.K, D2.K, R30.2, R38.1, T1.G
- net SW: now also C24.2; no longer R68.1
- net V-: now also R29.1, T3.S, T3.S1, T3.S2, T3.S3, T3.S4, T3.S5, T3.S6, T4.S, T4.S1, T4.S2, T4.S3, T4.S4, T4.S5, T4.S6
Other:
- moved on the sheet: C24
Changed lines of the file:
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@@
 <part name="GND24" library="supply1" library_urn="urn:adsk.eagle:library:371" deviceset="GND" device=""/>
 <part name="R11" library="ipc-7351-resistor" deviceset="RESISTOR_" device="0402" value="2E2"/>
-<part name="R12" library="ipc-7351-resistor" deviceset="RESISTOR_" device="0603" value="200k"/>
-<part name="R15" library="ipc-7351-resistor" deviceset="RESISTOR_" device="0603" value="100k"/>
+<part name="R12" library="ipc-7351-resistor" deviceset="RESISTOR_" device="0402" value="200k"/>
+<part name="R15" library="ipc-7351-resistor" deviceset="RESISTOR_" device="0402" value="100k"/>
 <part name="SUPPLY2" library="supply2" library_urn="urn:adsk.eagle:library:372" deviceset="GND" device=""/>
-<part name="R16" library="ipc-7351-resistor" deviceset="RESISTOR_" device="0603" value="1.6k"/>
+<part name="R16" library="ipc-7351-resistor" deviceset="RESISTOR_" device="0402" value="127E"/>
 <part name="C16" library="ipc-7351-capacitor" deviceset="CAPACITOR_" device="0402" value="1uF"/>
 <part name="GND25" library="supply1" library_urn="urn:adsk.eagle:library:371" deviceset="GND" device=""/>
 <part name="L1" library="GreenFuel" deviceset="XAL1010" device="-822MEB"/>
-<part name="R21" library="ipc-7351-resistor" deviceset="RESISTOR_" device="0603" value="16.2k"/>
-<part name="C17" library="ipc-7351-capacitor" deviceset="CAPACITOR_" device="0603" value=".1uF 100v"/>
-<part name="R22" library="ipc-7351-resistor" deviceset="RESISTOR_" device="0603" value="127E"/>
-<part name="R23" library="ipc-7351-resistor" deviceset="RESISTOR_" device="0603" value="127E"/>
+<part name="R21" library="ipc-7351-resistor" deviceset="RESISTOR_" device="0402" value="127E"/>
+<part name="C17" library="ipc-7351-capacitor" deviceset="CAPACITOR_" device="0402" value="47nF"/>
+<part name="R22" library="ipc-7351-resistor" deviceset="RESISTOR_" device="0402" value="127E"/>
+<part name="R23" library="ipc-7351-resistor" deviceset="RESISTOR_" device="0402" value="127E"/>
 <part name="C22" library="ipc-7351-capacitor" deviceset="CAPACITOR_" device="0603" value="47nF"/>
 <part name="C23" library="ipc-7351-capacitor" deviceset="CAPACITOR_" device="1210" value="47nF"/>
@@
 <part name="GND26" library="supply1" library_urn="urn:adsk.eagle:library:371" deviceset="GND" device=""/>
 <part name="SUPPLY5" library="supply2" library_urn="urn:adsk.eagle:library:372" deviceset="GND" device=""/>
-<part name="R24" library="ipc-7351-resistor" deviceset="RESISTOR_" device="0603" value="1.6k"/>
-<part name="C24" library="ipc-7351-capacitor" deviceset="CAPACITOR_" device="0402" value=".1u 100v"/>
+<part name="R24" library="ipc-7351-resistor" deviceset="RESISTOR_" device="0402" value="127E"/>
+<part name="C24" library="ipc-7351-capacitor" deviceset="CAPACITOR_" device="0402" value="47nF"/>
 <part name="VCC" library="supply1" library_urn="urn:adsk.eagle:library:371" deviceset="VCC" device="" value="+15v"/>
 <part name="C25" library="ipc-7351-capacitor" deviceset="CAPACITOR_" device="1210" value="47nF"/>
 <part name="GND30" library="supply1" library_urn="urn:adsk.eagle:library:371" deviceset="GND" device=""/>
-<part name="C26" library="ipc-7351-capacitor" deviceset="CAPACITOR_" device="0603" value="1uF 100v"/>
+<part name="C26" library="ipc-7351-capacitor" deviceset="CAPACITOR_" device="0402" value="47nF"/>
 <part name="GND31" library="supply1" library_urn="urn:adsk.eagle:library:371" deviceset="GND" device=""/>
-<part name="R25" library="ipc-7351-resistor" deviceset="RESISTOR_" device="0603" value="2R"/>
+<part name="R25" library="ipc-7351-resistor" deviceset="RESISTOR_" device="0402" value="127E"/>
 <part name="SUPPLY6" library="supply2" library_urn="urn:adsk.eagle:library:372" deviceset="GND" device=""/>
 <part name="GND32" library="supply1" library_urn="urn:adsk.eagle:library:371" deviceset="GND" device=""/>
@@
 <part name="C38" library="ipc-7351-capacitor" deviceset="POLARISED_" device="CASE_E"/>
 <part name="GND40" library="supply1" library_urn="urn:adsk.eagle:library:371" deviceset="GND" device=""/>
-<part name="R68" library="ipc-7351-resistor" deviceset="RESISTOR_" device="0603" value="0R"/>
 </parts>
 <sheets>
@@
 <attribute name="VALUE" x="266.7" y="85.598" size="1.778" layer="96"/>
 </instance>
-<instance part="C24" gate="G$1" x="264.16" y="109.22">
-<attribute name="NAME" x="261.62" y="111.76" size="1.778" layer="95"/>
-<attribute name="VALUE" x="261.62" y="104.902" size="1.778" layer="96"/>
+<instance part="C24" gate="G$1" x="274.32" y="104.14" rot="R270">
+<attribute name="NAME" x="276.86" y="106.68" size="1.778" layer="95" rot="R270"/>
+<attribute name="VALUE" x="270.002" y="106.68" size="1.778" layer="96" rot="R270"/>
 </instance>
 <instance part="VCC" gate="VCC" x="325.12" y="99.06">
@@
 <attribute name="VALUE" x="251.46" y="114.3" size="1.778" layer="96"/>
 </instance>
-<instance part="R68" gate="G$1" x="274.32" y="101.6" rot="R90">
-<attribute name="NAME" x="272.796" y="99.06" size="1.778" layer="95" rot="R90"/>
-<attribute name="VALUE" x="277.622" y="99.06" size="1.778" layer="96" rot="R90"/>
-</instance>
 </instances>
 <busses>
@@
 <wire x1="274.32" y1="93.98" x2="281.94" y2="93.98" width="0.1524" layer="91"/>
 <junction x="281.94" y="93.98"/>
+<pinref part="C24" gate="G$1" pin="2"/>
+<wire x1="274.32" y1="99.06" x2="274.32" y2="93.98" width="0.1524" layer="91"/>
 <junction x="274.32" y="93.98"/>
 <wire x1="274.32" y1="93.98" x2="269.24" y2="93.98" width="0.1524" layer="91"/>
 <label x="269.24" y="93.98" size="1.778" layer="95"/>
-<pinref part="R68" gate="G$1" pin="1"/>
-<wire x1="274.32" y1="96.52" x2="274.32" y2="93.98" width="0.1524" layer="91"/>
 </segment>
 <segment>
@@
 <segment>
 <pinref part="C24" gate="G$1" pin="1"/>
-<wire x1="259.08" y1="109.22" x2="251.46" y2="109.22" width="0.1524" layer="91"/>
-<label x="251.46" y="109.22" size="1.778" layer="95"/>
+<wire x1="274.32" y1="109.22" x2="266.7" y2="109.22" width="0.1524" layer="91"/>
+<label x="266.7" y="109.22" size="1.778" layer="95"/>
 </segment>
 <segment>
@@
 </segment>
 </net>
-<net name="N$10" class="0">
-<segment>
-<pinref part="C24" gate="G$1" pin="2"/>
-<pinref part="R68" gate="G$1" pin="2"/>
-<wire x1="269.24" y1="109.22" x2="274.32" y2="109.22" width="0.1524" layer="91"/>
-<wire x1="274.32" y1="109.22" x2="274.32" y2="106.68" width="0.1524" layer="91"/>
-</segment>
-</net>
 </nets>
 </sheet>
@@
 </segment>
 </net>
-<net name="N$61" class="0">
+<net name="V-" class="0">
 <segment>
 <wire x1="30.48" y1="198.12" x2="27.94" y2="198.12" width="0.1524" layer="91"/>
@@
 </segment>
 </net>
-<net name="N$67" class="0">
+<net name="V+" class="0">
 <segment>
 <wire x1="83.82" y1="182.88" x2="86.36" y2="182.88" width="0.1524" layer="91"/>
@@
 <label x="165.1" y="228.6" size="1.778" layer="95"/>
 </segment>
+<segment>
+<pinref part="R38" gate="G$1" pin="1"/>
+<wire x1="78.74" y1="152.4" x2="81.28" y2="152.4" width="0.1524" layer="91"/>
+<wire x1="81.28" y1="152.4" x2="81.28" y2="162.56" width="0.1524" layer="91"/>
+<pinref part="D2" gate="G$1" pin="K"/>
+<wire x1="76.2" y1="162.56" x2="81.28" y2="162.56" width="0.1524" layer="91"/>
+<wire x1="81.28" y1="175.768" x2="81.28" y2="175.26" width="0.1524" layer="91"/>
+<pinref part="D1" gate="G$1" pin="K"/>
+<wire x1="81.28" y1="175.26" x2="81.28" y2="167.64" width="0.1524" layer="91"/>
+<wire x1="91.44" y1="167.64" x2="81.28" y2="167.64" width="0.1524" layer="91"/>
+<pinref part="R30" gate="G$1" pin="2"/>
+<wire x1="88.9" y1="175.26" x2="81.28" y2="175.26" width="0.1524" layer="91"/>
+<junction x="81.28" y="175.26"/>
+<wire x1="81.28" y1="162.56" x2="81.28" y2="167.64" width="0.1524" layer="91"/>
+<junction x="81.28" y="162.56"/>
+<junction x="81.28" y="167.64"/>
+<pinref part="T1" gate="G$1" pin="G"/>
+<label x="81.28" y="175.26" size="1.778" layer="95" rot="R180"/>
+</segment>
 </net>
 <net name="DSG_GATE" class="0">
@@
 </segment>
 </net>
-<net name="N$23" class="0">
-<segment>
-<pinref part="R38" gate="G$1" pin="1"/>
-<wire x1="78.74" y1="152.4" x2="81.28" y2="152.4" width="0.1524" layer="91"/>
-<wire x1="81.28" y1="152.4" x2="81.28" y2="162.56" width="0.1524" layer="91"/>
-<pinref part="D2" gate="G$1" pin="K"/>
-<wire x1="76.2" y1="162.56" x2="81.28" y2="162.56" width="0.1524" layer="91"/>
-<wire x1="81.28" y1="175.768" x2="81.28" y2="175.26" width="0.1524" layer="91"/>
-<pinref part="D1" gate="G$1" pin="K"/>
-<wire x1="81.28" y1="175.26" x2="81.28" y2="167.64" width="0.1524" layer="91"/>
-<wire x1="91.44" y1="167.64" x2="81.28" y2="167.64" width="0.1524" layer="91"/>
-<pinref part="R30" gate="G$1" pin="2"/>
-<wire x1="88.9" y1="175.26" x2="81.28" y2="175.26" width="0.1524" layer="91"/>
-<junction x="81.28" y="175.26"/>
-<wire x1="81.28" y1="162.56" x2="81.28" y2="167.64" width="0.1524" layer="91"/>
-<junction x="81.28" y="162.56"/>
-<junction x="81.28" y="167.64"/>
-<pinref part="T1" gate="G$1" pin="G"/>
-</segment>
-</net>
 <net name="CHG_FET" class="0">
 <segment>
@@
 <wire x1="279.4" y1="170.18" x2="279.4" y2="172.72" width="0.1524" layer="91"/>
 <wire x1="279.4" y1="172.72" x2="287.02" y2="172.72" width="0.1524" layer="91"/>
-<label x="287.02" y="172.72" size="1.778" layer="95"/>
+<label x="299.72" y="172.72" size="1.778" layer="95" rot="R180"/>
 </segment>
 <segment>
