File: BMS_hw/AFE_PCB/BMSV1.0.sch (EAGLE design)
At the start: 242 parts, among them IC1 MC33771BEP, IC2 SFH6156, IC3 MIC28515V1, IC4 FOD8384-COC, IC5 FOD8384-COC, IC6 FOD8384-COC, J1 NTC, Q1 IRLML5203, Q2 IRLML5203, T1 IPT020N10N3V1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

Commit message: itt@6 itt@6
Other:
- moved on the sheet: JP5
Changed lines of the file:
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@@
 <attribute name="VALUE" x="267.462" y="218.44" size="1.778" layer="96" rot="R270"/>
 </instance>
-<instance part="JP5" gate="A" x="365.76" y="215.9">
-<attribute name="NAME" x="359.41" y="236.855" size="1.778" layer="95"/>
-<attribute name="VALUE" x="359.41" y="193.04" size="1.778" layer="96"/>
+<instance part="JP5" gate="A" x="353.06" y="205.74">
+<attribute name="NAME" x="346.71" y="226.695" size="1.778" layer="95"/>
+<attribute name="VALUE" x="346.71" y="182.88" size="1.778" layer="96"/>
 </instance>
 </instances>
@@
 <segment>
 <pinref part="JP5" gate="A" pin="13"/>
-<wire x1="363.22" y1="203.2" x2="347.98" y2="203.2" width="0.1524" layer="91"/>
-<label x="332.74" y="203.2" size="1.778" layer="95"/>
+<wire x1="350.52" y1="193.04" x2="332.74" y2="193.04" width="0.1524" layer="91"/>
+<label x="317.5" y="193.04" size="1.778" layer="95"/>
 </segment>
 </net>
@@
 <segment>
 <pinref part="JP5" gate="A" pin="12"/>
-<wire x1="363.22" y1="205.74" x2="347.98" y2="205.74" width="0.1524" layer="91"/>
-<label x="332.74" y="205.74" size="1.778" layer="95"/>
+<wire x1="350.52" y1="195.58" x2="332.74" y2="195.58" width="0.1524" layer="91"/>
+<label x="317.5" y="195.58" size="1.778" layer="95"/>
 </segment>
 </net>
@@
 <segment>
 <pinref part="JP5" gate="A" pin="11"/>
-<wire x1="363.22" y1="208.28" x2="347.98" y2="208.28" width="0.1524" layer="91"/>
-<label x="332.74" y="208.28" size="1.778" layer="95"/>
+<wire x1="350.52" y1="198.12" x2="332.74" y2="198.12" width="0.1524" layer="91"/>
+<label x="317.5" y="198.12" size="1.778" layer="95"/>
 </segment>
 </net>
@@
 <segment>
 <pinref part="JP5" gate="A" pin="15"/>
-<wire x1="363.22" y1="198.12" x2="347.98" y2="198.12" width="0.1524" layer="91"/>
-<label x="332.74" y="198.12" size="1.778" layer="95"/>
+<wire x1="350.52" y1="187.96" x2="332.74" y2="187.96" width="0.1524" layer="91"/>
+<label x="317.5" y="187.96" size="1.778" layer="95"/>
 </segment>
 </net>
@@
 <segment>
 <pinref part="JP5" gate="A" pin="7"/>
-<wire x1="363.22" y1="218.44" x2="347.98" y2="218.44" width="0.1524" layer="91"/>
-<label x="332.74" y="218.44" size="1.778" layer="95"/>
+<wire x1="350.52" y1="208.28" x2="332.74" y2="208.28" width="0.1524" layer="91"/>
+<label x="317.5" y="208.28" size="1.778" layer="95"/>
 </segment>
 </net>
@@
 <segment>
 <pinref part="JP5" gate="A" pin="5"/>
-<wire x1="363.22" y1="223.52" x2="347.98" y2="223.52" width="0.1524" layer="91"/>
-<label x="332.74" y="223.52" size="1.778" layer="95"/>
+<wire x1="350.52" y1="213.36" x2="332.74" y2="213.36" width="0.1524" layer="91"/>
+<label x="317.5" y="213.36" size="1.778" layer="95"/>
 </segment>
 </net>
@@
 <segment>
 <pinref part="JP5" gate="A" pin="9"/>
-<wire x1="363.22" y1="213.36" x2="347.98" y2="213.36" width="0.1524" layer="91"/>
-<label x="332.74" y="213.36" size="1.778" layer="95"/>
+<wire x1="350.52" y1="203.2" x2="332.74" y2="203.2" width="0.1524" layer="91"/>
+<label x="317.5" y="203.2" size="1.778" layer="95"/>
 </segment>
 </net>
@@
 <segment>
 <pinref part="JP5" gate="A" pin="3"/>
-<wire x1="363.22" y1="228.6" x2="347.98" y2="228.6" width="0.1524" layer="91"/>
-<label x="337.82" y="228.6" size="1.778" layer="95"/>
+<wire x1="350.52" y1="218.44" x2="332.74" y2="218.44" width="0.1524" layer="91"/>
+<label x="322.58" y="218.44" size="1.778" layer="95"/>
 </segment>
 </net>
@@
 <segment>
 <pinref part="JP5" gate="A" pin="2"/>
-<wire x1="363.22" y1="231.14" x2="347.98" y2="231.14" width="0.1524" layer="91"/>
-<label x="337.82" y="231.14" size="1.778" layer="95"/>
+<wire x1="350.52" y1="220.98" x2="332.74" y2="220.98" width="0.1524" layer="91"/>
+<label x="322.58" y="220.98" size="1.778" layer="95"/>
 </segment>
 </net>
@@
 <segment>
 <pinref part="JP5" gate="A" pin="1"/>
-<wire x1="363.22" y1="233.68" x2="347.98" y2="233.68" width="0.1524" layer="91"/>
-<label x="340.36" y="233.68" size="1.778" layer="95"/>
+<wire x1="350.52" y1="223.52" x2="332.74" y2="223.52" width="0.1524" layer="91"/>
+<label x="325.12" y="223.52" size="1.778" layer="95"/>
 </segment>
 </net>
@@
 <segment>
 <pinref part="JP5" gate="A" pin="14"/>
-<wire x1="363.22" y1="200.66" x2="347.98" y2="200.66" width="0.1524" layer="91"/>
-<label x="332.74" y="200.66" size="1.778" layer="95"/>
+<wire x1="350.52" y1="190.5" x2="332.74" y2="190.5" width="0.1524" layer="91"/>
+<label x="317.5" y="190.5" size="1.778" layer="95"/>
 </segment>
 </net>
@@
 <segment>
 <pinref part="JP5" gate="A" pin="4"/>
-<wire x1="363.22" y1="226.06" x2="347.98" y2="226.06" width="0.1524" layer="91"/>
-<label x="337.82" y="226.06" size="1.778" layer="95"/>
+<wire x1="350.52" y1="215.9" x2="332.74" y2="215.9" width="0.1524" layer="91"/>
+<label x="322.58" y="215.9" size="1.778" layer="95"/>
 </segment>
 </net>
@@
 <segment>
 <pinref part="JP5" gate="A" pin="6"/>
-<wire x1="363.22" y1="220.98" x2="347.98" y2="220.98" width="0.1524" layer="91"/>
-<label x="335.28" y="220.98" size="1.778" layer="95"/>
+<wire x1="350.52" y1="210.82" x2="332.74" y2="210.82" width="0.1524" layer="91"/>
+<label x="320.04" y="210.82" size="1.778" layer="95"/>
 </segment>
 </net>
@@
 <segment>
 <pinref part="JP5" gate="A" pin="8"/>
-<wire x1="363.22" y1="215.9" x2="347.98" y2="215.9" width="0.1524" layer="91"/>
-<label x="337.82" y="215.9" size="1.778" layer="95"/>
+<wire x1="350.52" y1="205.74" x2="332.74" y2="205.74" width="0.1524" layer="91"/>
+<label x="322.58" y="205.74" size="1.778" layer="95"/>
 </segment>
 <segment>
@@
 <segment>
 <pinref part="JP5" gate="A" pin="10"/>
-<wire x1="363.22" y1="210.82" x2="347.98" y2="210.82" width="0.1524" layer="91"/>
-<label x="332.74" y="210.82" size="1.778" layer="95"/>
-</segment>
-<segment>
+<wire x1="350.52" y1="200.66" x2="332.74" y2="200.66" width="0.1524" layer="91"/>
+<label x="317.5" y="200.66" size="1.778" layer="95"/>
+</segment>
+<segment>

Commit message: itt@7
Connections:
- removed net CB_13/12_C2: JP5.15
- removed net CB_14/13C: IC1.CB_14:13C
- net CB_10/9_C: now also JP5.10; no longer JP5.9
- net CB_11/10_C: now also JP5.11; no longer JP5.10
- net CB_12/11_C: now also JP5.12; no longer JP5.11
- net CB_13/12_C: now also JP5.13; no longer JP5.12
- net CB_14+/14_C: now also JP5.15; no longer JP5.14
- net CB_14/13_C: now also IC1.CB_14:13C, JP5.14; no longer JP5.13
- net CB_3/2_C: now also JP5.3
- net CB_4/3_C: now also JP5.4; no longer JP5.3
- net CB_5/4_C: now also JP5.5; no longer JP5.4
- net CB_6/5_C: now also JP5.6; no longer JP5.5
- net CB_7/6_C: now also JP5.7; no longer JP5.6
- net CB_8/7_C: now also JP5.8; no longer JP5.7
- net CB_9/8_C: now also JP5.9; no longer JP5.8
Changed lines of the file:
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@@
 </segment>
 <segment>
-<pinref part="JP5" gate="A" pin="13"/>
-<wire x1="350.52" y1="193.04" x2="332.74" y2="193.04" width="0.1524" layer="91"/>
-<label x="317.5" y="193.04" size="1.778" layer="95"/>
+<pinref part="JP5" gate="A" pin="14"/>
+<wire x1="350.52" y1="190.5" x2="332.74" y2="190.5" width="0.1524" layer="91"/>
+<label x="317.5" y="190.5" size="1.778" layer="95"/>
+</segment>
+<segment>
+<pinref part="IC1" gate="G$1" pin="CB_14:13C"/>
+<wire x1="177.8" y1="208.28" x2="175.26" y2="208.28" width="0.1524" layer="91"/>
+<label x="175.26" y="209.296" size="1.778" layer="95" rot="R180"/>
 </segment>
 </net>
@@
 </segment>
 <segment>
-<pinref part="JP5" gate="A" pin="12"/>
-<wire x1="350.52" y1="195.58" x2="332.74" y2="195.58" width="0.1524" layer="91"/>
-<label x="317.5" y="195.58" size="1.778" layer="95"/>
+<pinref part="JP5" gate="A" pin="13"/>
+<wire x1="350.52" y1="193.04" x2="332.74" y2="193.04" width="0.1524" layer="91"/>
+<label x="317.5" y="193.04" size="1.778" layer="95"/>
 </segment>
 </net>
@@
 </segment>
 <segment>
-<pinref part="JP5" gate="A" pin="11"/>
-<wire x1="350.52" y1="198.12" x2="332.74" y2="198.12" width="0.1524" layer="91"/>
-<label x="317.5" y="198.12" size="1.778" layer="95"/>
+<pinref part="JP5" gate="A" pin="12"/>
+<wire x1="350.52" y1="195.58" x2="332.74" y2="195.58" width="0.1524" layer="91"/>
+<label x="317.5" y="195.58" size="1.778" layer="95"/>
 </segment>
 </net>
@@
 </segment>
 </net>
-<net name="CB_13/12_C2" class="0">
-<segment>
-<pinref part="JP5" gate="A" pin="15"/>
-<wire x1="350.52" y1="187.96" x2="332.74" y2="187.96" width="0.1524" layer="91"/>
-<label x="317.5" y="187.96" size="1.778" layer="95"/>
-</segment>
-</net>
 <net name="CB_9" class="0">
 <segment>
@@
 </segment>
 <segment>
-<pinref part="JP5" gate="A" pin="7"/>
-<wire x1="350.52" y1="208.28" x2="332.74" y2="208.28" width="0.1524" layer="91"/>
-<label x="317.5" y="208.28" size="1.778" layer="95"/>
+<pinref part="JP5" gate="A" pin="8"/>
+<wire x1="350.52" y1="205.74" x2="332.74" y2="205.74" width="0.1524" layer="91"/>
+<label x="322.58" y="205.74" size="1.778" layer="95"/>
 </segment>
 </net>
@@
 </segment>
 <segment>
-<pinref part="JP5" gate="A" pin="5"/>
-<wire x1="350.52" y1="213.36" x2="332.74" y2="213.36" width="0.1524" layer="91"/>
-<label x="317.5" y="213.36" size="1.778" layer="95"/>
+<pinref part="JP5" gate="A" pin="6"/>
+<wire x1="350.52" y1="210.82" x2="332.74" y2="210.82" width="0.1524" layer="91"/>
+<label x="320.04" y="210.82" size="1.778" layer="95"/>
 </segment>
 </net>
@@
 </segment>
 <segment>
-<pinref part="JP5" gate="A" pin="9"/>
-<wire x1="350.52" y1="203.2" x2="332.74" y2="203.2" width="0.1524" layer="91"/>
-<label x="317.5" y="203.2" size="1.778" layer="95"/>
+<pinref part="JP5" gate="A" pin="10"/>
+<wire x1="350.52" y1="200.66" x2="332.74" y2="200.66" width="0.1524" layer="91"/>
+<label x="317.5" y="200.66" size="1.778" layer="95"/>
 </segment>
 </net>
@@
 </segment>
 <segment>
-<pinref part="JP5" gate="A" pin="3"/>
-<wire x1="350.52" y1="218.44" x2="332.74" y2="218.44" width="0.1524" layer="91"/>
-<label x="322.58" y="218.44" size="1.778" layer="95"/>
+<pinref part="JP5" gate="A" pin="4"/>
+<wire x1="350.52" y1="215.9" x2="332.74" y2="215.9" width="0.1524" layer="91"/>
+<label x="322.58" y="215.9" size="1.778" layer="95"/>
 </segment>
 </net>
@@
 <wire x1="34.82" y1="25.16" x2="34.82" y2="248.18" width="0.1524" layer="91"/>
 <wire x1="134.36" y1="25.16" x2="34.82" y2="25.16" width="0.1524" layer="91"/>
-</segment>
-</net>
-<net name="CB_14/13C" class="0">
-<segment>
-<pinref part="IC1" gate="G$1" pin="CB_14:13C"/>
-<wire x1="177.8" y1="208.28" x2="175.26" y2="208.28" width="0.1524" layer="91"/>
-<label x="175.26" y="209.296" size="1.778" layer="95" rot="R180"/>
 </segment>
 </net>
@@
 </segment>
 <segment>
-<pinref part="JP5" gate="A" pin="14"/>
-<wire x1="350.52" y1="190.5" x2="332.74" y2="190.5" width="0.1524" layer="91"/>
-<label x="317.5" y="190.5" size="1.778" layer="95"/>
-</segment>
-</net>
-<net name="CB_5/4_C" class="0">
-<segment>
-<pinref part="JP5" gate="A" pin="4"/>
-<wire x1="350.52" y1="215.9" x2="332.74" y2="215.9" width="0.1524" layer="91"/>
-<label x="322.58" y="215.9" size="1.778" layer="95"/>
-</segment>
-</net>
-<net name="CB_7/6_C" class="0">
-<segment>
-<pinref part="JP5" gate="A" pin="6"/>
-<wire x1="350.52" y1="210.82" x2="332.74" y2="210.82" width="0.1524" layer="91"/>
-<label x="320.04" y="210.82" size="1.778" layer="95"/>
+<pinref part="JP5" gate="A" pin="15"/>
+<wire x1="350.52" y1="187.96" x2="332.74" y2="187.96" width="0.1524" layer="91"/>
+<label x="317.5" y="187.96" size="1.778" layer="95"/>
 </segment>
 </net>
 <net name="CB_9/8_C" class="0">
-<segment>
-<pinref part="JP5" gate="A" pin="8"/>
-<wire x1="350.52" y1="205.74" x2="332.74" y2="205.74" width="0.1524" layer="91"/>
-<label x="322.58" y="205.74" size="1.778" layer="95"/>
-</segment>
 <segment>
 <pinref part="C2" gate="G$1" pin="1"/>
@@
 <label x="71.12" y="63.5" size="1.778" layer="95"/>
 </segment>
+<segment>
+<pinref part="JP5" gate="A" pin="9"/>
+<wire x1="350.52" y1="203.2" x2="332.74" y2="203.2" width="0.1524" layer="91"/>
+<label x="317.5" y="203.2" size="1.778" layer="95"/>
+</segment>
 </net>
 <net name="CB_11/10_C" class="0">
-<segment>
-<pinref part="JP5" gate="A" pin="10"/>
-<wire x1="350.52" y1="200.66" x2="332.74" y2="200.66" width="0.1524" layer="91"/>
-<label x="317.5" y="200.66" size="1.778" layer="95"/>
-</segment>
 <segment>
 <pinref part="C4" gate="G$1" pin="1"/>
@@
 <label x="73.66" y="116.84" size="1.778" layer="95"/>
 </segment>
-</net>
+<segment>
+<pinref part="JP5" gate="A" pin="11"/>
+<wire x1="350.52" y1="198.12" x2="332.74" y2="198.12" width="0.1524" layer="91"/>
+<label x="317.5" y="198.12" size="1.778" layer="95"/>
+</segment>
+</net>
+<net name="CB_3/2_C" class="0">
+<segment>
+<pinref part="JP5" gate="A" pin="3"/>
+<wire x1="350.52" y1="218.44" x2="332.74" y2="218.44" width="0.1524" layer="91"/>
+<label x="322.58" y="218.44" size="1.778" layer="95"/>
+</segment>
+</net>
+<net name="CB_5/4_C" class="0">
+<segment>
+<pinref part="JP5" gate="A" pin="5"/>
+<wire x1="350.52" y1="213.36" x2="332.74" y2="213.36" width="0.1524" layer="91"/>
+<label x="317.5" y="213.36" size="1.778" layer="95"/>
+</segment>
+</net>
+<net name="CB_7/6_C" class="0">
+<segment>
+<pinref part="JP5" gate="A" pin="7"/>
+<wire x1="350.52" y1="208.28" x2="332.74" y2="208.28" width="0.1524" layer="91"/>
+<label x="317.5" y="208.28" size="1.778" layer="95"/>
+</segment>
+</net>

Commit message: itt@7
Parts:
- removed J1: NTC, con-molex:22-27-2081-08
- added TP2, TP3, TP4, TP5, TP6, TP7, TP8, TP9: TPTH7035, simpa:TPTH7035
- C48, C49, C50, C51, C52, C53, C54: value 2.2uF -> 2200pF
- C55, C56, C57, C58, C59, C60, C62: value 1uF -> 1nF
- R72, R73, R74, R75, R76, R77, R78: value 10k -> 1k
Connections:
- new net CSB: IC1.CSB
- net GND: now also TP8.P$1; no longer J1-1.S
- net N$49: now also TP2.P$1; no longer J1-8.S
- net N$50: now also TP3.P$1; no longer J1-7.S
- net N$51: now also TP4.P$1; no longer J1-6.S
- net N$52: now also TP5.P$1; no longer J1-5.S
- net N$53: now also TP6.P$1; no longer J1-4.S
- net N$54: now also TP7.P$1; no longer J1-3.S
- net N$55: now also TP9.P$1; no longer J1-2.S

Commit message: itt@8
Parts:
- removed TP1: TPTH7035, simpa:TPTH7035
- added BGND, PACK-: (no value), simpa:WPAD
- R31: value 10k -> 127E
Connections:
- net BGND: now also BGND.P$1
- net V+: now also PACK-.P$1
Changed lines of the file:
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@@
 <part name="IC2" library="optocoupler" library_urn="urn:adsk.eagle:library:320" deviceset="SFH6156" device="" package3d_urn="urn:adsk.eagle:package:21969/1"/>
 <part name="GND21" library="supply1" library_urn="urn:adsk.eagle:library:371" deviceset="GND" device=""/>
-<part name="R31" library="ipc-7351-resistor" deviceset="RESISTOR_" device="0402" value="10k"/>
+<part name="R31" library="ipc-7351-resistor" deviceset="RESISTOR_" device="0402" value="127E"/>
 <part name="R29" library="ipc-7351-resistor" deviceset="RESISTOR_" device="0402" value="10k"/>
 <part name="R30" library="ipc-7351-resistor" deviceset="RESISTOR_" device="0402" value="10k"/>
@@
 <part name="GND56" library="supply1" library_urn="urn:adsk.eagle:library:371" deviceset="GND" device=""/>
 <part name="R34" library="ipc-7351-resistor" deviceset="RESISTOR_" device="0402" value="0R"/>
-<part name="TP1" library="simpa" deviceset="TP" device="TH7035"/>
 <part name="D20" library="ipc-7351-diode" deviceset="ZENER_" device="SOD-123" value="8.2V"/>
 <part name="C79" library="ipc-7351-capacitor" deviceset="CAPACITOR_" device="0603" value="0.1uF"/>
@@
 <part name="TP8" library="simpa" deviceset="TP" device="TH7035"/>
 <part name="TP9" library="simpa" deviceset="TP" device="TH7035"/>
+<part name="BGND" library="simpa" deviceset="WPAD" device=""/>
+<part name="PACK-" library="simpa" deviceset="WPAD" device=""/>
 </parts>
 <sheets>
@@
 <attribute name="VALUE" x="259.08" y="198.032" size="1.778" layer="96"/>
 </instance>
-<instance part="TP1" gate="G$1" x="309.88" y="50.8">
-<attribute name="NAME" x="311.15" y="50.165" size="1.016" layer="95" font="vector" ratio="12"/>
-</instance>
 <instance part="C79" gate="G$1" x="271.78" y="215.9" rot="R270">
 <attribute name="NAME" x="274.32" y="218.44" size="1.778" layer="95" rot="R270"/>
@@
 <attribute name="NAME" x="194.31" y="120.015" size="1.016" layer="95" font="vector" ratio="12" rot="R180"/>
 </instance>
+<instance part="BGND" gate="G$1" x="261.62" y="238.76" rot="R180">
+<attribute name="NAME" x="259.08" y="238.76" size="1.778" layer="95" font="vector" ratio="18" rot="R180"/>
+</instance>
 </instances>
 <busses>
@@
 <wire x1="279.4" y1="236.22" x2="279.4" y2="238.76" width="0.1524" layer="91"/>
 <wire x1="279.4" y1="238.76" x2="289.56" y2="238.76" width="0.1524" layer="91"/>
-<wire x1="279.4" y1="238.76" x2="269.24" y2="238.76" width="0.1524" layer="91"/>
+<wire x1="279.4" y1="238.76" x2="266.7" y2="238.76" width="0.1524" layer="91"/>
 <junction x="279.4" y="238.76"/>
 <label x="269.24" y="238.76" size="1.778" layer="95"/>
+<pinref part="BGND" gate="G$1" pin="P$1"/>
 </segment>
 <segment>
@@
 <attribute name="VALUE" x="129.54" y="170.18" size="1.778" layer="96"/>
 </instance>
+<instance part="PACK-" gate="G$1" x="83.82" y="208.28" rot="R180">
+<attribute name="NAME" x="81.28" y="208.28" size="1.778" layer="95" font="vector" ratio="18" rot="R180"/>
+</instance>
 </instances>
 <busses>
@@
 <wire x1="86.36" y1="198.12" x2="86.36" y2="195.58" width="0.1524" layer="91"/>
 <junction x="86.36" y="195.58"/>
-<wire x1="86.36" y1="195.58" x2="88.9" y2="195.58" width="0.1524" layer="91"/>
-<wire x1="88.9" y1="195.58" x2="91.44" y2="195.58" width="0.1524" layer="91"/>
-<wire x1="91.44" y1="195.58" x2="91.44" y2="226.06" width="0.1524" layer="91"/>
+<wire x1="86.36" y1="195.58" x2="91.44" y2="195.58" width="0.1524" layer="91"/>
+<wire x1="91.44" y1="195.58" x2="91.44" y2="208.28" width="0.1524" layer="91"/>
+<wire x1="91.44" y1="208.28" x2="91.44" y2="226.06" width="0.1524" layer="91"/>
 <wire x1="83.82" y1="238.76" x2="86.36" y2="238.76" width="0.1524" layer="91"/>
 <wire x1="86.36" y1="238.76" x2="86.36" y2="236.22" width="0.1524" layer="91"/>
@@
 <wire x1="91.44" y1="226.06" x2="86.36" y2="226.06" width="0.1524" layer="91"/>
 <wire x1="86.36" y1="228.6" x2="93.98" y2="228.6" width="0.1524" layer="91"/>
-<wire x1="93.98" y1="228.6" x2="93.98" y2="193.04" width="0.1524" layer="91"/>
+<wire x1="93.98" y1="228.6" x2="93.98" y2="208.28" width="0.1524" layer="91"/>
+<wire x1="93.98" y1="208.28" x2="93.98" y2="193.04" width="0.1524" layer="91"/>
 <wire x1="93.98" y1="193.04" x2="86.36" y2="193.04" width="0.1524" layer="91"/>
 <wire x1="86.36" y1="190.5" x2="96.52" y2="190.5" width="0.1524" layer="91"/>
-<wire x1="96.52" y1="190.5" x2="96.52" y2="231.14" width="0.1524" layer="91"/>
+<wire x1="96.52" y1="190.5" x2="96.52" y2="208.28" width="0.1524" layer="91"/>
+<wire x1="96.52" y1="208.28" x2="96.52" y2="231.14" width="0.1524" layer="91"/>
 <wire x1="96.52" y1="231.14" x2="86.36" y2="231.14" width="0.1524" layer="91"/>
 <wire x1="86.36" y1="233.68" x2="99.06" y2="233.68" width="0.1524" layer="91"/>
-<wire x1="99.06" y1="233.68" x2="99.06" y2="187.96" width="0.1524" layer="91"/>
+<wire x1="99.06" y1="233.68" x2="99.06" y2="208.28" width="0.1524" layer="91"/>
+<wire x1="99.06" y1="208.28" x2="99.06" y2="187.96" width="0.1524" layer="91"/>
 <wire x1="99.06" y1="187.96" x2="86.36" y2="187.96" width="0.1524" layer="91"/>
 <wire x1="86.36" y1="185.42" x2="101.6" y2="185.42" width="0.1524" layer="91"/>
-<wire x1="101.6" y1="185.42" x2="101.6" y2="236.22" width="0.1524" layer="91"/>
+<wire x1="101.6" y1="185.42" x2="101.6" y2="208.28" width="0.1524" layer="91"/>
+<wire x1="101.6" y1="208.28" x2="101.6" y2="236.22" width="0.1524" layer="91"/>
 <wire x1="101.6" y1="236.22" x2="86.36" y2="236.22" width="0.1524" layer="91"/>
 <pinref part="R94" gate="G$1" pin="1"/>
@@
 <pinref part="T3" gate="G$1" pin="S5"/>
 <pinref part="T3" gate="G$1" pin="S6"/>
+<pinref part="PACK-" gate="G$1" pin="P$1"/>
+<wire x1="88.9" y1="208.28" x2="91.44" y2="208.28" width="0.1524" layer="91"/>
+<junction x="91.44" y="208.28"/>
+<wire x1="91.44" y1="208.28" x2="93.98" y2="208.28" width="0.1524" layer="91"/>
+<junction x="93.98" y="208.28"/>
+<wire x1="93.98" y1="208.28" x2="96.52" y2="208.28" width="0.1524" layer="91"/>
+<junction x="96.52" y="208.28"/>
+<wire x1="96.52" y1="208.28" x2="99.06" y2="208.28" width="0.1524" layer="91"/>
+<junction x="99.06" y="208.28"/>
+<wire x1="99.06" y1="208.28" x2="101.6" y2="208.28" width="0.1524" layer="91"/>
+<junction x="101.6" y="208.28"/>
 </segment>
 </net>
