File: BMS_hw/AFE_PCB/BMSV1.0.sch (EAGLE design)
At the start: 255 parts, among them IC1 MC33771BEP, IC2 SFH6156-1, IC3 MIC28515V1, IC4 FOD8384-COC, IC5 FOD8384-COC, IC6 FOD8384-COC, IC7 SFH6156-1, IC8 SFH6156-1, Q1 IRLML5203, Q2 IRLML5203, T1 IPT020N10N3V1, T2 IPT020N10N3V1, T3 IPT020N10N3V1, T4 IPT020N10N3V1, X2 87758-2016, X3 87758-2016, X4 22-23-2051, X5 22-23-2041

Commit message: @board layout schmeatic itt@10
Connections:
- net CB_14+/14_C: now also R66.1
- net CELL14+: no longer R66.1
Changed lines of the file:
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@@
-</segment>
-</net>
-<net name="CELL14+" class="0">
-<segment>
-<pinref part="R66" gate="G$1" pin="1"/>
-<wire x1="152.4" y1="78.74" x2="149.86" y2="78.74" width="0.1524" layer="91"/>
-<label x="149.86" y="78.74" size="1.778" layer="95" rot="R180" xref="yes"/>
 </segment>
 </net>
@@
 </segment>
 </net>
+<net name="CB_14+/14_C" class="0">
+<segment>
+<pinref part="R66" gate="G$1" pin="1"/>
+<wire x1="152.4" y1="78.74" x2="149.86" y2="78.74" width="0.1524" layer="91"/>
+<label x="149.86" y="78.74" size="1.778" layer="95" rot="R180" xref="yes"/>
+</segment>
+</net>

Commit message: hjhk
Parts:
- removed X2, X3: 87758-2016, con-molex:87758-2016
- added JP4, JP6: (no value), GreenFuel:PINHD-1X15
Connections:
- net !MCLR: no longer X2-10.S
- net +15V: no longer X2-17.S
- net 3.3V: no longer X2-12.S, X3-16.S
- net CHG_GATE: no longer X2-9.S
- net CSB: no longer X3-7.S
- net DSG_GATE: no longer X2-19.S
- net FAULT_OUT: no longer X2-5.S
- net GND: no longer X2-15.S, X2-18.S, X2-2.S, X2-20.S, X2-3.S, X2-7.S, X2-8.S, X3-1.S, X3-10.S, X3-14.S, X3-18.S, X3-2.S, X3-20.S, X3-3.S, X3-8.S
- net MISO: no longer X2-11.S
- net MOSI: no longer X2-6.S
- net OLED_SCL: no longer X3-6.S
- net OLED_SDA: no longer X3-4.S
- net PCHG_GATE: no longer X2-4.S
- net RDTX_OUT+: no longer X3-5.S
- net RDTX_OUT-: no longer X3-9.S
- net RX_O: no longer X2-14.S
- net S-LED_1: no longer X3-11.S
- net S-LED_2: no longer X3-13.S
- net S-LED_3: no longer X3-15.S
- net S-LED_4: no longer X3-17.S
- net S-LED_5: no longer X3-19.S
- net SCLK: no longer X2-1.S
- net TX_O: no longer X2-16.S
- net VDD: no longer X2-13.S, X3-12.S

Commit message: asdasd
Parts:
- added S1: PGBRD6030-6030, GreenFuel:PGBRD6030-6030
Changed lines of the file:
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@@
 <part name="JP4" library="GreenFuel" deviceset="PINHD-1X15" device=""/>
 <part name="JP6" library="GreenFuel" deviceset="PINHD-1X15" device=""/>
+<part name="S1" library="GreenFuel" deviceset="PGBRD6030" device="-6030"/>
 </parts>
 <sheets>
@@
 <attribute name="VALUE" x="85.09" y="121.92" size="1.778" layer="96" rot="R180"/>
 </instance>
+<instance part="S1" gate="G$1" x="281.94" y="101.6">
+<attribute name="NAME" x="284.48" y="111.76" size="1.27" layer="95" font="vector" ratio="12" rot="R180"/>
+<attribute name="VALUE" x="279.4" y="91.44" size="1.27" layer="96" font="vector" ratio="12"/>
+</instance>
 </instances>

Commit message: ITT@112
Connections:
- net CSB: now also JP6.4
- net MISO: now also JP6.3
- net MOSI: now also JP6.1
- net SCLK: now also JP6.2
Changed lines of the file:
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@@
 </instance>
 <instance part="JP6" gate="A" x="78.74" y="99.06" rot="R180">
-<attribute name="NAME" x="85.09" y="78.105" size="1.778" layer="95" rot="R180"/>
+<attribute name="NAME" x="85.09" y="78.105" size="1.778" layer="95" font="vector" ratio="12" rot="R180"/>
 <attribute name="VALUE" x="85.09" y="121.92" size="1.778" layer="96" rot="R180"/>
 </instance>
@@
 </segment>
 </net>
+<net name="CSB" class="0">
+<segment>
+<pinref part="JP6" gate="A" pin="4"/>
+<wire x1="81.28" y1="88.9" x2="88.9" y2="88.9" width="0.1524" layer="91"/>
+<label x="88.9" y="88.9" size="1.778" layer="95" font="vector" ratio="12"/>
+</segment>
+</net>
+<net name="MISO" class="0">
+<segment>
+<pinref part="JP6" gate="A" pin="3"/>
+<wire x1="81.28" y1="86.36" x2="88.9" y2="86.36" width="0.1524" layer="91"/>
+<label x="88.9" y="86.36" size="1.778" layer="95" font="vector" ratio="12"/>
+</segment>
+</net>
+<net name="SCLK" class="0">
+<segment>
+<pinref part="JP6" gate="A" pin="2"/>
+<wire x1="81.28" y1="83.82" x2="88.9" y2="83.82" width="0.1524" layer="91"/>
+<label x="88.9" y="83.82" size="1.778" layer="95" font="vector" ratio="12"/>
+</segment>
+</net>
+<net name="MOSI" class="0">
+<segment>
+<pinref part="JP6" gate="A" pin="1"/>
+<wire x1="81.28" y1="81.28" x2="88.9" y2="81.28" width="0.1524" layer="91"/>
+<label x="88.9" y="81.28" size="1.778" layer="95" font="vector" ratio="12"/>
+</segment>
+</net>

Commit message: brd layout and sch updated!
Connections:
- net 3.3V: now also JP4.1
Changed lines of the file:
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@@
 <pinref part="X4" gate="-4" pin="S"/>
+</segment>
+<segment>
+<pinref part="JP4" gate="A" pin="1"/>
+<wire x1="68.58" y1="116.84" x2="63.5" y2="116.84" width="0.1524" layer="91"/>
+<label x="58.42" y="116.84" size="1.778" layer="95" font="vector" ratio="12"/>
 </segment>
 </net>

Commit message: board layout and schematic files updated@12
Parts:
- added C69, C70: 10uF, ipc-7351-capacitor:CAPACITOR_0402
- added C81, C82: 10uF, ipc-7351-capacitor:CAPACITOR_0603
- added U1, U2: NCP1117LP-PG, GreenFuel:NCP1117LP-PG
Connections:
- new net 15V_AUX: C70.2, C82.2, U1.IN, U2.IN
- new net 5V: C81.2, U2.OUT
- net 3.3V: now also C69.2, U1.OUT
- net GND: now also C69.1, C70.1, C81.1, C82.1, U1.ADJ/GND, U2.ADJ/GND
Other:
- note added: "Voltage regulator 3.3 volt"
- note added: "Voltage regulator 5 volt"
- moved on the sheet: JP4, JP6

Commit message: @itt@17
Parts:
- added R108: 0R, ipc-7351-resistor:RESISTOR_0603
- C77: value 2.2uF -> 4.7uF; device ipc-7351-capacitor:CAPACITOR_0603 -> ipc-7351-capacitor:CAPACITOR_0805
- R107: value (none) -> 100k
- R91: value 2E2 -> 1R
Connections:
- removed net N$29: C63.2, C64.2, C80.2, IC3.VIN, IC3.VIN@1, IC3.VIN@2, IC3.VIN@3, IC3.VIN@4, IC3.VIN@5, IC3.VIN@6, R79.1
- new net N$13: C65.2, R108.1
- net SW: now also R108.2; no longer C65.2
- net VIN: now also C63.2, C64.2, C80.2, IC3.VIN, IC3.VIN@1, IC3.VIN@2, IC3.VIN@3, IC3.VIN@4, IC3.VIN@5, IC3.VIN@6, R79.1
Other:
- moved on the sheet: C65

Commit message: @dsdwsw
Parts:
- removed D17: SFH48225, GreenFuel:SFH48225
- added C83, C84, C85: 47uF, ipc-7351-capacitor:CAPACITOR_1210
- added LED2: L-59EGW-CAGR, GreenFuel:L-59EGW-CAGR
Connections:
- new net S-LED_6: D19.A, JP4.6
- new net VCC: C83.1, C84.1, C85.1, L1.2, R85.1
- net +15V: no longer L1.2, R85.1
- net 3.3V: now also JP4.7, R102.2; no longer JP4.1
- net GND: now also C83.2, C84.2, C85.2; no longer R102.2
- net N$74: now also LED2.A; no longer D17.C
- net OLED_SCL: now also JP6.5
- net OLED_SDA: now also JP6.6
- net S-LED_1: now also JP4.1
- net S-LED_2: now also JP4.2
- net S-LED_3: now also JP4.3, LED2.CR; no longer D17.A
- net S-LED_4: now also JP4.4, LED2.CG; no longer D18.A
- net S-LED_5: now also D18.A, JP4.5; no longer D19.A
Other:
- moved on the sheet: C63, C64, C65, C66, C73, C74, C76, C77, C80, D18, D19, IC3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
