File: BMS_hw/AFE_PCB/BMSV1.1.brd (EAGLE design)
At the start: 272 x 60 mm, 288 parts, among them IC1 MC33771BEP, IC10 TLP152-COUPLERTOSHIBA, IC11 TLP152-COUPLERTOSHIBA, IC2 SFH6156-1, IC3 MIC28515V1, IC7 SFH6156-1, IC8 SFH6156-1, IC9 TLP152-COUPLERTOSHIBA, Q1 IRLML5203, Q2 BSS138PW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

Commit message: last
Parts:
- removed BGND@1: (no value), simpa:WPAD
- added +12V, +3.3V, +5V, GND, GND@1, WAKE: TP-SMD60, simpa:TP-SMD60
- C69, C70, C81, C82: device ipc-7351-capacitor:CAPC1005X60N -> ipc-7351-capacitor:CAPC2012X145AN
- C74: value 47nF -> 1uF 100V; device ipc-7351-capacitor:CAPC1608X92N -> ipc-7351-capacitor:CAPC2012X145AN
- R79: value 2E -> 2.2E
- R98: value 300E -> 330E
- moved C70 1.42 mm to (222.9, 30.5)
- moved C81 1.42 mm to (221.0, 24.1), turned to 180 degrees
- moved C82 0.64 mm to (222.9, 27.9)
Connections:
- net +12V: now also +12V.P$1
- net 3.3V: now also +3.3V.P$1
- net 5V: now also +5V.P$1
- net BGND: no longer BGND@1.1
- net GND: now also GND.P$1, GND@1.P$1
- net WAKE: now also WAKE.P$1
Routing:
- net 3.3V: track 155.3 -> 173.3 mm
- net BGND: track 47.8 -> 36.0 mm
- net WAKE: track 18.2 -> 28.2 mm
- net 5V: track 22.0 -> 29.0 mm
- net +12V: track 249.7 -> 256.0 mm
- net GND: track 58.8 -> 55.6 mm, vias 155 -> 153
- added copper zone on layer 16, net BGND

Commit message: board schematic and part updated
Parts:
- added R120: 1K, ipc-7351-resistor:RESC5025X70N
- C75: device ipc-7351-capacitor:CAPC1005X60N -> ipc-7351-capacitor:CAPC2012X145AN
- Q2: value BSS138PW -> SI2392ADS-T1-GE3; device simpa:SOT323 -> GreenFuel:SOT23-3
- R100, R99: device ipc-7351-resistor:RESC1005X40AN -> ipc-7351-resistor:RESC1608X55N
- R101, R102, R116, R117: value 33E -> 75E
- R103, R104: value 330E -> 75E
- R111, R112, R113, R114, R115, R80: value 330E -> 1K
- R86: value 380E -> 526E; device ipc-7351-resistor:RESC1005X40AN -> ipc-7351-resistor:RESC1608X55N
- R98: value 330E -> 1K; device ipc-7351-resistor:RESC1005X40AN -> ipc-7351-resistor:RESC5025X70N
- U1: value NCP1117LP-PG -> NCV1117ST33T3G
- U2: value NCP1117LP-PG -> NCV1117ST50T3G
- moved R98 10.2 mm to (127.6, 18.4), flipped to the bottom, turned to 180 degrees
- moved Q2 4.58 mm to (137.2, 15.9), flipped to the bottom
- moved C23 2.62 mm to (84.5, 41.9), turned to 135 degrees
- moved C81 2.29 mm to (222.9, 25.4)
- moved C74 1.91 mm to (242.6, 32.6)
- moved R100 1.42 mm to (226.1, 28.6), turned to 90 degrees
- moved R30 1.27 mm to (83.2, 40.6), turned to 135 degrees
- moved C71 0.90 mm to (89.5, 38.1), turned to 315 degrees
- moved R86 0.68 mm to (239.5, 38.8), turned to 225 degrees
- moved Q1 0.63 mm to (186.7, 52.1), turned to 270 degrees
- moved C72 0.19 mm to (87.5, 40.0), turned to 135 degrees
Connections:
- net +12V: now also LED1.2, LED2.2, LED3.A, LED4.A
- net 3.3V: no longer LED1.2, LED2.2, LED3.A, LED4.A
- net BGND: now also R120.1
- net N$28: now also R120.2
Routing:
- net 3.3V: track 173.3 -> 135.7 mm
- net BGND: track 36.0 -> 10.6 mm
- net +12V: track 256.0 -> 280.6 mm
- net PCHG_FET: track 41.5 -> 35.2 mm
- net N$19: track 43.3 -> 37.6 mm
- net PWR_DRAIN: track 12.7 -> 7.16 mm
- net CHG_FET: track 33.0 -> 27.6 mm
- net N$28: track 3.91 -> 0.00 mm
- net N$31: track 144.7 -> 148.2 mm
- net 5V: track 29.0 -> 25.6 mm, vias 2 -> 0
- net GND: track 55.6 -> 53.9 mm
- net WAKE: track 28.2 -> 29.5 mm
- net N$21: track 4.81 -> 6.14 mm
- net ISENSE+: track 9.71 -> 8.68 mm
- net ISENSE-: track 9.04 -> 8.30 mm
- added copper zone on layer 16, net PWR_DRAIN1
Other:
- board text added: "v1.1"

Commit message: sch board updated
Parts:
- removed R120: 1K, ipc-7351-resistor:RESC5025X70N
- moved Q2 2.54 mm to (137.2, 18.4), flipped to the top, turned to 270 degrees
- moved R98 0.64 mm to (128.3, 18.4)
Connections:
- net BGND: no longer R120.1
- net N$28: no longer R120.2
Routing:
- net N$19: track 37.6 -> 22.8 mm
- net +12V: track 280.6 -> 291.0 mm
- net PWR_DRAIN: track 7.16 -> 13.6 mm
- net N$28: track 0.00 -> 5.83 mm, vias 0 -> 1
- net PCHG_FET: track 35.2 -> 34.2 mm
Changed lines of the file:
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@@
 <attribute name="VALUE" x="128.9355" y="44.507" size="1.27" layer="27" rot="R270"/>
 </element>
-<element name="Q2" library="GreenFuel" package="SOT23-3" value="SI2392ADS-T1-GE3" x="137.16" y="15.875" smashed="yes" rot="MR90">
-<attribute name="NAME" x="134.315" y="15.545" size="0.762" layer="26" font="vector" ratio="12" rot="MR90"/>
-<attribute name="VALUE" x="133.76" y="14.375" size="1.778" layer="28" rot="MR90"/>
-</element>
-<element name="R98" library="ipc-7351-resistor" package="RESC5025X70N" value="1K" x="127.635" y="18.415" smashed="yes" rot="MR180">
-<attribute name="NAME" x="126.504" y="19.893" size="0.762" layer="26" font="vector" ratio="12" rot="MR180"/>
-<attribute name="VALUE" x="126.885" y="20.239" size="1.27" layer="28" font="vector" ratio="10" rot="MR180"/>
+<element name="Q2" library="GreenFuel" package="SOT23-3" value="SI2392ADS-T1-GE3" x="137.16" y="18.415" smashed="yes" rot="R270">
+<attribute name="NAME" x="140.665" y="18.745" size="0.762" layer="25" font="vector" ratio="12" rot="R270"/>
+<attribute name="VALUE" x="133.76" y="19.915" size="1.778" layer="27" rot="R270"/>
+</element>
+<element name="R98" library="ipc-7351-resistor" package="RESC5025X70N" value="1K" x="128.27" y="18.415" smashed="yes" rot="MR180">
+<attribute name="NAME" x="127.139" y="20.528" size="0.762" layer="26" font="vector" ratio="12" rot="MR180"/>
+<attribute name="VALUE" x="127.52" y="20.239" size="1.27" layer="28" font="vector" ratio="10" rot="MR180"/>
 </element>
 <element name="R3" library="ipc-7351-resistor" package="RESC1005X40AN" value="0E" x="250.825" y="53.34" smashed="yes" rot="R180">
@@
 </element>
 <element name="R81" library="GreenFuel" package="SMD4" value="LRMAP3920SUNT" x="120.65" y="40.005" smashed="yes" rot="R180">
-<attribute name="NAME" x="125.65" y="35.505" size="1.27" layer="25" font="vector" ratio="12" rot="R180"/>
+<attribute name="NAME" x="119.435" y="35.48" size="1.27" layer="25" font="vector" ratio="12" rot="R270"/>
 <attribute name="VALUE" x="125.65" y="45.505" size="1.27" layer="27" rot="R180"/>
 </element>
 <element name="R84" library="GreenFuel" package="SMD4" value="LRMAP3920SUNT" x="120.65" y="27.305" smashed="yes" rot="R180">
-<attribute name="NAME" x="125.65" y="22.805" size="1.27" layer="25" font="vector" ratio="12" rot="R180"/>
+<attribute name="NAME" x="120.07" y="20.875" size="1.27" layer="25" font="vector" ratio="12" rot="R270"/>
 <attribute name="VALUE" x="125.65" y="32.805" size="1.27" layer="27" rot="R180"/>
 </element>
@@
 <attribute name="NAME" x="260.985" y="6.35" size="1.016" layer="25" ratio="12"/>
 </element>
-<element name="R120" library="ipc-7351-resistor" package="RESC5025X70N" value="1K" x="127.635" y="14.605" smashed="yes" rot="MR180">
-<attribute name="NAME" x="123.96" y="12.5875" size="1.27" layer="26" font="vector" ratio="10" rot="MR180"/>
-<attribute name="VALUE" x="123.96" y="17.8925" size="1.27" layer="28" font="vector" ratio="10" rot="MR180"/>
-</element>
 </elements>
 <signals>
@@
 <wire x1="180.135" y1="45.515" x2="180.34" y2="45.72" width="0.3048" layer="16"/>
 <via x="180.34" y="45.72" extent="1-16" drill="0.3048"/>
-<wire x1="194.2846" y1="49.27749375" x2="194.2846" y2="49.78250625" width="0.3048" layer="1"/>
-<wire x1="194.2846" y1="49.78250625" x2="193.92750625" y2="50.1396" width="0.3048" layer="1"/>
 <wire x1="180.34" y1="45.72" x2="182.9794" y2="48.3594" width="0.3048" layer="1"/>
-<wire x1="193.92750625" y1="50.1396" x2="191.77" y2="50.1396" width="0.3048" layer="1"/>
-<wire x1="193.36650625" y1="48.3594" x2="194.2846" y2="49.27749375" width="0.3048" layer="1"/>
-<wire x1="182.9794" y1="48.3594" x2="193.36650625" y2="48.3594" width="0.3048" layer="1"/>
-<wire x1="191.77" y1="50.1396" x2="187.69" y2="52.07" width="0" layer="19" extent="1-1"/>
+<wire x1="187.69" y1="52.07" x2="182.9794" y2="48.3594" width="0" layer="19" extent="1-1"/>
 </signal>
 <signal name="PWR_DRAIN">
@@
 <via x="144.145" y="24.765" extent="1-16" drill="0.5" diameter="0.8128"/>
 <contactref element="Q2" pad="3"/>
-<wire x1="142.5375" y1="23.6975" x2="142.5375" y2="21.6375" width="0.2286" layer="1"/>
+<wire x1="142.5375" y1="21.6375" x2="142.5375" y2="23.6975" width="0.2286" layer="1"/>
 <wire x1="138.93" y1="27.305" x2="142.5375" y2="23.6975" width="0.2286" layer="1"/>
-<wire x1="142.5375" y1="21.6375" x2="138.26" y2="15.875" width="0" layer="19" extent="1-16"/>
+<wire x1="137.625" y1="18.415" x2="138.43" y2="18.415" width="0.8128" layer="1"/>
+<wire x1="138.43" y1="18.415" x2="139.065" y2="18.415" width="0.8128" layer="1"/>
+<wire x1="139.065" y1="18.415" x2="142.2875" y2="21.6375" width="0.8128" layer="1"/>
+<wire x1="142.2875" y1="21.6375" x2="142.5375" y2="21.6375" width="0.8128" layer="1"/>
+<wire x1="138.26" y1="18.415" x2="138.43" y2="18.415" width="0.3048" layer="1"/>
 </signal>
 <signal name="PGND">
@@
 <signal name="PCHG_FET">
 <contactref element="Q2" pad="1"/>
-<via x="135.89" y="18.415" extent="1-16" drill="0.3048"/>
-<wire x1="135.89" y1="18.415" x2="136.017" y2="18.542" width="0.3048" layer="16"/>
 <contactref element="IC11" pad="5"/>
 <wire x1="136.525" y1="50.8" x2="139.09" y2="50.8" width="0.3048" layer="16"/>
-<wire x1="136.017" y1="18.542" x2="136.017" y2="50.292" width="0.3048" layer="16"/>
+<wire x1="136.017" y1="50.292" x2="136.017" y2="20.447" width="0.3048" layer="16"/>
 <wire x1="136.017" y1="50.292" x2="136.525" y2="50.8" width="0.3048" layer="16"/>
-<wire x1="136.06" y1="14.925" x2="135.89" y2="18.415" width="0" layer="19" extent="16-16"/>
+<via x="136.017" y="20.447" extent="1-16" drill="0.35"/>
+<wire x1="136.017" y1="19.408" x2="136.017" y2="20.447" width="0.3048" layer="1"/>
+<wire x1="136.06" y1="19.365" x2="136.017" y2="19.408" width="0.3048" layer="1"/>
 </signal>
 <signal name="DSG_FET">
@@
 <vertex x="110.49" y="22.225"/>
 </polygon>
-<contactref element="R120" pad="1"/>
 <polygon width="0.3048" layer="16">
-<vertex x="114.3" y="22.225"/>
-<vertex x="114.3" y="14.605"/>
-<vertex x="116.205" y="12.7"/>
-<vertex x="127.635" y="12.7"/>
-<vertex x="127.635" y="19.685"/>
+<vertex x="114.935" y="22.225"/>
+<vertex x="114.935" y="16.51"/>
+<vertex x="127" y="16.51"/>
 <vertex x="127" y="20.32"/>
 <vertex x="119.38" y="20.32"/>
@@
 <wire x1="182.245" y1="28.575" x2="182.88" y2="28.575" width="0.3048" layer="1"/>
 <wire x1="182.88" y1="28.575" x2="184.15" y2="29.845" width="0.3048" layer="1"/>
+<wire x1="183.515" y1="36.195" x2="185.42" y2="38.1" width="0.3048" layer="1"/>
+<wire x1="185.42" y1="38.1" x2="185.42" y2="45.72" width="0.3048" layer="1"/>
 <wire x1="189.38526875" y1="52.07" x2="185.42" y2="45.72" width="0" layer="19" extent="16-16"/>
-<wire x1="185.42" y1="38.1" x2="185.42" y2="45.72" width="0" layer="19" extent="1-1"/>
-<wire x1="183.515" y1="36.195" x2="185.42" y2="38.1" width="0" layer="19" extent="1-1"/>
 </signal>
 <signal name="S-LED_3">
@@
 <contactref element="Q2" pad="2"/>
 <contactref element="R98" pad="2"/>
-<contactref element="R120" pad="2"/>
-<wire x1="129.985" y1="18.415" x2="136.06" y2="16.825" width="0" layer="19" extent="16-16"/>
-<wire x1="129.985" y1="14.605" x2="129.985" y2="18.415" width="0" layer="19" extent="16-16"/>
+<wire x1="130.62" y1="18.415" x2="132.715" y2="18.415" width="0.8128" layer="16"/>
+<via x="132.715" y="18.415" extent="1-16" drill="0.8"/>
+<wire x1="132.715" y1="18.415" x2="133.665" y2="17.465" width="0.8128" layer="1"/>
+<wire x1="135.425" y1="17.465" x2="133.665" y2="17.465" width="0.8128" layer="1"/>
+<wire x1="136.06" y1="17.465" x2="135.425" y2="17.465" width="0.3048" layer="1"/>
 </signal>
 <signal name="N$22">

Commit message: updated afe shmetatic rectification stage of MCU PCB
Parts:
- removed +12V: TP-SMD60, simpa:TP-SMD60
- removed JP2: (no value), adafruit:1X01-CLEANBIG
- removed X5: 22-23-2041, GreenFuel:22-23-2041
- added CG, CH, CL, KI: TPTH7035, simpa:TP7035
- added FD1, FD2, FD3, FD4, FD5, FD6: FIDUCIAL, adafruit:FIDUCIAL_1MM
- C90, C91: device ipc-7351-capacitor:CAPAE430X540N -> ipc-7351-capacitor:CAPAE830X1020N
- Q1: value IRLML5203 -> ZXMP10A17G; device transistor-power:MICRO3 -> GreenFuel:SOT23-3
- R108: device ipc-7351-resistor:RESC1608X55N -> ipc-7351-resistor:RESC1005X40AN
- R119, R31, R95, R97: device ipc-7351-resistor:RESC1005X40AN -> ipc-7351-resistor:RESC1608X55N
- moved JP7 52.2 mm to (226.1, 8.89), turned to 0 degrees
- moved C66 21.5 mm to (240.7, 37.1), turned to 0 degrees
- moved R85 19.1 mm to (260.4, 45.2), turned to 180 degrees
- moved C83 15.9 mm to (267.6, 22.2), turned to 270 degrees
- moved C84 13.1 mm to (264.2, 22.2), turned to 270 degrees
- moved R79 11.7 mm to (247.7, 23.5), turned to 180 degrees
- moved C63 10.8 mm to (253.4, 26.7), turned to 180 degrees
- moved C85 8.91 mm to (256.5, 21.6)
- moved C90 8.89 mm to (250.8, 10.8)
- moved R108 6.48 mm to (246.4, 27.3), turned to 180 degrees
- moved C64 5.92 mm to (247.7, 19.7)
- moved R83 5.85 mm to (257.3, 44.2)
- moved C87 4.62 mm to (256.8, 24.5)
- moved R86 4.07 mm to (240.7, 34.9), turned to 180 degrees
- moved R118 3.41 mm to (244.5, 37.0), turned to 180 degrees
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Connections:
- removed net INTL_OUT1: JP2.1, X5.2
- net +12V: no longer +12V.P$1
- net CANH: now also CH.P$1; no longer X5.4
- net CANL: now also CL.P$1; no longer X5.3
- net CB_14+/14_C: no longer C63.2, C64.2, C90.+, IC3.10, IC3.11, IC3.5, IC3.6, IC3.7, IC3.8, IC3.9, R79.1
- net CELL14+: now also C63.2, C64.2, C90.+, IC3.10, IC3.11, IC3.5, IC3.6, IC3.7, IC3.8, IC3.9, R79.1
- net GND: now also CG.P$1
- net INTL_IN2: now also KI.P$1; no longer X5.1
Routing:
- net CB_14+/14_C: track 414.4 -> 347.1 mm, vias 18 -> 8
- net CELL14+: track 8.50 -> 73.6 mm, vias 0 -> 57
- net N$14: track 90.2 -> 36.3 mm, vias 1 -> 2
- net V+: track 135.2 -> 110.6 mm
- net N$24: track 3.03 -> 22.9 mm, vias 0 -> 2
- net N$15: track 81.7 -> 65.2 mm, vias 3 -> 4
- net SW: track 32.3 -> 47.0 mm, vias 0 -> 2
- net VDD: track 29.9 -> 19.0 mm, vias 3 -> 2
- net N$21: track 6.14 -> 15.6 mm
- net INTL_OUT1: track 9.31 -> 0.00 mm
- net N$61: track 6.32 -> 2.65 mm
- net CHG_FET: track 27.6 -> 24.1 mm
- net N$19: track 22.8 -> 26.1 mm
- net N$13: track 4.68 -> 1.72 mm
- net PVDD: track 8.25 -> 5.92 mm
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- added copper zone on layer 16, net +12V
- added copper zone on layer 1, net CELL14+
- added copper zone on layer 16, net CELL14+
- removed copper zone on layer 1, net CB_14+/14_C
- removed copper zone on layer 16, net CB_14+/14_C

Commit message: updated
Parts:
- added R120: 10k, ipc-7351-resistor:RESC1608X55N
- added R121: 5.23k, ipc-7351-resistor:RESC1608X55N
- added R122, R123, R124: 0E, ipc-7351-resistor:RESC1005X40AN
- moved R34 1.91 mm to (10.2, 45.1)
- moved R38 1.91 mm to (8.26, 45.1)
Connections:
- new net N$62: JP6.3, R120.1, R121.1
- net BGND: now also R122.1, R123.1, R124.1
- net GND: now also R120.2, R122.2, R123.2, R124.2
- net MISO: now also R121.2; no longer JP6.3
Routing:
- net MISO: track 136.8 -> 11.0 mm
- net N$62: track 0.00 -> 125.4 mm
- net BGND: track 10.6 -> 35.9 mm
- net N$15: track 65.2 -> 58.4 mm
- net 3.3V: track 135.7 -> 131.9 mm
- net CELL1-: track 65.7 -> 63.8 mm
- net 5V: track 25.6 -> 24.7 mm
- net CT_11: track 31.2 -> 30.4 mm
- net N$36: track 15.7 -> 15.1 mm
- net CELL14+: track 73.6 -> 73.0 mm
- net CSB: track 140.5 -> 139.9 mm
- net GND: vias 239 -> 248
Other:
- board text added: "Greenfuel Energy Solutions Pvt. Ltd."
- board text added: "v1.2"
- board text removed: "v1.1"
