File: BMS_hw/MCU_PCB/BMS_MCUV1.0.brd (EAGLE design)
At the start: 60 x 30 mm, 49 parts, among them IC2 SST25VF020B804ISA, J1 22-27-2051-05, J2 22-27-2051-05, J3 22-27-2041-04, J4 22-27-2051-05, U1 NCP1117LP-PG, X1 87758-2016

Commit message: Testing git bash trial !
Parts:
- moved L4 9.55 mm to (14.0, -28.6)
Changed lines of the file:
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@@
 <attribute name="VALUE" x="33.533" y="12.8825" size="0.127" layer="27" font="vector" ratio="12" rot="R180"/>
 </element>
-<element name="L4" library="ipc-7351-inductor" package="INDC1608X95N" value="" x="14.605" y="-38.1">
-<attribute name="NAME" x="13.33" y="-37.2825" size="1.27" layer="25" font="vector" ratio="10"/>
-<attribute name="VALUE" x="13.965" y="-39.0445" size="0.127" layer="27" font="vector" ratio="12"/>
+<element name="L4" library="ipc-7351-inductor" package="INDC1608X95N" value="" x="13.97" y="-28.575">
+<attribute name="NAME" x="12.695" y="-27.7575" size="1.27" layer="25" font="vector" ratio="10"/>
+<attribute name="VALUE" x="13.33" y="-29.5195" size="0.127" layer="27" font="vector" ratio="12"/>
 </element>
 <element name="MCU2" library="GreenFuel" package="TQFP-64-I/PT" value="PIC32MK0512GPE064-I/PT" x="20.955" y="15.24" rot="R45">
@@
 <wire x1="14.616" y1="-54.864" x2="12.435" y2="-57.785" width="0" layer="19" extent="1-1"/>
 <wire x1="12.662" y1="-50.292" x2="14.616" y2="-54.864" width="0" layer="19" extent="1-1"/>
-<wire x1="13.805" y1="-38.1" x2="12.662" y2="-50.292" width="0" layer="19" extent="1-1"/>
+<wire x1="13.17" y1="-28.575" x2="12.662" y2="-50.292" width="0" layer="19" extent="1-1"/>
 </signal>
 <signal name="N$6">
@@
 <contactref element="L4" pad="2"/>
 <wire x1="32.22" y1="8.89" x2="32.093" y2="11.938" width="0" layer="19" extent="1-1"/>
-<wire x1="15.405" y1="-38.1" x2="32.22" y2="8.89" width="0" layer="19" extent="1-1"/>
+<wire x1="14.77" y1="-28.575" x2="32.22" y2="8.89" width="0" layer="19" extent="1-1"/>
 </signal>
 <signal name="N$9">

Commit message: updated schematic inductor part no 3.3 5v ldo net naaming
Parts:
- added C5, C6: 10uF, ipc-7351-capacitor:CAPC1608X92N
- added U2: NCP1117LP-PG, GreenFuel:SOT-223
- C3, C4: value .01uF -> 10uF
- L2, L3, L4: value (none) -> MMZ2012R301ATD25; device ipc-7351-inductor:INDC1608X95N -> ipc-7351-resistor:RESC2012X70N
Connections:
- removed net N$12: C8.1, U$1.11, U$1.16
- removed net N$8: C12.1, U$1.1
- new net 5V: C5.2, C8.1, U$1.11, U$1.16, U2.2
- net 15V_AUX: now also C6.2, U2.3
- net 3.3V: now also C12.1, U$1.1
- net GND: now also C5.1, C6.1, U2.1, U2.4

Commit message: hjhk
Parts:
- removed X1: 87758-2016, con-molex:87758-2016
- removed X2, X3: (no value), con-molex:KK-156-10
- added JP1, JP5: (no value), GreenFuel:1X15
- moved U$1 107.3 mm to (49.5, 16.5)
- moved U1 82.7 mm to (-11.4, 19.7)
- moved Q1 2.29 mm to (31.8, 22.2)
Connections:
- net 15V_AUX: no longer X1.17
- net C_FET: no longer X1.9
- net D_FET: no longer X1.19
- net FAULT: no longer X1.5
- net GND: no longer U$1.2, X1.1, X1.10, X1.14, X1.15, X1.16, X1.18, X1.2, X1.20, X1.3, X1.6, X1.7, X1.8
- net ISP: no longer X1.11
- net N$7: now also U$1.2
- net PCHG_FET: no longer X1.4
- net VDD: no longer X1.12, X1.13
Routing:
- net GND: track 0.00 -> 21.8 mm

Commit message: asdasd
Parts:
- C1, C2, C21: device ipc-7351-capacitor:CAPC1608X92N -> ipc-7351-capacitor:CAPC1005X60N
Changed lines of the file:
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@@
 <setting verticaltext="up"/>
 </settings>
-<grid distance="25" unitdist="mil" unit="mil" style="dots" multiple="1" display="yes" altdistance="5" altunitdist="mil" altunit="mil"/>
+<grid distance="25" unitdist="mil" unit="mm" style="dots" multiple="1" display="yes" altdistance="5" altunitdist="mil" altunit="mm"/>
 <layers>
 <layer number="1" name="Top" color="4" fill="1" visible="yes" active="yes"/>
@@
 <layer number="45" name="Holes" color="7" fill="1" visible="no" active="yes"/>
 <layer number="46" name="Milling" color="3" fill="1" visible="no" active="yes"/>
-<layer number="47" name="Measures" color="7" fill="1" visible="no" active="yes"/>
+<layer number="47" name="Measures" color="7" fill="1" visible="yes" active="yes"/>
 <layer number="48" name="Document" color="7" fill="1" visible="yes" active="yes"/>
 <layer number="49" name="Reference" color="7" fill="1" visible="no" active="yes"/>
@@
 </autorouter>
 <elements>
-<element name="C1" library="ipc-7351-capacitor" package="CAPC1608X92N" value="20pF" x="31.75" y="16.51">
+<element name="C1" library="ipc-7351-capacitor" package="CAPC1005X60N" value="20pF" x="31.75" y="16.51">
 <attribute name="NAME" x="30.5" y="17.2775" size="1.27" layer="25" font="vector" ratio="10"/>
 <attribute name="VALUE" x="30.5" y="14.4725" size="1.27" layer="27" font="vector" ratio="10"/>
@@
 <attribute name="VALUE" x="12.68" y="9.0225" size="1.27" layer="27" font="vector" ratio="10" rot="R180"/>
 </element>
-<element name="C2" library="ipc-7351-capacitor" package="CAPC1608X92N" value="20pF" x="40.005" y="22.225">
+<element name="C2" library="ipc-7351-capacitor" package="CAPC1005X60N" value="20pF" x="40.005" y="22.225">
 <attribute name="NAME" x="38.755" y="22.9925" size="1.27" layer="25" font="vector" ratio="10"/>
 <attribute name="VALUE" x="38.755" y="20.1875" size="1.27" layer="27" font="vector" ratio="10"/>
@@
 <attribute name="VALUE" x="37.445" y="17.2775" size="1.27" layer="27" font="vector" ratio="10" rot="R180"/>
 </element>
-<element name="C21" library="ipc-7351-capacitor" package="CAPC1608X92N" value="0.1uF" x="6.985" y="6.985" rot="R180">
+<element name="C21" library="ipc-7351-capacitor" package="CAPC1005X60N" value="0.1uF" x="6.985" y="6.985" rot="R180">
 <attribute name="NAME" x="8.235" y="6.2175" size="1.27" layer="25" font="vector" ratio="10" rot="R180"/>
 <attribute name="VALUE" x="8.235" y="9.0225" size="1.27" layer="27" font="vector" ratio="10" rot="R180"/>
@@
 <wire x1="26.035" y1="20.32" x2="28.575" y2="17.78" width="0.2794" layer="1"/>
 <wire x1="32.385" y1="17.78" x2="32.55" y2="17.615" width="0.2794" layer="1"/>
-<wire x1="32.55" y1="17.615" x2="32.55" y2="16.51" width="0.2794" layer="1"/>
+<wire x1="32.55" y1="17.615" x2="32.2" y2="16.51" width="0.2794" layer="1"/>
 <wire x1="28.575" y1="17.78" x2="32.385" y2="17.78" width="0.2794" layer="1"/>
 <wire x1="-9.055" y1="-127.635" x2="-14.135" y2="-127.635" width="0" layer="19" extent="1-1"/>
@@
 <contactref element="Q1" pad="3"/>
 <wire x1="25.5158375" y1="18.740178125" x2="29.55" y2="21.025" width="0" layer="19" extent="1-1"/>
-<wire x1="30.95" y1="16.51" x2="29.55" y2="21.025" width="0" layer="19" extent="1-1"/>
+<wire x1="31.3" y1="16.51" x2="29.55" y2="21.025" width="0" layer="19" extent="1-1"/>
 </signal>
 <signal name="N$2">
@@
 <contactref element="MCU2" pad="40"/>
 <contactref element="Q1" pad="1"/>
-<wire x1="33.95" y1="23.425" x2="39.205" y2="22.225" width="0" layer="19" extent="1-1"/>
+<wire x1="33.95" y1="23.425" x2="39.555" y2="22.225" width="0" layer="19" extent="1-1"/>
 <wire x1="25.162284375" y1="19.09373125" x2="33.95" y2="23.425" width="0" layer="19" extent="1-1"/>
 </signal>
@@
 <contactref element="C21" pad="1"/>
 <wire x1="7.7088" y1="9.8044" x2="10.6046" y2="9.906" width="0" layer="19" extent="1-1"/>
-<wire x1="7.785" y1="6.985" x2="7.7088" y2="9.8044" width="0" layer="19" extent="1-1"/>
+<wire x1="7.435" y1="6.985" x2="7.7088" y2="9.8044" width="0" layer="19" extent="1-1"/>
 </signal>
 <signal name="N$33">

Commit message: brd layout and sch updated!
Parts:
- C10, C13, C7, C9: device ipc-7351-capacitor:CAPC2012X145AN -> ipc-7351-capacitor:CAPC1005X60N
- C11, C12, C8: device adafruit:C0805 -> ipc-7351-capacitor:CAPC1005X60N
- C14, C17, C18, C19, C20, C22, C3, C4: device ipc-7351-capacitor:CAPC1608X92N -> ipc-7351-capacitor:CAPC1005X60N
- Q1: value (none) -> CRYSTALS-GND-LID-IQXC-42; device adafruit:CTS406 -> IQD-Frequency-Products:2.0X1.6-4-PAD
- R10, R11, R12, R13, R14, R3, R4, R5, R6, R7, R8, R9: device ipc-7351-resistor:RESC2012X70N -> ipc-7351-resistor:RESC1005X40AN
- R15, R16: device ipc-7351-resistor:RESC1608X55N -> ipc-7351-resistor:RESC1005X40AN
- moved IC2 159.4 mm to (8.26, 24.1), turned to 45 degrees
- moved C5 149.6 mm to (46.4, 9.53), turned to 270 degrees
- moved C6 145.3 mm to (46.4, 6.99)
- moved U2 140.4 mm to (52.7, 9.53), turned to 270 degrees
- moved R6 107.4 mm to (47.6, 17.1), turned to 180 degrees
- moved R12 102.2 mm to (3.17, 14.0)
- moved R5 101.0 mm to (48.9, 14.6), turned to 180 degrees
- moved R11 99.6 mm to (3.17, 15.2)
- moved C11 95.6 mm to (31.1, 11.4), turned to 180 degrees
- moved R14 94.9 mm to (5.71, 14.0), turned to 180 degrees
- moved C12 94.8 mm to (47.0, 12.7), turned to 90 degrees
- moved R10 94.6 mm to (3.17, 16.5)
- moved C10 94.1 mm to (32.3, 17.1)
- moved R3 93.9 mm to (32.4, 13.3), turned to 180 degrees
- moved R9 92.6 mm to (3.17, 17.8), turned to 180 degrees
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Connections:
- new net N$3: C12.1, U$1.1
- net 3.3V: no longer C12.1, U$1.1
- net GND: now also Q1.2, Q1.4
Routing:
- net GND: track 21.9 -> 0.00 mm

Commit message: board layout and schematic files updated@12
Parts:
- removed C3, C4: 10uF, ipc-7351-capacitor:CAPC1005X60N
- removed C5, C6: 10uF, ipc-7351-capacitor:CAPC1608X92N
- removed J1, J2, J4: 22-27-2051-05, con-molex:6410-05
- removed J3: 22-27-2041-04, con-molex:6410-04
- removed U1, U2: NCP1117LP-PG, GreenFuel:SOT-223
- added JP2: (no value), GreenFuel:1X12X2
- Q1: device IQD-Frequency-Products:2.0X1.6-4-PAD -> GreenFuel:1.4X1.2-4-PAD
- moved R12 47.1 mm to (50.2, 10.8)
- moved R11 47.0 mm to (50.2, 13.3)
- moved R8 47.0 mm to (50.2, 21.0)
- moved R10 47.0 mm to (50.2, 15.9)
- moved R9 47.0 mm to (50.2, 18.4)
- moved L2 9.61 mm to (12.1, 5.71), turned to 135 degrees
- moved C7 9.55 mm to (24.8, 6.99)
- moved L4 9.25 mm to (21.0, 11.4)
- moved C14 8.98 mm to (3.09, 28.0), turned to 225 degrees
- moved JP5 8.89 mm to (29.2, 27.3)
- moved JP1 8.26 mm to (29.2, 3.17)
- moved C19 7.18 mm to (22.2, 6.35)
- moved C9 7.01 mm to (25.5, 14.7)
- moved C13 6.35 mm to (27.7, 8.00)
- moved R5 5.85 mm to (43.2, 13.3)
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Connections:
- removed net 15V_AUX: C4.2, C6.2, U1.3, U2.3
- removed net N$18: J1.1, R8.2
- removed net N$19: J1.2, R9.2
- removed net N$20: J1.3, R10.2
- removed net N$21: J1.4, R11.2
- removed net N$22: J1.5, R12.2
- removed net VSS: J2.3
- net !MCLR: no longer J2.1
- net 3.3V: no longer C3.2, U1.2
- net 5V: no longer C5.2, U2.2
- net CANH: no longer J4.3
- net CANL: no longer J4.4
- net DBG_RX: no longer J3.3
- net DBG_TX: no longer J3.2
- net GND: no longer C3.1, C4.1, C5.1, C6.1, J3.1, J3.4, J4.5, U1.1, U1.4, U2.1, U2.4
- net ICSPCLK: no longer J2.5
- net ICSPDAT: no longer J2.4
- net INTL_IN2: no longer J4.2
- net INTL_OUT: no longer J4.1
- net VDD: no longer J2.2
Routing:
- net CE#: track 0.00 -> 21.0 mm, vias 0 -> 2
- net SO: track 0.00 -> 19.4 mm, vias 0 -> 2
- net WP#: track 0.00 -> 18.4 mm, vias 0 -> 2
- net 5V: track 0.00 -> 13.7 mm
- net SCK: track 0.00 -> 13.6 mm, vias 0 -> 2
- net SI: track 0.00 -> 13.0 mm, vias 0 -> 2
- net N$32: track 0.00 -> 6.20 mm
- net GND: track 0.00 -> 3.82 mm
- net N$7: track 0.00 -> 3.78 mm
- net N$14: track 0.00 -> 3.54 mm
- net !MCLR: track 0.00 -> 3.26 mm
- net VDD: track 0.00 -> 2.89 mm
- net N$3: track 0.00 -> 2.67 mm
- net N$6: track 0.00 -> 2.51 mm
- net N$34: track 0.00 -> 1.90 mm

Commit message: brd layout and sch update @14
Parts:
- moved R14 47.0 mm to (48.3, 24.8), turned to 225 degrees
- moved R13 45.6 mm to (47.6, 22.2), turned to 225 degrees
- moved C9 18.6 mm to (43.7, 18.8), turned to 0 degrees
- moved R3 17.2 mm to (45.1, 16.5), turned to 270 degrees
- moved R5 16.1 mm to (27.9, 18.4), turned to 0 degrees
- moved C12 15.4 mm to (33.0, 22.9), turned to 0 degrees
- moved R6 15.3 mm to (27.9, 15.9), turned to 0 degrees
- moved R7 15.2 mm to (43.2, 16.8), turned to 90 degrees
- moved C8 14.8 mm to (42.5, 13.9), turned to 270 degrees
- moved R12 7.24 mm to (52.1, 17.8), turned to 0 degrees
- moved R10 7.24 mm to (52.1, 22.9), turned to 0 degrees
- moved R11 7.24 mm to (52.1, 20.3), turned to 0 degrees
- moved R9 6.63 mm to (52.1, 24.8), turned to 0 degrees
- moved C1 6.35 mm to (22.2, 16.5), turned to 225 degrees
- moved R8 6.02 mm to (52.1, 26.7), turned to 0 degrees
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Connections:
- removed net DBG_RX: MCU2.64
- removed net INTL_OUT: MCU2.49
- removed net N$68: MCU2.62
- removed net N$69: MCU2.63
- removed net N$76: MCU2.52
- new net N$12: JP2.10, R10.2
- new net N$13: JP2.9, R11.2
- new net N$15: JP2.8, R12.2
- new net N$4: JP2.12, R8.2
- new net N$8: JP2.11, R9.2
- net CANH: now also JP1.15
- net CANL: now also JP1.14
- net CE#: now also MCU2.64; no longer MCU2.17
- net SCK: now also MCU2.49; no longer MCU2.44
- net SI: now also MCU2.52; no longer MCU2.43
- net SO: now also MCU2.63; no longer MCU2.18
- net WP#: now also MCU2.62; no longer MCU2.32
Routing:
- net VDD: track 2.89 -> 87.6 mm, vias 0 -> 2
- net CANL: track 0.00 -> 39.1 mm, vias 0 -> 2
- net N$11: track 0.00 -> 24.5 mm, vias 0 -> 2
- net GND: track 3.82 -> 28.3 mm, vias 0 -> 30
- net CANH: track 0.00 -> 22.7 mm
- net CAN_RX: track 0.00 -> 20.7 mm, vias 0 -> 2
- net CAN_TX: track 0.00 -> 19.7 mm, vias 0 -> 2
- net CE#: track 21.0 -> 8.86 mm, vias 2 -> 0
- net WP#: track 18.4 -> 6.35 mm, vias 2 -> 0
- net SO: track 19.4 -> 7.60 mm, vias 2 -> 0
- net SCL: track 0.00 -> 11.4 mm
- net N$1: track 0.00 -> 11.1 mm
- net SI: track 13.0 -> 4.00 mm, vias 2 -> 0
- net N$2: track 0.00 -> 7.99 mm
- net SDA: track 0.00 -> 6.24 mm
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