File: BMS_hw/MCU_PCB/BMS_MCUV1.0.sch (EAGLE design)
At the start: 42 parts, among them IC2 SST25VF020B804ISA, Q1 CRYSTALS-GND-LID-IQXC-42

Commit message: brd layout and sch update @14
Connections:
- removed net DBG_RX: MCU2.TDO/PMD4/RA10
- removed net INTL_OUT: MCU2.TMS/OA5IN-/AN27/C5IN1-/RPB9/RB9
- removed net N$68: MCU2.RPB12/PMD2/RB12
- removed net N$69: MCU2.RPB13/CTPLS/PMD3/RB13
- removed net N$76: MCU2.TRD1/RPC8/PMWR/RC8
- new net N$12: JP2.10, R10.2
- new net N$13: JP2.9, R11.2
- new net N$15: JP2.8, R12.2
- new net N$4: JP2.12, R8.2
- new net N$8: JP2.11, R9.2
- net CANH: now also JP1.15
- net CANL: now also JP1.14
- net CE#: now also MCU2.TDO/PMD4/RA10; no longer MCU2.PGEC1/OA1IN+/AN4/C1IN1+/C1IN3-/C2IN3-/RPB2/RB2
- net SCK: now also MCU2.TMS/OA5IN-/AN27/C5IN1-/RPB9/RB9; no longer MCU2.PGEC2/RPB6/SCK2/PMA15/RB6
- net SI: now also MCU2.TRD1/RPC8/PMWR/RC8; no longer MCU2.PGED2/RPB5/USBID1/RB5
- net SO: now also MCU2.RPB13/CTPLS/PMD3/RB13; no longer MCU2.PGED1/OA1IN-/AN5/CTCMP/C1IN1-/RTCC/RPB3/RB3
- net WP#: now also MCU2.RPB12/PMD2/RB12; no longer MCU2.RPB4/PMA8/RB4
Other:
- moved on the sheet: JP2
Changed lines of the file:
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@@
 <attribute name="VALUE" x="10.16" y="104.14" size="1.778" layer="96"/>
 </instance>
-<instance part="JP2" gate="G$1" x="111.76" y="55.88" rot="R180">
-<attribute name="NAME" x="118.11" y="40.005" size="1.778" layer="95" rot="R180"/>
-<attribute name="VALUE" x="118.11" y="76.2" size="1.778" layer="96" rot="R180"/>
+<instance part="JP2" gate="G$1" x="353.06" y="172.72" rot="MR180">
+<attribute name="NAME" x="346.71" y="156.845" size="1.778" layer="95" rot="MR180"/>
+<attribute name="VALUE" x="346.71" y="193.04" size="1.778" layer="96" rot="MR180"/>
 </instance>
 </instances>
@@
 <label x="312.42" y="93.98" size="1.778" layer="95"/>
 </segment>
+<segment>
+<pinref part="JP1" gate="A" pin="14"/>
+<wire x1="86.36" y1="76.2" x2="93.98" y2="76.2" width="0.1524" layer="91"/>
+<label x="93.98" y="76.2" size="1.778" layer="95" font="vector" ratio="12"/>
+</segment>
 </net>
 <net name="N$11" class="0">
@@
 </segment>
 <segment>
-<pinref part="MCU2" gate="G$1" pin="PGEC1/OA1IN+/AN4/C1IN1+/C1IN3-/C2IN3-/RPB2/RB2"/>
-<wire x1="35.56" y1="200.66" x2="33.02" y2="200.66" width="0.1524" layer="91"/>
-<label x="20.32" y="200.66" size="1.778" layer="95"/>
+<pinref part="MCU2" gate="G$1" pin="TDO/PMD4/RA10"/>
+<wire x1="35.56" y1="215.9" x2="33.02" y2="215.9" width="0.1524" layer="91"/>
+<label x="27.94" y="215.9" size="1.778" layer="95" font="vector" ratio="12"/>
 </segment>
 </net>
@@
 </segment>
 <segment>
-<pinref part="MCU2" gate="G$1" pin="PGED1/OA1IN-/AN5/CTCMP/C1IN1-/RTCC/RPB3/RB3"/>
-<wire x1="35.56" y1="198.12" x2="33.02" y2="198.12" width="0.1524" layer="91"/>
-<label x="20.32" y="198.12" size="1.778" layer="95"/>
+<pinref part="MCU2" gate="G$1" pin="RPB13/CTPLS/PMD3/RB13"/>
+<wire x1="35.56" y1="172.72" x2="33.02" y2="172.72" width="0.1524" layer="91"/>
 </segment>
 </net>
@@
 </segment>
 <segment>
-<pinref part="MCU2" gate="G$1" pin="RPB4/PMA8/RB4"/>
-<wire x1="35.56" y1="195.58" x2="33.02" y2="195.58" width="0.1524" layer="91"/>
-<label x="20.32" y="195.58" size="1.778" layer="95"/>
+<pinref part="MCU2" gate="G$1" pin="RPB12/PMD2/RB12"/>
+<wire x1="35.56" y1="175.26" x2="33.02" y2="175.26" width="0.1524" layer="91"/>
+<label x="27.94" y="175.26" size="1.778" layer="95"/>
 </segment>
 </net>
@@
 </segment>
 <segment>
-<pinref part="MCU2" gate="G$1" pin="PGED2/RPB5/USBID1/RB5"/>
-<wire x1="35.56" y1="193.04" x2="33.02" y2="193.04" width="0.1524" layer="91"/>
-<label x="20.32" y="193.04" size="1.778" layer="95"/>
+<pinref part="MCU2" gate="G$1" pin="TRD1/RPC8/PMWR/RC8"/>
+<wire x1="35.56" y1="149.86" x2="33.02" y2="149.86" width="0.1524" layer="91"/>
+<label x="30.48" y="149.86" size="1.778" layer="95"/>
 </segment>
 </net>
@@
 </segment>
 <segment>
-<pinref part="MCU2" gate="G$1" pin="PGEC2/RPB6/SCK2/PMA15/RB6"/>
-<wire x1="35.56" y1="190.5" x2="33.02" y2="190.5" width="0.1524" layer="91"/>
-<label x="20.32" y="190.5" size="1.778" layer="95"/>
+<pinref part="MCU2" gate="G$1" pin="TMS/OA5IN-/AN27/C5IN1-/RPB9/RB9"/>
+<wire x1="35.56" y1="182.88" x2="33.02" y2="182.88" width="0.1524" layer="91"/>
+<label x="27.94" y="182.88" size="1.778" layer="95"/>
 </segment>
 </net>
@@
 </segment>
 </net>
-<net name="INTL_OUT" class="0">
-<segment>
-<pinref part="MCU2" gate="G$1" pin="TMS/OA5IN-/AN27/C5IN1-/RPB9/RB9"/>
-<wire x1="35.56" y1="182.88" x2="33.02" y2="182.88" width="0.1524" layer="91"/>
-<label x="20.32" y="182.88" size="1.778" layer="95"/>
-</segment>
-</net>
 <net name="CANH" class="0">
 <segment>
@@
 <label x="314.96" y="99.06" size="1.778" layer="95"/>
 </segment>
+<segment>
+<pinref part="JP1" gate="A" pin="15"/>
+<wire x1="86.36" y1="78.74" x2="93.98" y2="78.74" width="0.1524" layer="91"/>
+<label x="93.98" y="78.74" size="1.778" layer="95" font="vector" ratio="12"/>
+</segment>
 </net>
 <net name="PCHG_FET" class="0">
@@
 <wire x1="35.56" y1="213.36" x2="33.02" y2="213.36" width="0.1524" layer="91"/>
 <label x="20.32" y="213.36" size="1.778" layer="95"/>
-</segment>
-</net>
-<net name="DBG_RX" class="0">
-<segment>
-<pinref part="MCU2" gate="G$1" pin="TDO/PMD4/RA10"/>
-<wire x1="35.56" y1="215.9" x2="33.02" y2="215.9" width="0.1524" layer="91"/>
-<label x="20.32" y="215.9" size="1.778" layer="95"/>
 </segment>
 </net>
@@
 </segment>
 </net>
-<net name="N$68" class="0">
-<segment>
-<pinref part="MCU2" gate="G$1" pin="RPB12/PMD2/RB12"/>
-<wire x1="35.56" y1="175.26" x2="33.02" y2="175.26" width="0.1524" layer="91"/>
-</segment>
-</net>
-<net name="N$69" class="0">
-<segment>
-<pinref part="MCU2" gate="G$1" pin="RPB13/CTPLS/PMD3/RB13"/>
-<wire x1="35.56" y1="172.72" x2="33.02" y2="172.72" width="0.1524" layer="91"/>
-</segment>
-</net>
 <net name="N$70" class="0">
 <segment>
@@
 <pinref part="MCU2" gate="G$1" pin="TRD0/RPC7/RC7"/>
 <wire x1="35.56" y1="152.4" x2="33.02" y2="152.4" width="0.1524" layer="91"/>
-</segment>
-</net>
-<net name="N$76" class="0">
-<segment>
-<pinref part="MCU2" gate="G$1" pin="TRD1/RPC8/PMWR/RC8"/>
-<wire x1="35.56" y1="149.86" x2="33.02" y2="149.86" width="0.1524" layer="91"/>
 </segment>
 </net>
@@
 </segment>
 </net>
+<net name="N$4" class="0">
+<segment>
+<pinref part="R8" gate="G$1" pin="2"/>
+<wire x1="327.66" y1="190.5" x2="335.28" y2="190.5" width="0.1524" layer="91"/>
+<wire x1="335.28" y1="190.5" x2="335.28" y2="187.96" width="0.1524" layer="91"/>
+<pinref part="JP2" gate="G$1" pin="12"/>
+<wire x1="350.52" y1="187.96" x2="335.28" y2="187.96" width="0.1524" layer="91"/>
+</segment>
+</net>
+<net name="N$8" class="0">
+<segment>
+<pinref part="R9" gate="G$1" pin="2"/>
+<wire x1="327.66" y1="180.34" x2="335.28" y2="180.34" width="0.1524" layer="91"/>
+<wire x1="335.28" y1="180.34" x2="335.28" y2="185.42" width="0.1524" layer="91"/>
+<pinref part="JP2" gate="G$1" pin="11"/>
+<wire x1="350.52" y1="185.42" x2="335.28" y2="185.42" width="0.1524" layer="91"/>
+</segment>
+</net>
+<net name="N$12" class="0">
+<segment>
+<pinref part="R10" gate="G$1" pin="2"/>
+<wire x1="327.66" y1="170.18" x2="337.82" y2="170.18" width="0.1524" layer="91"/>
+<wire x1="337.82" y1="170.18" x2="337.82" y2="182.88" width="0.1524" layer="91"/>
+<pinref part="JP2" gate="G$1" pin="10"/>
+<wire x1="350.52" y1="182.88" x2="337.82" y2="182.88" width="0.1524" layer="91"/>
+</segment>
+</net>
+<net name="N$13" class="0">
+<segment>
+<pinref part="R11" gate="G$1" pin="2"/>
+<wire x1="340.36" y1="180.34" x2="340.36" y2="160.02" width="0.1524" layer="91"/>
+<wire x1="340.36" y1="160.02" x2="327.66" y2="160.02" width="0.1524" layer="91"/>
+<pinref part="JP2" gate="G$1" pin="9"/>
+<wire x1="350.52" y1="180.34" x2="340.36" y2="180.34" width="0.1524" layer="91"/>
+</segment>
+</net>
+<net name="N$15" class="0">
+<segment>
+<wire x1="342.9" y1="177.8" x2="342.9" y2="149.86" width="0.1524" layer="91"/>
+<pinref part="R12" gate="G$1" pin="2"/>
+<wire x1="342.9" y1="149.86" x2="327.66" y2="149.86" width="0.1524" layer="91"/>
+<pinref part="JP2" gate="G$1" pin="8"/>
+<wire x1="350.52" y1="177.8" x2="342.9" y2="177.8" width="0.1524" layer="91"/>
+</segment>
+</net>

Commit message: @dsdwsw
Parts:
- removed R10: 10, ipc-7351-resistor:RESISTOR_0402
- removed R8: 2.2k, ipc-7351-resistor:RESISTOR_0402
- removed R9: 220, ipc-7351-resistor:RESISTOR_0402
- removed TP1, TP2: TP-SMD60, simpa:TP-SMD60
- R11, R12: value 100 -> 100R
Connections:
- net N$42 renamed CS
- removed net C_FET: MCU2.OA2IN+/AN1/C2IN1+/RPA1/RA1
- removed net DBG_TX: MCU2.AN9/RPA11/RA11
- removed net D_FET: MCU2.TCK/RPA7/PMD5/RA7
- removed net FAULT: MCU2.OA2OUT/AN0/C2IN4-/C4IN3-/RPA0/RA0
- removed net ICSPCLK: MCU2.AN11/C1IN2-/PMA12/RC11
- removed net ICSPDAT: MCU2.AN10/RPA12/RA12
- removed net INTL_IN2: MCU2.OA5OUT/AN25/C5IN4-/RPB7/SCK1/INT0/RB7
- removed net ISP: MCU2.OA5IN+/CDAC1/AN24/C5IN1+/C5IN3-/RPA4/T1CK/RA4
- removed net N$10: MCU2.TRD3/RPD6/RD6
- removed net N$12: JP2.10, R10.2
- removed net N$13: JP2.9, R11.2
- removed net N$15: JP2.8, R12.2
- removed net N$16: MCU2.SOSCI/RPC13/RC13, TP2.P$1
- removed net N$29: MCU2.AN12/C2IN2-/C5IN2-/PMA11/RE12
- removed net N$30: MCU2.AN13/C3IN2-/PMA10/RE13
- removed net N$4: JP2.12, R8.2
- removed net N$40: MCU2.AN14/RPE14/PMA1/RE14
- removed net N$41: MCU2.AN15/RPE15/PMA0/RE15
- removed net N$43: MCU2.RPF1/RF1
- removed net N$45: MCU2.AN18/RPG7/PMA4/RG7
- removed net N$46: MCU2.AN17/RPG8/PMA3/RG8
- removed net N$47: MCU2.AN16/RPG9/PMA2/RG9
- removed net N$5: MCU2.SOSCO/RPB8/RB8, TP1.P$1
- removed net N$66: MCU2.RPB10/PMD0/RB10
- removed net N$67: MCU2.RPB11/PMD1/RB11
- removed net N$70: MCU2.RPB15/PMD7/RB15
- removed net N$71: MCU2.OA3OUT/AN6/C3IN4-/C4IN1+/C4IN4-/RPC0/RC0
- removed net N$72: MCU2.OA3IN-/AN7/C3IN1-/C4IN1-/RPC1/PMA7/RC1
- removed net N$74: MCU2.TRCLK/RPC6/RC6
- removed net N$75: MCU2.TRD0/RPC7/RC7
- removed net N$77: MCU2.RPC9/RC9
- removed net N$78: MCU2.CDAC2/AN48/RPC10/PMA14/RC10
- removed net N$79: MCU2.D1-
- removed net N$8: JP2.11, R9.2
- removed net N$80: MCU2.D1+
- removed net N$81: MCU2.RPB14/VBUSON1/PMD6/RB14
- removed net N$9: MCU2.TRD2/RPD5/PMRD/RD5
- removed net PCHG_FET: MCU2.TDI/CDAC3/AN26/RPA8/PMA9/RA8
- removed net RX: R8.1
- removed net SCL: R12.1, R14.2
- removed net SDA: R11.1, R13.2
- removed net TX: R9.1
- new net !OLED_SCL: JP1.5, R12.2
- new net !OLED_SDA: JP1.6, R11.2
- new net CSB: JP1.4, MCU2.PGED1/OA1IN-/AN5/CTCMP/C1IN1-/RTCC/RPB3/RB3
- new net MISO: JP1.3, MCU2.PGEC1/OA1IN+/AN4/C1IN1+/C1IN3-/C2IN3-/RPB2/RB2
- new net MOSI: JP1.1, MCU2.PGED3/VREF-/OA2IN-/AN2/C2IN1-/RPB0/CTED2/RB0
- new net OLED_SCL: MCU2.OA3OUT/AN6/C3IN4-/C4IN1+/C4IN4-/RPC0/RC0, R12.1, R14.2
- new net OLED_SDA: MCU2.OA3IN-/AN7/C3IN1-/C4IN1-/RPC1/PMA7/RC1, R11.1, R13.2
- new net PGEC2: JP2.12, MCU2.PGEC2/RPB6/SCK2/PMA15/RB6
- new net PGED2: JP2.11, MCU2.PGED2/RPB5/USBID1/RB5
- new net RX_1: JP2.9, MCU2.TCK/RPA7/PMD5/RA7
- new net RX_2: JP2.8, MCU2.RPB14/VBUSON1/PMD6/RB14
- new net S-LED_1: JP5.1, MCU2.TMS/OA5IN-/AN27/C5IN1-/RPB9/RB9
- new net S-LED_2: JP5.2, MCU2.TRCLK/RPC6/RC6
- new net S-LED_3: JP5.3, MCU2.TRD0/RPC7/RC7
- new net S-LED_4: JP5.4, MCU2.TRD1/RPC8/PMWR/RC8
- new net S-LED_5: JP5.5, MCU2.TRD2/RPD5/PMRD/RD5
- new net S-LED_6: JP5.6, MCU2.TRD3/RPD6/RD6
- new net SCLK: JP1.2, MCU2.PGEC3/OA1OUT/VREF+/AN3/C1IN4-/C4IN2-/RPB1/CTED1/PMA6/RB1
- new net TX_1: JP2.7, MCU2.RPB15/PMD7/RB15
- new net TX_2: JP2.6, MCU2.AN18/RPG7/PMA4/RG7
- net !MCLR: now also JP2.10
- net 3.3V: now also JP5.7
- net CAN_RX: now also MCU2.TDI/CDAC3/AN26/RPA8/PMA9/RA8; no longer MCU2.PGED3/VREF-/OA2IN-/AN2/C2IN1-/RPB0/CTED2/RB0
- net CAN_TX: now also MCU2.AN15/RPE15/PMA0/RE15; no longer MCU2.PGEC3/OA1OUT/VREF+/AN3/C1IN4-/C4IN2-/RPB1/CTED1/PMA6/RB1
- net SCK: now also MCU2.RPB10/PMD0/RB10; no longer MCU2.TMS/OA5IN-/AN27/C5IN1-/RPB9/RB9
- net SI: now also MCU2.RPF1/RF1; no longer MCU2.TRD1/RPC8/PMWR/RC8
- net SO: now also MCU2.RPB11/PMD1/RB11; no longer MCU2.RPB13/CTPLS/PMD3/RB13
- net VDD: no longer R10.1
- net WP#: no longer MCU2.RPB12/PMD2/RB12
Other:
- moved on the sheet: JP1, JP2, JP5, R11, R12, R13, R14
